File: 12VBuck.kicad_sch (KiCad schematic)
At the start: 14 parts, among them U1 LMR51635XDDCR

Commit message: lv 1.2
Parts:
- renumbered C3 to C10, C4 to C11, C5 to C12, C6 to C13, C1 to C8, C2 to C9, R2 to R10, R1 to R9
Changed lines of the file:
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@@
-		)
-	)
-	(hierarchical_label "V_out_5V"
-		(shape output)
-		(at 2.8448 3.3496 0)
-		(effects
-			(font
-				(size 1.27 1.27)
-			)
-			(justify left)
 		)
 	)
@@
 		)
 	)
-	(hierarchical_label "Vin"
-		(shape input)
-		(at 4.3793 0.8096 180)
-		(effects
-			(font
-				(size 1.27 1.27)
-			)
-			(justify right)
-		)
-	)
 	(hierarchical_label "GND"
 		(shape bidirectional)
@@
 		(shape bidirectional)
 		(at 147.32 96.52 0)
-		(effects
-			(font
-				(size 1.27 1.27)
-			)
-			(justify left)
-		)
-	)
-	(hierarchical_label "V_out_5V"
-		(shape output)
-		(at 5.3848 5.8896 0)
 		(effects
 			(font
@@
 		(dnp no)
 		(fields_autoplaced yes)
-		(property "Reference" "#FLG02"
+		(property "Reference" "#FLG04"
 			(at 149.86 79.375 0)
 			(hide yes)
@@
 			(project "PS-PrechargeBoard"
 				(path "/74d17fe6-68d4-4bd7-954a-e2bbb58b1f1e/66a9177f-bd25-4fda-b01a-2c74f98dabbc"
-					(reference "#FLG02")
+					(reference "#FLG04")
 					(unit 1)
 				)
@@
 		(dnp no)
 		(fields_autoplaced yes)
-		(property "Reference" "C1"
+		(property "Reference" "C8"
 			(at 96.52 85.0962 0)
 			(show_name no)
@@
 			(project "PS-PrechargeBoard"
 				(path "/74d17fe6-68d4-4bd7-954a-e2bbb58b1f1e/66a9177f-bd25-4fda-b01a-2c74f98dabbc"
-					(reference "C1")
+					(reference "C8")
 					(unit 1)
 				)
@@
 		(dnp no)
 		(fields_autoplaced yes)
-		(property "Reference" "#FLG04"
+		(property "Reference" "#FLG06"
 			(at 179.07 84.455 0)
 			(hide yes)
@@
 			(project "PS-PrechargeBoard"
 				(path "/74d17fe6-68d4-4bd7-954a-e2bbb58b1f1e/66a9177f-bd25-4fda-b01a-2c74f98dabbc"
-					(reference "#FLG04")
+					(reference "#FLG06")
 					(unit 1)
 				)
@@
 		(dnp no)
 		(fields_autoplaced yes)
-		(property "Reference" "#FLG01"
+		(property "Reference" "#FLG03"
 			(at 88.9 79.375 0)
 			(hide yes)
@@
 			(project "PS-PrechargeBoard"
 				(path "/74d17fe6-68d4-4bd7-954a-e2bbb58b1f1e/66a9177f-bd25-4fda-b01a-2c74f98dabbc"
-					(reference "#FLG01")
+					(reference "#FLG03")
 					(unit 1)
 				)
@@
 		(in_pos_files yes)
 		(dnp no)
-		(property "Reference" "C4"
+		(property "Reference" "C11"
 			(at 164.084 93.98 0)
 			(show_name no)
@@
 			(project "PS-PrechargeBoard"
 				(path "/74d17fe6-68d4-4bd7-954a-e2bbb58b1f1e/66a9177f-bd25-4fda-b01a-2c74f98dabbc"
-					(reference "C4")
+					(reference "C11")
 					(unit 1)
 				)
@@
 		(in_pos_files yes)
 		(dnp no)
-		(property "Reference" "C6"
+		(property "Reference" "C13"
 			(at 189.992 93.98 0)
 			(show_name no)
@@
 			(project "PS-PrechargeBoard"
 				(path "/74d17fe6-68d4-4bd7-954a-e2bbb58b1f1e/66a9177f-bd25-4fda-b01a-2c74f98dabbc"
-					(reference "C6")
+					(reference "C13")
 					(unit 1)
 				)
@@
 		(in_pos_files yes)
 		(dnp no)
-		(property "Reference" "C3"
+		(property "Reference" "C10"
 			(at 156.718 80.01 0)
 			(show_name no)
@@
 			(project "PS-PrechargeBoard"
 				(path "/74d17fe6-68d4-4bd7-954a-e2bbb58b1f1e/66a9177f-bd25-4fda-b01a-2c74f98dabbc"
-					(reference "C3")
+					(reference "C10")
 					(unit 1)
 				)
@@
 		(in_pos_files yes)
 		(dnp no)
-		(property "Reference" "#FLG03"
+		(property "Reference" "#FLG05"
 			(at 149.86 84.455 0)
 			(hide yes)
@@
 			(project "PS-PrechargeBoard"
 				(path "/74d17fe6-68d4-4bd7-954a-e2bbb58b1f1e/66a9177f-bd25-4fda-b01a-2c74f98dabbc"
-					(reference "#FLG03")
+					(reference "#FLG05")
 					(unit 1)
 				)
@@
 		(dnp no)
 		(fields_autoplaced yes)
-		(property "Reference" "R1"
+		(property "Reference" "R9"
 			(at 227.33 85.0899 0)
 			(show_name no)
@@
 			(project "PS-PrechargeBoard"
 				(path "/74d17fe6-68d4-4bd7-954a-e2bbb58b1f1e/66a9177f-bd25-4fda-b01a-2c74f98dabbc"
-					(reference "R1")
+					(reference "R9")
 					(unit 1)
 				)
@@
 		(dnp no)
 		(fields_autoplaced yes)
-		(property "Reference" "C2"
+		(property "Reference" "C9"
 			(at 105.41 87.6362 0)
 			(show_name no)
@@
 			(project "PS-PrechargeBoard"
 				(path "/74d17fe6-68d4-4bd7-954a-e2bbb58b1f1e/66a9177f-bd25-4fda-b01a-2c74f98dabbc"
-					(reference "C2")
+					(reference "C9")
 					(unit 1)
 				)
@@
 		(dnp no)
 		(fields_autoplaced yes)
-		(property "Reference" "R2"
+		(property "Reference" "R10"
 			(at 227.33 92.7099 0)
 			(show_name no)
@@
 			(project "PS-PrechargeBoard"
 				(path "/74d17fe6-68d4-4bd7-954a-e2bbb58b1f1e/66a9177f-bd25-4fda-b01a-2c74f98dabbc"
-					(reference "R2")
+					(reference "R10")
 					(unit 1)
 				)
@@
 		(in_pos_files yes)
 		(dnp no)
-		(property "Reference" "C5"
+		(property "Reference" "C12"
 			(at 173.482 94.234 0)
 			(show_name no)
@@
 			(project "PS-PrechargeBoard"
 				(path "/74d17fe6-68d4-4bd7-954a-e2bbb58b1f1e/66a9177f-bd25-4fda-b01a-2c74f98dabbc"
-					(reference "C5")
-					(unit 1)
-				)
+					(reference "C12")
+					(unit 1)
+				)

Commit message: hv 1.0
Parts:
- renumbered R9 to R13, R10 to R14, TP1 to TP5, TP2 to TP6, TP3 to TP7, TP4 to TP8
Changed lines of the file:
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@@
 		(dnp no)
 		(fields_autoplaced yes)
-		(property "Reference" "#FLG04"
+		(property "Reference" "#FLG06"
 			(at 149.86 79.375 0)
 			(hide yes)
@@
 			(project "PS-PrechargeBoard"
 				(path "/74d17fe6-68d4-4bd7-954a-e2bbb58b1f1e/66a9177f-bd25-4fda-b01a-2c74f98dabbc"
-					(reference "#FLG04")
+					(reference "#FLG06")
 					(unit 1)
 				)
@@
 		(in_pos_files yes)
 		(dnp no)
-		(property "Reference" "TP1"
+		(property "Reference" "TP5"
 			(at 229.87 123.6979 0)
 			(hide yes)
@@
 			(project "PS-PrechargeBoard"
 				(path "/74d17fe6-68d4-4bd7-954a-e2bbb58b1f1e/66a9177f-bd25-4fda-b01a-2c74f98dabbc"
-					(reference "TP1")
+					(reference "TP5")
 					(unit 1)
 				)
@@
 		(in_pos_files yes)
 		(dnp no)
-		(property "Reference" "TP3"
+		(property "Reference" "TP7"
 			(at 242.57 123.6979 0)
 			(hide yes)
@@
 			(project "PS-PrechargeBoard"
 				(path "/74d17fe6-68d4-4bd7-954a-e2bbb58b1f1e/66a9177f-bd25-4fda-b01a-2c74f98dabbc"
-					(reference "TP3")
+					(reference "TP7")
 					(unit 1)
 				)
@@
 		(in_pos_files yes)
 		(dnp no)
-		(property "Reference" "TP2"
+		(property "Reference" "TP6"
 			(at 229.87 136.3979 0)
 			(hide yes)
@@
 			(project "PS-PrechargeBoard"
 				(path "/74d17fe6-68d4-4bd7-954a-e2bbb58b1f1e/66a9177f-bd25-4fda-b01a-2c74f98dabbc"
-					(reference "TP2")
+					(reference "TP6")
 					(unit 1)
 				)
@@
 		(in_pos_files yes)
 		(dnp no)
-		(property "Reference" "TP4"
+		(property "Reference" "TP8"
 			(at 242.57 136.3979 0)
 			(hide yes)
@@
 			(project "PS-PrechargeBoard"
 				(path "/74d17fe6-68d4-4bd7-954a-e2bbb58b1f1e/66a9177f-bd25-4fda-b01a-2c74f98dabbc"
-					(reference "TP4")
+					(reference "TP8")
 					(unit 1)
 				)
@@
 		(dnp no)
 		(fields_autoplaced yes)
-		(property "Reference" "#FLG06"
+		(property "Reference" "#FLG08"
 			(at 179.07 84.455 0)
 			(hide yes)
@@
 			(project "PS-PrechargeBoard"
 				(path "/74d17fe6-68d4-4bd7-954a-e2bbb58b1f1e/66a9177f-bd25-4fda-b01a-2c74f98dabbc"
-					(reference "#FLG06")
+					(reference "#FLG08")
 					(unit 1)
 				)
@@
 		(dnp no)
 		(fields_autoplaced yes)
-		(property "Reference" "#FLG03"
+		(property "Reference" "#FLG05"
 			(at 88.9 79.375 0)
 			(hide yes)
@@
 			(project "PS-PrechargeBoard"
 				(path "/74d17fe6-68d4-4bd7-954a-e2bbb58b1f1e/66a9177f-bd25-4fda-b01a-2c74f98dabbc"
-					(reference "#FLG03")
+					(reference "#FLG05")
 					(unit 1)
 				)
@@
 		(in_pos_files yes)
 		(dnp no)
-		(property "Reference" "#FLG05"
+		(property "Reference" "#FLG07"
 			(at 149.86 84.455 0)
 			(hide yes)
@@
 			(project "PS-PrechargeBoard"
 				(path "/74d17fe6-68d4-4bd7-954a-e2bbb58b1f1e/66a9177f-bd25-4fda-b01a-2c74f98dabbc"
-					(reference "#FLG05")
+					(reference "#FLG07")
 					(unit 1)
 				)
@@
 		(dnp no)
 		(fields_autoplaced yes)
-		(property "Reference" "R9"
+		(property "Reference" "R13"
 			(at 227.33 85.0899 0)
 			(show_name no)
@@
 			(project "PS-PrechargeBoard"
 				(path "/74d17fe6-68d4-4bd7-954a-e2bbb58b1f1e/66a9177f-bd25-4fda-b01a-2c74f98dabbc"
-					(reference "R9")
+					(reference "R13")
 					(unit 1)
 				)
@@
 		(dnp no)
 		(fields_autoplaced yes)
-		(property "Reference" "R10"
+		(property "Reference" "R14"
 			(at 227.33 92.7099 0)
 			(show_name no)
@@
 			(project "PS-PrechargeBoard"
 				(path "/74d17fe6-68d4-4bd7-954a-e2bbb58b1f1e/66a9177f-bd25-4fda-b01a-2c74f98dabbc"
-					(reference "R10")
-					(unit 1)
-				)
+					(reference "R14")
+					(unit 1)
+				)

Commit message: hv 1.1
Parts:
- renumbered R13 to R12, R14 to R13
Changed lines of the file:
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@@
 		(dnp no)
 		(fields_autoplaced yes)
-		(property "Reference" "R13"
+		(property "Reference" "R12"
 			(at 227.33 85.0899 0)
 			(show_name no)
@@
 			(project "PS-PrechargeBoard"
 				(path "/74d17fe6-68d4-4bd7-954a-e2bbb58b1f1e/66a9177f-bd25-4fda-b01a-2c74f98dabbc"
-					(reference "R13")
+					(reference "R12")
 					(unit 1)
 				)
@@
 		(dnp no)
 		(fields_autoplaced yes)
-		(property "Reference" "R14"
+		(property "Reference" "R13"
 			(at 227.33 92.7099 0)
 			(show_name no)
@@
 			(project "PS-PrechargeBoard"
 				(path "/74d17fe6-68d4-4bd7-954a-e2bbb58b1f1e/66a9177f-bd25-4fda-b01a-2c74f98dabbc"
-					(reference "R14")
-					(unit 1)
-				)
+					(reference "R13")
+					(unit 1)
+				)

Commit message: hv 1.3
Parts:
- renumbered C8 to C?, C11 to C?, C13 to C?, C10 to C?, C9 to C?, C12 to C?, L1 to L?, R12 to R?, R13 to R?, TP5 to TP?, TP7 to TP?, TP6 to TP?, TP8 to TP?, U1 to U?
