File: 12VBuck.kicad_sch (KiCad schematic)
At the start: 14 parts

Commit message: CAN nano & CAN debug nano
Parts:
- gave numbers to parts that had none: 14

Commit message: battery voltage & motor voltage
Parts:
- renumbered C28 to C16, C29 to C17, C30 to C18, C31 to C19, C32 to C20, C33 to C21, R19 to R23, R20 to R24, TP1 to TP11, TP2 to TP12, TP3 to TP13, TP4 to TP14, U2 to U4
Changed lines of the file:
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@@
 		(dnp no)
 		(fields_autoplaced yes)
-		(property "Reference" "#FLG03"
+		(property "Reference" "#FLG08"
 			(at 149.86 79.375 0)
 			(hide yes)
@@
 			(project "PS-PrechargeBoard"
 				(path "/74d17fe6-68d4-4bd7-954a-e2bbb58b1f1e/0def18ef-81e8-47ac-b719-2d9f8237a855/cd8ca406-e250-4c51-b6e8-7777acbf36c8"
-					(reference "#FLG03")
+					(reference "#FLG08")
 					(unit 1)
 				)
@@
 		(dnp no)
 		(fields_autoplaced yes)
-		(property "Reference" "C28"
+		(property "Reference" "C16"
 			(at 96.52 85.0962 0)
 			(show_name no)
@@
 			(project "PS-PrechargeBoard"
 				(path "/74d17fe6-68d4-4bd7-954a-e2bbb58b1f1e/0def18ef-81e8-47ac-b719-2d9f8237a855/cd8ca406-e250-4c51-b6e8-7777acbf36c8"
-					(reference "C28")
+					(reference "C16")
 					(unit 1)
 				)
@@
 		(in_pos_files yes)
 		(dnp no)
-		(property "Reference" "TP1"
+		(property "Reference" "TP11"
 			(at 229.87 123.6979 0)
 			(hide yes)
@@
 			(project "PS-PrechargeBoard"
 				(path "/74d17fe6-68d4-4bd7-954a-e2bbb58b1f1e/0def18ef-81e8-47ac-b719-2d9f8237a855/cd8ca406-e250-4c51-b6e8-7777acbf36c8"
-					(reference "TP1")
+					(reference "TP11")
 					(unit 1)
 				)
@@
 		(in_pos_files yes)
 		(dnp no)
-		(property "Reference" "TP3"
+		(property "Reference" "TP13"
 			(at 242.57 123.6979 0)
 			(hide yes)
@@
 			(project "PS-PrechargeBoard"
 				(path "/74d17fe6-68d4-4bd7-954a-e2bbb58b1f1e/0def18ef-81e8-47ac-b719-2d9f8237a855/cd8ca406-e250-4c51-b6e8-7777acbf36c8"
-					(reference "TP3")
+					(reference "TP13")
 					(unit 1)
 				)
@@
 		(in_pos_files yes)
 		(dnp no)
-		(property "Reference" "TP2"
+		(property "Reference" "TP12"
 			(at 229.87 136.3979 0)
 			(hide yes)
@@
 			(project "PS-PrechargeBoard"
 				(path "/74d17fe6-68d4-4bd7-954a-e2bbb58b1f1e/0def18ef-81e8-47ac-b719-2d9f8237a855/cd8ca406-e250-4c51-b6e8-7777acbf36c8"
-					(reference "TP2")
+					(reference "TP12")
 					(unit 1)
 				)
@@
 		(dnp no)
 		(fields_autoplaced yes)
-		(property "Reference" "U2"
+		(property "Reference" "U4"
 			(at 129.54 71.12 0)
 			(show_name no)
@@
 			(project "PS-PrechargeBoard"
 				(path "/74d17fe6-68d4-4bd7-954a-e2bbb58b1f1e/0def18ef-81e8-47ac-b719-2d9f8237a855/cd8ca406-e250-4c51-b6e8-7777acbf36c8"
-					(reference "U2")
+					(reference "U4")
 					(unit 1)
 				)
@@
 		(in_pos_files yes)
 		(dnp no)
-		(property "Reference" "TP4"
+		(property "Reference" "TP14"
 			(at 242.57 136.3979 0)
 			(hide yes)
@@
 			(project "PS-PrechargeBoard"
 				(path "/74d17fe6-68d4-4bd7-954a-e2bbb58b1f1e/0def18ef-81e8-47ac-b719-2d9f8237a855/cd8ca406-e250-4c51-b6e8-7777acbf36c8"
-					(reference "TP4")
+					(reference "TP14")
 					(unit 1)
 				)
@@
 		(dnp no)
 		(fields_autoplaced yes)
-		(property "Reference" "#FLG05"
+		(property "Reference" "#FLG010"
 			(at 179.07 84.455 0)
 			(hide yes)
@@
 			(project "PS-PrechargeBoard"
 				(path "/74d17fe6-68d4-4bd7-954a-e2bbb58b1f1e/0def18ef-81e8-47ac-b719-2d9f8237a855/cd8ca406-e250-4c51-b6e8-7777acbf36c8"
-					(reference "#FLG05")
+					(reference "#FLG010")
 					(unit 1)
 				)
@@
 		(dnp no)
 		(fields_autoplaced yes)
-		(property "Reference" "#FLG02"
+		(property "Reference" "#FLG07"
 			(at 88.9 79.375 0)
 			(hide yes)
@@
 			(project "PS-PrechargeBoard"
 				(path "/74d17fe6-68d4-4bd7-954a-e2bbb58b1f1e/0def18ef-81e8-47ac-b719-2d9f8237a855/cd8ca406-e250-4c51-b6e8-7777acbf36c8"
-					(reference "#FLG02")
+					(reference "#FLG07")
 					(unit 1)
 				)
@@
 		(in_pos_files yes)
 		(dnp no)
-		(property "Reference" "C31"
+		(property "Reference" "C19"
 			(at 164.084 93.98 0)
 			(show_name no)
@@
 			(project "PS-PrechargeBoard"
 				(path "/74d17fe6-68d4-4bd7-954a-e2bbb58b1f1e/0def18ef-81e8-47ac-b719-2d9f8237a855/cd8ca406-e250-4c51-b6e8-7777acbf36c8"
-					(reference "C31")
+					(reference "C19")
 					(unit 1)
 				)
@@
 		(in_pos_files yes)
 		(dnp no)
-		(property "Reference" "C33"
+		(property "Reference" "C21"
 			(at 189.992 93.98 0)
 			(show_name no)
@@
 			(project "PS-PrechargeBoard"
 				(path "/74d17fe6-68d4-4bd7-954a-e2bbb58b1f1e/0def18ef-81e8-47ac-b719-2d9f8237a855/cd8ca406-e250-4c51-b6e8-7777acbf36c8"
-					(reference "C33")
+					(reference "C21")
 					(unit 1)
 				)
@@
 		(in_pos_files yes)
 		(dnp no)
-		(property "Reference" "C30"
+		(property "Reference" "C18"
 			(at 156.718 80.01 0)
 			(show_name no)
@@
 			(project "PS-PrechargeBoard"
 				(path "/74d17fe6-68d4-4bd7-954a-e2bbb58b1f1e/0def18ef-81e8-47ac-b719-2d9f8237a855/cd8ca406-e250-4c51-b6e8-7777acbf36c8"
-					(reference "C30")
+					(reference "C18")
 					(unit 1)
 				)
@@
 		(in_pos_files yes)
 		(dnp no)
-		(property "Reference" "#FLG04"
+		(property "Reference" "#FLG09"
 			(at 149.86 84.455 0)
 			(hide yes)
@@
 			(project "PS-PrechargeBoard"
 				(path "/74d17fe6-68d4-4bd7-954a-e2bbb58b1f1e/0def18ef-81e8-47ac-b719-2d9f8237a855/cd8ca406-e250-4c51-b6e8-7777acbf36c8"
-					(reference "#FLG04")
+					(reference "#FLG09")
 					(unit 1)
 				)
@@
 		(dnp no)
 		(fields_autoplaced yes)
-		(property "Reference" "R19"
+		(property "Reference" "R23"
 			(at 227.33 85.0899 0)
 			(show_name no)
@@
 			(project "PS-PrechargeBoard"
 				(path "/74d17fe6-68d4-4bd7-954a-e2bbb58b1f1e/0def18ef-81e8-47ac-b719-2d9f8237a855/cd8ca406-e250-4c51-b6e8-7777acbf36c8"
-					(reference "R19")
+					(reference "R23")
 					(unit 1)
 				)
@@
 		(dnp no)
 		(fields_autoplaced yes)
-		(property "Reference" "C29"
+		(property "Reference" "C17"
 			(at 105.41 87.6362 0)
 			(show_name no)
@@
 			(project "PS-PrechargeBoard"
 				(path "/74d17fe6-68d4-4bd7-954a-e2bbb58b1f1e/0def18ef-81e8-47ac-b719-2d9f8237a855/cd8ca406-e250-4c51-b6e8-7777acbf36c8"
-					(reference "C29")
+					(reference "C17")
 					(unit 1)
 				)
@@
 		(dnp no)
 		(fields_autoplaced yes)
-		(property "Reference" "R20"
+		(property "Reference" "R24"
 			(at 227.33 92.7099 0)
 			(show_name no)
@@
 			(project "PS-PrechargeBoard"
 				(path "/74d17fe6-68d4-4bd7-954a-e2bbb58b1f1e/0def18ef-81e8-47ac-b719-2d9f8237a855/cd8ca406-e250-4c51-b6e8-7777acbf36c8"
-					(reference "R20")
+					(reference "R24")
 					(unit 1)
 				)
@@
 		(in_pos_files yes)
 		(dnp no)
-		(property "Reference" "C32"
+		(property "Reference" "C20"
 			(at 173.482 94.234 0)
 			(show_name no)
@@
 			(project "PS-PrechargeBoard"
 				(path "/74d17fe6-68d4-4bd7-954a-e2bbb58b1f1e/0def18ef-81e8-47ac-b719-2d9f8237a855/cd8ca406-e250-4c51-b6e8-7777acbf36c8"
-					(reference "C32")
-					(unit 1)
-				)
+					(reference "C20")
+					(unit 1)
+				)

Commit message: mini review notes
Parts:
- U4: now not fitted
Changed lines of the file:
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@@
 		(dnp no)
 		(fields_autoplaced yes)
-		(property "Reference" "#FLG08"
+		(property "Reference" "#FLG06"
 			(at 149.86 79.375 0)
 			(hide yes)
@@
 			(project "PS-PrechargeBoard"
 				(path "/74d17fe6-68d4-4bd7-954a-e2bbb58b1f1e/0def18ef-81e8-47ac-b719-2d9f8237a855/cd8ca406-e250-4c51-b6e8-7777acbf36c8"
-					(reference "#FLG08")
+					(reference "#FLG06")
 					(unit 1)
 				)
@@
 		(on_board yes)
 		(in_pos_files yes)
-		(dnp no)
+		(dnp yes)
 		(fields_autoplaced yes)
 		(property "Reference" "U4"
@@
 		(dnp no)
 		(fields_autoplaced yes)
-		(property "Reference" "#FLG010"
+		(property "Reference" "#FLG08"
 			(at 179.07 84.455 0)
 			(hide yes)
@@
 			(project "PS-PrechargeBoard"
 				(path "/74d17fe6-68d4-4bd7-954a-e2bbb58b1f1e/0def18ef-81e8-47ac-b719-2d9f8237a855/cd8ca406-e250-4c51-b6e8-7777acbf36c8"
-					(reference "#FLG010")
+					(reference "#FLG08")
 					(unit 1)
 				)
@@
 		(dnp no)
 		(fields_autoplaced yes)
-		(property "Reference" "#FLG07"
+		(property "Reference" "#FLG05"
 			(at 88.9 79.375 0)
 			(hide yes)
@@
 			(project "PS-PrechargeBoard"
 				(path "/74d17fe6-68d4-4bd7-954a-e2bbb58b1f1e/0def18ef-81e8-47ac-b719-2d9f8237a855/cd8ca406-e250-4c51-b6e8-7777acbf36c8"
-					(reference "#FLG07")
+					(reference "#FLG05")
 					(unit 1)
 				)
@@
 		(in_pos_files yes)
 		(dnp no)
-		(property "Reference" "#FLG09"
+		(property "Reference" "#FLG07"
 			(at 149.86 84.455 0)
 			(hide yes)
@@
 			(project "PS-PrechargeBoard"
 				(path "/74d17fe6-68d4-4bd7-954a-e2bbb58b1f1e/0def18ef-81e8-47ac-b719-2d9f8237a855/cd8ca406-e250-4c51-b6e8-7777acbf36c8"
-					(reference "#FLG09")
-					(unit 1)
-				)
+					(reference "#FLG07")
+					(unit 1)
+				)

Commit message: shifted hierarchical sheets
Parts:
- renumbered C16 to C?, C19 to C?, C21 to C?, C18 to C?, C17 to C?, C20 to C?, L1 to L?, R23 to R?, R24 to R?, TP11 to TP?, TP13 to TP?, TP12 to TP?, TP14 to TP?, U4 to U?

Commit message: V_OUT_BAT & V_OUT_MOT & PRECHARGE_CTRL to MCU
Parts:
- gave numbers to parts that had none: 14
Changed lines of the file:
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@@
 		(dnp no)
 		(fields_autoplaced yes)
-		(property "Reference" "#FLG012"
+		(property "Reference" "#FLG06"
 			(at 149.86 79.375 0)
 			(hide yes)
@@
 			(project "PS-PrechargeBoard"
 				(path "/74d17fe6-68d4-4bd7-954a-e2bbb58b1f1e/88068a34-f22d-4106-a80b-45e353d7d848"
-					(reference "#FLG012")
+					(reference "#FLG06")
 					(unit 1)
 				)
@@
 		(dnp no)
 		(fields_autoplaced yes)
-		(property "Reference" "C?"
+		(property "Reference" "C22"
 			(at 96.52 85.0962 0)
 			(show_name no)
@@
 			(project "PS-PrechargeBoard"
 				(path "/74d17fe6-68d4-4bd7-954a-e2bbb58b1f1e/88068a34-f22d-4106-a80b-45e353d7d848"
-					(reference "C?")
+					(reference "C22")
 					(unit 1)
 				)
@@
 		(in_pos_files yes)
 		(dnp no)
-		(property "Reference" "TP?"
+		(property "Reference" "TP17"
 			(at 229.87 123.6979 0)
 			(hide yes)
@@
 			(project "PS-PrechargeBoard"
 				(path "/74d17fe6-68d4-4bd7-954a-e2bbb58b1f1e/88068a34-f22d-4106-a80b-45e353d7d848"
-					(reference "TP?")
+					(reference "TP17")
 					(unit 1)
 				)
@@
 		(in_pos_files yes)
 		(dnp no)
-		(property "Reference" "L?"
+		(property "Reference" "L1"
 			(at 161.29 87.884 90)
 			(show_name no)
@@
 			(project "PS-PrechargeBoard"
 				(path "/74d17fe6-68d4-4bd7-954a-e2bbb58b1f1e/88068a34-f22d-4106-a80b-45e353d7d848"
-					(reference "L?")
+					(reference "L1")
 					(unit 1)
 				)
@@
 		(in_pos_files yes)
 		(dnp no)
-		(property "Reference" "TP?"
+		(property "Reference" "TP19"
 			(at 242.57 123.6979 0)
 			(hide yes)
@@
 			(project "PS-PrechargeBoard"
 				(path "/74d17fe6-68d4-4bd7-954a-e2bbb58b1f1e/88068a34-f22d-4106-a80b-45e353d7d848"
-					(reference "TP?")
+					(reference "TP19")
 					(unit 1)
 				)
@@
 		(in_pos_files yes)
 		(dnp no)
-		(property "Reference" "TP?"
+		(property "Reference" "TP18"
 			(at 229.87 136.3979 0)
 			(hide yes)
@@
 			(project "PS-PrechargeBoard"
 				(path "/74d17fe6-68d4-4bd7-954a-e2bbb58b1f1e/88068a34-f22d-4106-a80b-45e353d7d848"
-					(reference "TP?")
+					(reference "TP18")
 					(unit 1)
 				)
@@
 		(dnp yes)
 		(fields_autoplaced yes)
-		(property "Reference" "U?"
+		(property "Reference" "U4"
 			(at 129.54 71.12 0)
 			(show_name no)
@@
 			(project "PS-PrechargeBoard"
 				(path "/74d17fe6-68d4-4bd7-954a-e2bbb58b1f1e/88068a34-f22d-4106-a80b-45e353d7d848"
-					(reference "U?")
+					(reference "U4")
 					(unit 1)
 				)
@@
 		(in_pos_files yes)
 		(dnp no)
-		(property "Reference" "TP?"
+		(property "Reference" "TP20"
 			(at 242.57 136.3979 0)
 			(hide yes)
@@
 			(project "PS-PrechargeBoard"
 				(path "/74d17fe6-68d4-4bd7-954a-e2bbb58b1f1e/88068a34-f22d-4106-a80b-45e353d7d848"
-					(reference "TP?")
+					(reference "TP20")
 					(unit 1)
 				)
@@
 		(dnp no)
 		(fields_autoplaced yes)
-		(property "Reference" "#FLG014"
+		(property "Reference" "#FLG08"
 			(at 179.07 84.455 0)
 			(hide yes)
@@
 			(project "PS-PrechargeBoard"
 				(path "/74d17fe6-68d4-4bd7-954a-e2bbb58b1f1e/88068a34-f22d-4106-a80b-45e353d7d848"
-					(reference "#FLG014")
+					(reference "#FLG08")
 					(unit 1)
 				)
@@
 		(dnp no)
 		(fields_autoplaced yes)
-		(property "Reference" "#FLG011"
+		(property "Reference" "#FLG05"
 			(at 88.9 79.375 0)
 			(hide yes)
@@
 			(project "PS-PrechargeBoard"
 				(path "/74d17fe6-68d4-4bd7-954a-e2bbb58b1f1e/88068a34-f22d-4106-a80b-45e353d7d848"
-					(reference "#FLG011")
+					(reference "#FLG05")
 					(unit 1)
 				)
@@
 		(in_pos_files yes)
 		(dnp no)
-		(property "Reference" "C?"
+		(property "Reference" "C25"
 			(at 164.084 93.98 0)
 			(show_name no)
@@
 			(project "PS-PrechargeBoard"
 				(path "/74d17fe6-68d4-4bd7-954a-e2bbb58b1f1e/88068a34-f22d-4106-a80b-45e353d7d848"
-					(reference "C?")
+					(reference "C25")
 					(unit 1)
 				)
@@
 		(in_pos_files yes)
 		(dnp no)
-		(property "Reference" "C?"
+		(property "Reference" "C27"
 			(at 189.992 93.98 0)
 			(show_name no)
@@
 			(project "PS-PrechargeBoard"
 				(path "/74d17fe6-68d4-4bd7-954a-e2bbb58b1f1e/88068a34-f22d-4106-a80b-45e353d7d848"
-					(reference "C?")
+					(reference "C27")
 					(unit 1)
 				)
@@
 		(in_pos_files yes)
 		(dnp no)
-		(property "Reference" "C?"
+		(property "Reference" "C24"
 			(at 156.718 80.01 0)
 			(show_name no)
@@
 			(project "PS-PrechargeBoard"
 				(path "/74d17fe6-68d4-4bd7-954a-e2bbb58b1f1e/88068a34-f22d-4106-a80b-45e353d7d848"
-					(reference "C?")
+					(reference "C24")
 					(unit 1)
 				)
@@
 		(in_pos_files yes)
 		(dnp no)
-		(property "Reference" "#FLG013"
+		(property "Reference" "#FLG07"
 			(at 149.86 84.455 0)
 			(hide yes)
@@
 			(project "PS-PrechargeBoard"
 				(path "/74d17fe6-68d4-4bd7-954a-e2bbb58b1f1e/88068a34-f22d-4106-a80b-45e353d7d848"
-					(reference "#FLG013")
+					(reference "#FLG07")
 					(unit 1)
 				)
@@
 		(dnp no)
 		(fields_autoplaced yes)
-		(property "Reference" "R?"
+		(property "Reference" "R29"
 			(at 227.33 85.0899 0)
 			(show_name no)
@@
 			(project "PS-PrechargeBoard"
 				(path "/74d17fe6-68d4-4bd7-954a-e2bbb58b1f1e/88068a34-f22d-4106-a80b-45e353d7d848"
-					(reference "R?")
+					(reference "R29")
 					(unit 1)
 				)
@@
 		(dnp no)
 		(fields_autoplaced yes)
-		(property "Reference" "C?"
+		(property "Reference" "C23"
 			(at 105.41 87.6362 0)
 			(show_name no)
@@
 			(project "PS-PrechargeBoard"
 				(path "/74d17fe6-68d4-4bd7-954a-e2bbb58b1f1e/88068a34-f22d-4106-a80b-45e353d7d848"
-					(reference "C?")
+					(reference "C23")
 					(unit 1)
 				)
@@
 		(dnp no)
 		(fields_autoplaced yes)
-		(property "Reference" "R?"
+		(property "Reference" "R30"
 			(at 227.33 92.7099 0)
 			(show_name no)
@@
 			(project "PS-PrechargeBoard"
 				(path "/74d17fe6-68d4-4bd7-954a-e2bbb58b1f1e/88068a34-f22d-4106-a80b-45e353d7d848"
-					(reference "R?")
+					(reference "R30")
 					(unit 1)
 				)
@@
 		(in_pos_files yes)
 		(dnp no)
-		(property "Reference" "C?"
+		(property "Reference" "C26"
 			(at 173.482 94.234 0)
 			(show_name no)
@@
 			(project "PS-PrechargeBoard"
 				(path "/74d17fe6-68d4-4bd7-954a-e2bbb58b1f1e/88068a34-f22d-4106-a80b-45e353d7d848"
-					(reference "C?")
-					(unit 1)
-				)
+					(reference "C26")
+					(unit 1)
+				)
