File: 12VBuck.kicad_sch (KiCad schematic)
At the start: 14 parts, among them U4 LMR51635XDDCR

Commit message: precharges & voltage sensors
Parts:
- renumbered C22 to C18, C23 to C19, C24 to C20, C25 to C21, C26 to C22, C27 to C23, R29 to R24, R30 to R25, TP17 to TP11, TP18 to TP12, TP19 to TP13, TP20 to TP14, U4 to U3
Changed lines of the file:
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@@
 		(dnp no)
 		(fields_autoplaced yes)
-		(property "Reference" "#FLG06"
+		(property "Reference" "#FLG02"
 			(at 149.86 79.375 0)
 			(hide yes)
@@
 		(instances
 			(project "PS-PrechargeBoard"
-				(path "/74d17fe6-68d4-4bd7-954a-e2bbb58b1f1e/88068a34-f22d-4106-a80b-45e353d7d848"
-					(reference "#FLG06")
+				(path "/74d17fe6-68d4-4bd7-954a-e2bbb58b1f1e/c6e51092-efec-40a8-afae-63cae62691f2/d0a2e77c-6f3b-4bbc-a3d8-ef9f85477fa8"
+					(reference "#FLG02")
 					(unit 1)
 				)
@@
 		(dnp no)
 		(fields_autoplaced yes)
-		(property "Reference" "C22"
+		(property "Reference" "C18"
 			(at 96.52 85.0962 0)
 			(show_name no)
@@
 		(instances
 			(project "PS-PrechargeBoard"
-				(path "/74d17fe6-68d4-4bd7-954a-e2bbb58b1f1e/88068a34-f22d-4106-a80b-45e353d7d848"
-					(reference "C22")
+				(path "/74d17fe6-68d4-4bd7-954a-e2bbb58b1f1e/c6e51092-efec-40a8-afae-63cae62691f2/d0a2e77c-6f3b-4bbc-a3d8-ef9f85477fa8"
+					(reference "C18")
 					(unit 1)
 				)
@@
 		(in_pos_files yes)
 		(dnp no)
-		(property "Reference" "TP17"
+		(property "Reference" "TP11"
 			(at 229.87 123.6979 0)
 			(hide yes)
@@
 		(instances
 			(project "PS-PrechargeBoard"
-				(path "/74d17fe6-68d4-4bd7-954a-e2bbb58b1f1e/88068a34-f22d-4106-a80b-45e353d7d848"
-					(reference "TP17")
+				(path "/74d17fe6-68d4-4bd7-954a-e2bbb58b1f1e/c6e51092-efec-40a8-afae-63cae62691f2/d0a2e77c-6f3b-4bbc-a3d8-ef9f85477fa8"
+					(reference "TP11")
 					(unit 1)
 				)
@@
 		(instances
 			(project "PS-PrechargeBoard"
-				(path "/74d17fe6-68d4-4bd7-954a-e2bbb58b1f1e/88068a34-f22d-4106-a80b-45e353d7d848"
+				(path "/74d17fe6-68d4-4bd7-954a-e2bbb58b1f1e/c6e51092-efec-40a8-afae-63cae62691f2/d0a2e77c-6f3b-4bbc-a3d8-ef9f85477fa8"
 					(reference "L1")
 					(unit 1)
@@
 		(in_pos_files yes)
 		(dnp no)
-		(property "Reference" "TP19"
+		(property "Reference" "TP13"
 			(at 242.57 123.6979 0)
 			(hide yes)
@@
 		(instances
 			(project "PS-PrechargeBoard"
-				(path "/74d17fe6-68d4-4bd7-954a-e2bbb58b1f1e/88068a34-f22d-4106-a80b-45e353d7d848"
-					(reference "TP19")
+				(path "/74d17fe6-68d4-4bd7-954a-e2bbb58b1f1e/c6e51092-efec-40a8-afae-63cae62691f2/d0a2e77c-6f3b-4bbc-a3d8-ef9f85477fa8"
+					(reference "TP13")
 					(unit 1)
 				)
@@
 		(in_pos_files yes)
 		(dnp no)
-		(property "Reference" "TP18"
+		(property "Reference" "TP12"
 			(at 229.87 136.3979 0)
 			(hide yes)
@@
 		(instances
 			(project "PS-PrechargeBoard"
-				(path "/74d17fe6-68d4-4bd7-954a-e2bbb58b1f1e/88068a34-f22d-4106-a80b-45e353d7d848"
-					(reference "TP18")
+				(path "/74d17fe6-68d4-4bd7-954a-e2bbb58b1f1e/c6e51092-efec-40a8-afae-63cae62691f2/d0a2e77c-6f3b-4bbc-a3d8-ef9f85477fa8"
+					(reference "TP12")
 					(unit 1)
 				)
@@
 		(dnp yes)
 		(fields_autoplaced yes)
-		(property "Reference" "U4"
+		(property "Reference" "U3"
 			(at 129.54 71.12 0)
 			(show_name no)
@@
 		(instances
 			(project "PS-PrechargeBoard"
-				(path "/74d17fe6-68d4-4bd7-954a-e2bbb58b1f1e/88068a34-f22d-4106-a80b-45e353d7d848"
-					(reference "U4")
+				(path "/74d17fe6-68d4-4bd7-954a-e2bbb58b1f1e/c6e51092-efec-40a8-afae-63cae62691f2/d0a2e77c-6f3b-4bbc-a3d8-ef9f85477fa8"
+					(reference "U3")
 					(unit 1)
 				)
@@
 		(in_pos_files yes)
 		(dnp no)
-		(property "Reference" "TP20"
+		(property "Reference" "TP14"
 			(at 242.57 136.3979 0)
 			(hide yes)
@@
 		(instances
 			(project "PS-PrechargeBoard"
-				(path "/74d17fe6-68d4-4bd7-954a-e2bbb58b1f1e/88068a34-f22d-4106-a80b-45e353d7d848"
-					(reference "TP20")
+				(path "/74d17fe6-68d4-4bd7-954a-e2bbb58b1f1e/c6e51092-efec-40a8-afae-63cae62691f2/d0a2e77c-6f3b-4bbc-a3d8-ef9f85477fa8"
+					(reference "TP14")
 					(unit 1)
 				)
@@
 		(dnp no)
 		(fields_autoplaced yes)
-		(property "Reference" "#FLG08"
+		(property "Reference" "#FLG04"
 			(at 179.07 84.455 0)
 			(hide yes)
@@
 		(instances
 			(project "PS-PrechargeBoard"
-				(path "/74d17fe6-68d4-4bd7-954a-e2bbb58b1f1e/88068a34-f22d-4106-a80b-45e353d7d848"
-					(reference "#FLG08")
+				(path "/74d17fe6-68d4-4bd7-954a-e2bbb58b1f1e/c6e51092-efec-40a8-afae-63cae62691f2/d0a2e77c-6f3b-4bbc-a3d8-ef9f85477fa8"
+					(reference "#FLG04")
 					(unit 1)
 				)
@@
 		(dnp no)
 		(fields_autoplaced yes)
-		(property "Reference" "#FLG05"
+		(property "Reference" "#FLG01"
 			(at 88.9 79.375 0)
 			(hide yes)
@@
 		(instances
 			(project "PS-PrechargeBoard"
-				(path "/74d17fe6-68d4-4bd7-954a-e2bbb58b1f1e/88068a34-f22d-4106-a80b-45e353d7d848"
-					(reference "#FLG05")
+				(path "/74d17fe6-68d4-4bd7-954a-e2bbb58b1f1e/c6e51092-efec-40a8-afae-63cae62691f2/d0a2e77c-6f3b-4bbc-a3d8-ef9f85477fa8"
+					(reference "#FLG01")
 					(unit 1)
 				)
@@
 		(in_pos_files yes)
 		(dnp no)
-		(property "Reference" "C25"
+		(property "Reference" "C21"
 			(at 164.084 93.98 0)
 			(show_name no)
@@
 		(instances
 			(project "PS-PrechargeBoard"
-				(path "/74d17fe6-68d4-4bd7-954a-e2bbb58b1f1e/88068a34-f22d-4106-a80b-45e353d7d848"
-					(reference "C25")
+				(path "/74d17fe6-68d4-4bd7-954a-e2bbb58b1f1e/c6e51092-efec-40a8-afae-63cae62691f2/d0a2e77c-6f3b-4bbc-a3d8-ef9f85477fa8"
+					(reference "C21")
 					(unit 1)
 				)
@@
 		(in_pos_files yes)
 		(dnp no)
-		(property "Reference" "C27"
+		(property "Reference" "C23"
 			(at 189.992 93.98 0)
 			(show_name no)
@@
 		(instances
 			(project "PS-PrechargeBoard"
-				(path "/74d17fe6-68d4-4bd7-954a-e2bbb58b1f1e/88068a34-f22d-4106-a80b-45e353d7d848"
-					(reference "C27")
+				(path "/74d17fe6-68d4-4bd7-954a-e2bbb58b1f1e/c6e51092-efec-40a8-afae-63cae62691f2/d0a2e77c-6f3b-4bbc-a3d8-ef9f85477fa8"
+					(reference "C23")
 					(unit 1)
 				)
@@
 		(in_pos_files yes)
 		(dnp no)
-		(property "Reference" "C24"
+		(property "Reference" "C20"
 			(at 156.718 80.01 0)
 			(show_name no)
@@
 		(instances
 			(project "PS-PrechargeBoard"
-				(path "/74d17fe6-68d4-4bd7-954a-e2bbb58b1f1e/88068a34-f22d-4106-a80b-45e353d7d848"
-					(reference "C24")
+				(path "/74d17fe6-68d4-4bd7-954a-e2bbb58b1f1e/c6e51092-efec-40a8-afae-63cae62691f2/d0a2e77c-6f3b-4bbc-a3d8-ef9f85477fa8"
+					(reference "C20")
 					(unit 1)
 				)
@@
 		(in_pos_files yes)
 		(dnp no)
-		(property "Reference" "#FLG07"
+		(property "Reference" "#FLG03"
 			(at 149.86 84.455 0)
 			(hide yes)
@@
 		(instances
 			(project "PS-PrechargeBoard"
-				(path "/74d17fe6-68d4-4bd7-954a-e2bbb58b1f1e/88068a34-f22d-4106-a80b-45e353d7d848"
-					(reference "#FLG07")
+				(path "/74d17fe6-68d4-4bd7-954a-e2bbb58b1f1e/c6e51092-efec-40a8-afae-63cae62691f2/d0a2e77c-6f3b-4bbc-a3d8-ef9f85477fa8"
+					(reference "#FLG03")
 					(unit 1)
 				)
@@
 		(dnp no)
 		(fields_autoplaced yes)
-		(property "Reference" "R29"
+		(property "Reference" "R24"
 			(at 227.33 85.0899 0)
 			(show_name no)
@@
 		(instances
 			(project "PS-PrechargeBoard"
-				(path "/74d17fe6-68d4-4bd7-954a-e2bbb58b1f1e/88068a34-f22d-4106-a80b-45e353d7d848"
-					(reference "R29")
+				(path "/74d17fe6-68d4-4bd7-954a-e2bbb58b1f1e/c6e51092-efec-40a8-afae-63cae62691f2/d0a2e77c-6f3b-4bbc-a3d8-ef9f85477fa8"
+					(reference "R24")
 					(unit 1)
 				)
@@
 		(dnp no)
 		(fields_autoplaced yes)
-		(property "Reference" "C23"
+		(property "Reference" "C19"
 			(at 105.41 87.6362 0)
 			(show_name no)
@@
 		(instances
 			(project "PS-PrechargeBoard"
-				(path "/74d17fe6-68d4-4bd7-954a-e2bbb58b1f1e/88068a34-f22d-4106-a80b-45e353d7d848"
-					(reference "C23")
+				(path "/74d17fe6-68d4-4bd7-954a-e2bbb58b1f1e/c6e51092-efec-40a8-afae-63cae62691f2/d0a2e77c-6f3b-4bbc-a3d8-ef9f85477fa8"
+					(reference "C19")
 					(unit 1)
 				)
@@
 		(dnp no)
 		(fields_autoplaced yes)
-		(property "Reference" "R30"
+		(property "Reference" "R25"
 			(at 227.33 92.7099 0)
 			(show_name no)
@@
 		(instances
 			(project "PS-PrechargeBoard"
-				(path "/74d17fe6-68d4-4bd7-954a-e2bbb58b1f1e/88068a34-f22d-4106-a80b-45e353d7d848"
-					(reference "R30")
+				(path "/74d17fe6-68d4-4bd7-954a-e2bbb58b1f1e/c6e51092-efec-40a8-afae-63cae62691f2/d0a2e77c-6f3b-4bbc-a3d8-ef9f85477fa8"
+					(reference "R25")
 					(unit 1)
 				)
@@
 		(in_pos_files yes)
 		(dnp no)
-		(property "Reference" "C26"
+		(property "Reference" "C22"
 			(at 173.482 94.234 0)
 			(show_name no)
@@
 		(instances
 			(project "PS-PrechargeBoard"
-				(path "/74d17fe6-68d4-4bd7-954a-e2bbb58b1f1e/88068a34-f22d-4106-a80b-45e353d7d848"
-					(reference "C26")
-					(unit 1)
-				)
+				(path "/74d17fe6-68d4-4bd7-954a-e2bbb58b1f1e/c6e51092-efec-40a8-afae-63cae62691f2/d0a2e77c-6f3b-4bbc-a3d8-ef9f85477fa8"
+					(reference "C22")
+					(unit 1)
+				)
