File: CAN_Transceiver.kicad_sch (KiCad schematic)
At the start: 9 parts, among them IC1 TCAN3413DR

Commit message: lv 1.2
Parts:
- renumbered C5 to C36, C6 to C37, C7 to C38, C8 to C39, D8 to D9, IC1 to IC2, JP2 to JP1
Changed lines of the file:
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@@
-	(hierarchical_label "CAN_L"
-		(shape bidirectional)
-		(at 7.2217 0.8096 180)
-		(effects
-			(font
-				(size 1.27 1.27)
-			)
-			(justify right)
-		)
-	)
 	(hierarchical_label "CAN_L"
 		(shape bidirectional)
@@
 		(in_pos_files yes)
 		(dnp no)
-		(property "Reference" "C6"
+		(property "Reference" "C37"
 			(at 76.2 73.66 0)
 			(show_name no)
@@
 			(project "PS-PrechargeBoard"
 				(path "/74d17fe6-68d4-4bd7-954a-e2bbb58b1f1e/47eb15e8-7080-422c-b470-d12560c6f586"
-					(reference "C6")
+					(reference "C37")
 					(unit 1)
 				)
@@
 		(in_pos_files yes)
 		(dnp no)
-		(property "Reference" "C8"
+		(property "Reference" "C39"
 			(at 194.564 88.646 0)
 			(show_name no)
@@
 			(project "PS-PrechargeBoard"
 				(path "/74d17fe6-68d4-4bd7-954a-e2bbb58b1f1e/47eb15e8-7080-422c-b470-d12560c6f586"
-					(reference "C8")
+					(reference "C39")
 					(unit 1)
 				)
@@
 		(dnp no)
 		(fields_autoplaced yes)
-		(property "Reference" "JP2"
+		(property "Reference" "JP1"
 			(at 215.9 78.74 0)
 			(show_name no)
@@
 			(project "PS-PrechargeBoard"
 				(path "/74d17fe6-68d4-4bd7-954a-e2bbb58b1f1e/47eb15e8-7080-422c-b470-d12560c6f586"
-					(reference "JP2")
+					(reference "JP1")
 					(unit 1)
 				)
@@
 		(in_pos_files yes)
 		(dnp no)
-		(property "Reference" "C7"
+		(property "Reference" "C38"
 			(at 88.138 73.66 0)
 			(show_name no)
@@
 			(project "PS-PrechargeBoard"
 				(path "/74d17fe6-68d4-4bd7-954a-e2bbb58b1f1e/47eb15e8-7080-422c-b470-d12560c6f586"
-					(reference "C7")
+					(reference "C38")
 					(unit 1)
 				)
@@
 		(in_pos_files yes)
 		(dnp no)
-		(property "Reference" "C5"
+		(property "Reference" "C36"
 			(at 65.278 73.66 0)
 			(show_name no)
@@
 			(project "PS-PrechargeBoard"
 				(path "/74d17fe6-68d4-4bd7-954a-e2bbb58b1f1e/47eb15e8-7080-422c-b470-d12560c6f586"
-					(reference "C5")
+					(reference "C36")
 					(unit 1)
 				)
@@
 		(dnp no)
 		(fields_autoplaced yes)
-		(property "Reference" "D8"
+		(property "Reference" "D9"
 			(at 196.85 46.99 0)
 			(show_name no)
@@
 			(project "PS-PrechargeBoard"
 				(path "/74d17fe6-68d4-4bd7-954a-e2bbb58b1f1e/47eb15e8-7080-422c-b470-d12560c6f586"
-					(reference "D8")
+					(reference "D9")
 					(unit 1)
 				)
@@
 		(dnp no)
 		(fields_autoplaced yes)
-		(property "Reference" "IC1"
+		(property "Reference" "IC2"
 			(at 128.27 63.5 0)
 			(show_name no)
@@
 			(project "PS-PrechargeBoard"
 				(path "/74d17fe6-68d4-4bd7-954a-e2bbb58b1f1e/47eb15e8-7080-422c-b470-d12560c6f586"
-					(reference "IC1")
-					(unit 1)
-				)
+					(reference "IC2")
+					(unit 1)
+				)

Commit message: hv 1.0
Parts:
- renumbered R22 to R26, R23 to R27
Changed lines of the file:
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@@
 		(in_pos_files yes)
 		(dnp no)
-		(property "Reference" "R23"
+		(property "Reference" "R27"
 			(at 201.93 80.01 90)
 			(show_name no)
@@
 			(project "PS-PrechargeBoard"
 				(path "/74d17fe6-68d4-4bd7-954a-e2bbb58b1f1e/47eb15e8-7080-422c-b470-d12560c6f586"
-					(reference "R23")
+					(reference "R27")
 					(unit 1)
 				)
@@
 		(in_pos_files yes)
 		(dnp no)
-		(property "Reference" "R22"
+		(property "Reference" "R26"
 			(at 176.53 80.01 90)
 			(show_name no)
@@
 			(project "PS-PrechargeBoard"
 				(path "/74d17fe6-68d4-4bd7-954a-e2bbb58b1f1e/47eb15e8-7080-422c-b470-d12560c6f586"
-					(reference "R22")
-					(unit 1)
-				)
+					(reference "R26")
+					(unit 1)
+				)

Commit message: hv 1.1
Parts:
- renumbered R26 to R25, R27 to R26
Changed lines of the file:
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@@
 		(in_pos_files yes)
 		(dnp no)
-		(property "Reference" "R27"
+		(property "Reference" "R26"
 			(at 201.93 80.01 90)
 			(show_name no)
@@
 			(project "PS-PrechargeBoard"
 				(path "/74d17fe6-68d4-4bd7-954a-e2bbb58b1f1e/47eb15e8-7080-422c-b470-d12560c6f586"
-					(reference "R27")
+					(reference "R26")
 					(unit 1)
 				)
@@
 		(in_pos_files yes)
 		(dnp no)
-		(property "Reference" "R26"
+		(property "Reference" "R25"
 			(at 176.53 80.01 90)
 			(show_name no)
@@
 			(project "PS-PrechargeBoard"
 				(path "/74d17fe6-68d4-4bd7-954a-e2bbb58b1f1e/47eb15e8-7080-422c-b470-d12560c6f586"
-					(reference "R26")
-					(unit 1)
-				)
+					(reference "R25")
+					(unit 1)
+				)

Commit message: hv 1.3
Parts:
- renumbered C37 to C?, C39 to C?, C38 to C?, C36 to C?, D9 to D?, IC2 to IC?, JP1 to JP?, R26 to R?, R25 to R?
Changed lines of the file:
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@@
 		(in_pos_files yes)
 		(dnp no)
-		(property "Reference" "C37"
+		(property "Reference" "C?"
 			(at 76.2 73.66 0)
 			(show_name no)
@@
 		)
 		(instances
-			(project ""
-				(path "/69b823fd-c065-40ff-9bb9-c5835555f3eb/9d9eae1e-c713-4323-9845-a569cff8d5d3"
-					(reference "C6")
-					(unit 1)
-				)
-			)
 			(project "PS-PrechargeBoard"
-				(path "/74d17fe6-68d4-4bd7-954a-e2bbb58b1f1e/47eb15e8-7080-422c-b470-d12560c6f586"
-					(reference "C37")
-					(unit 1)
-				)
-			)
-			(project "CAN_Transceiver"
-				(path "/a09f9696-80ee-4697-8aaa-225f287b667b"
-					(reference "C2")
+				(path "/11743897-1544-4e3c-979c-dcc54ac7093b/b1f43d5a-c322-4586-a0be-8c986728595c"
+					(reference "C?")
 					(unit 1)
 				)
@@
 		(in_pos_files yes)
 		(dnp no)
-		(property "Reference" "C39"
+		(property "Reference" "C?"
 			(at 194.564 88.646 0)
 			(show_name no)
@@
 		)
 		(instances
-			(project ""
-				(path "/69b823fd-c065-40ff-9bb9-c5835555f3eb/9d9eae1e-c713-4323-9845-a569cff8d5d3"
-					(reference "C8")
-					(unit 1)
-				)
-			)
 			(project "PS-PrechargeBoard"
-				(path "/74d17fe6-68d4-4bd7-954a-e2bbb58b1f1e/47eb15e8-7080-422c-b470-d12560c6f586"
-					(reference "C39")
-					(unit 1)
-				)
-			)
-			(project "CAN_Transceiver"
-				(path "/a09f9696-80ee-4697-8aaa-225f287b667b"
-					(reference "C4")
+				(path "/11743897-1544-4e3c-979c-dcc54ac7093b/b1f43d5a-c322-4586-a0be-8c986728595c"
+					(reference "C?")
 					(unit 1)
 				)
@@
 		(dnp no)
 		(fields_autoplaced yes)
-		(property "Reference" "JP1"
+		(property "Reference" "JP?"
 			(at 215.9 78.74 0)
 			(show_name no)
@@
 		)
 		(instances
-			(project ""
-				(path "/69b823fd-c065-40ff-9bb9-c5835555f3eb/9d9eae1e-c713-4323-9845-a569cff8d5d3"
-					(reference "JP2")
-					(unit 1)
-				)
-			)
 			(project "PS-PrechargeBoard"
-				(path "/74d17fe6-68d4-4bd7-954a-e2bbb58b1f1e/47eb15e8-7080-422c-b470-d12560c6f586"
-					(reference "JP1")
-					(unit 1)
-				)
-			)
-			(project ""
-				(path "/81d906df-a099-480a-8398-28a8e913d125"
-					(reference "JP1")
-					(unit 1)
-				)
-			)
-			(project "CAN_Transceiver"
-				(path "/a09f9696-80ee-4697-8aaa-225f287b667b"
-					(reference "JP1")
+				(path "/11743897-1544-4e3c-979c-dcc54ac7093b/b1f43d5a-c322-4586-a0be-8c986728595c"
+					(reference "JP?")
 					(unit 1)
 				)
@@
 		(in_pos_files yes)
 		(dnp no)
-		(property "Reference" "C38"
+		(property "Reference" "C?"
 			(at 88.138 73.66 0)
 			(show_name no)
@@
 		)
 		(instances
-			(project ""
-				(path "/69b823fd-c065-40ff-9bb9-c5835555f3eb/9d9eae1e-c713-4323-9845-a569cff8d5d3"
-					(reference "C7")
-					(unit 1)
-				)
-			)
 			(project "PS-PrechargeBoard"
-				(path "/74d17fe6-68d4-4bd7-954a-e2bbb58b1f1e/47eb15e8-7080-422c-b470-d12560c6f586"
-					(reference "C38")
-					(unit 1)
-				)
-			)
-			(project "CAN_Transceiver"
-				(path "/a09f9696-80ee-4697-8aaa-225f287b667b"
-					(reference "C3")
+				(path "/11743897-1544-4e3c-979c-dcc54ac7093b/b1f43d5a-c322-4586-a0be-8c986728595c"
+					(reference "C?")
 					(unit 1)
 				)
@@
 		(in_pos_files yes)
 		(dnp no)
-		(property "Reference" "C36"
+		(property "Reference" "C?"
 			(at 65.278 73.66 0)
 			(show_name no)
@@
 		)
 		(instances
-			(project ""
-				(path "/69b823fd-c065-40ff-9bb9-c5835555f3eb/9d9eae1e-c713-4323-9845-a569cff8d5d3"
-					(reference "C5")
-					(unit 1)
-				)
-			)
 			(project "PS-PrechargeBoard"
-				(path "/74d17fe6-68d4-4bd7-954a-e2bbb58b1f1e/47eb15e8-7080-422c-b470-d12560c6f586"
-					(reference "C36")
-					(unit 1)
-				)
-			)
-			(project ""
-				(path "/81d906df-a099-480a-8398-28a8e913d125"
-					(reference "C1")
-					(unit 1)
-				)
-			)
-			(project "CAN_Transceiver"
-				(path "/a09f9696-80ee-4697-8aaa-225f287b667b"
-					(reference "C1")
+				(path "/11743897-1544-4e3c-979c-dcc54ac7093b/b1f43d5a-c322-4586-a0be-8c986728595c"
+					(reference "C?")
 					(unit 1)
 				)
@@
 		(in_pos_files yes)
 		(dnp no)
-		(property "Reference" "R26"
+		(property "Reference" "R?"
 			(at 201.93 80.01 90)
 			(show_name no)
@@
 		)
 		(instances
-			(project "kk36984"
-				(path "/69b823fd-c065-40ff-9bb9-c5835555f3eb/9d9eae1e-c713-4323-9845-a569cff8d5d3"
-					(reference "R23")
-					(unit 1)
-				)
-			)
 			(project "PS-PrechargeBoard"
-				(path "/74d17fe6-68d4-4bd7-954a-e2bbb58b1f1e/47eb15e8-7080-422c-b470-d12560c6f586"
-					(reference "R26")
-					(unit 1)
-				)
-			)
-			(project "CAN_Transceiver"
-				(path "/a09f9696-80ee-4697-8aaa-225f287b667b"
-					(reference "R2")
+				(path "/11743897-1544-4e3c-979c-dcc54ac7093b/b1f43d5a-c322-4586-a0be-8c986728595c"
+					(reference "R?")
 					(unit 1)
 				)
@@
 		(dnp no)
 		(fields_autoplaced yes)
-		(property "Reference" "D9"
+		(property "Reference" "D?"
 			(at 196.85 46.99 0)
 			(show_name no)
@@
 		)
 		(instances
-			(project ""
-				(path "/69b823fd-c065-40ff-9bb9-c5835555f3eb/9d9eae1e-c713-4323-9845-a569cff8d5d3"
-					(reference "D8")
-					(unit 1)
-				)
-			)
 			(project "PS-PrechargeBoard"
-				(path "/74d17fe6-68d4-4bd7-954a-e2bbb58b1f1e/47eb15e8-7080-422c-b470-d12560c6f586"
-					(reference "D9")
-					(unit 1)
-				)
-			)
-			(project "CAN_Transceiver"
-				(path "/a09f9696-80ee-4697-8aaa-225f287b667b"
-					(reference "D1")
+				(path "/11743897-1544-4e3c-979c-dcc54ac7093b/b1f43d5a-c322-4586-a0be-8c986728595c"
+					(reference "D?")
 					(unit 1)
 				)
@@
 		(dnp no)
 		(fields_autoplaced yes)
-		(property "Reference" "IC2"
+		(property "Reference" "IC?"
 			(at 128.27 63.5 0)
 			(show_name no)
@@
 		)
 		(instances
-			(project ""
-				(path "/69b823fd-c065-40ff-9bb9-c5835555f3eb/9d9eae1e-c713-4323-9845-a569cff8d5d3"
-					(reference "IC1")
-					(unit 1)
-				)
-			)
 			(project "PS-PrechargeBoard"
-				(path "/74d17fe6-68d4-4bd7-954a-e2bbb58b1f1e/47eb15e8-7080-422c-b470-d12560c6f586"
-					(reference "IC2")
-					(unit 1)
-				)
-			)
-			(project "CAN_Transceiver"
-				(path "/a09f9696-80ee-4697-8aaa-225f287b667b"
-					(reference "IC1")
+				(path "/11743897-1544-4e3c-979c-dcc54ac7093b/b1f43d5a-c322-4586-a0be-8c986728595c"
+					(reference "IC?")
 					(unit 1)
 				)
@@
 		(in_pos_files yes)
 		(dnp no)
-		(property "Reference" "R25"
+		(property "Reference" "R?"
 			(at 176.53 80.01 90)
 			(show_name no)
@@
 		)
 		(instances
-			(project ""
-				(path "/69b823fd-c065-40ff-9bb9-c5835555f3eb/9d9eae1e-c713-4323-9845-a569cff8d5d3"
-					(reference "R22")
+			(project "PS-PrechargeBoard"
+				(path "/11743897-1544-4e3c-979c-dcc54ac7093b/b1f43d5a-c322-4586-a0be-8c986728595c"
+					(reference "R?")
 					(unit 1)
 				)
-			)
-			(project "PS-PrechargeBoard"
-				(path "/74d17fe6-68d4-4bd7-954a-e2bbb58b1f1e/47eb15e8-7080-422c-b470-d12560c6f586"
-					(reference "R25")
-					(unit 1)
-				)
-			)
-			(project ""
-				(path "/81d906df-a099-480a-8398-28a8e913d125"
-					(reference "R1")
-					(unit 1)
-				)
-			)
-			(project "CAN_Transceiver"
-				(path "/a09f9696-80ee-4697-8aaa-225f287b667b"
-					(reference "R1")
-					(unit 1)
-				)
