File: CAN_Transceiver.kicad_sch (KiCad schematic)
At the start: 9 parts

Commit message: CAN nano & CAN debug nano
Parts:
- gave numbers to parts that had none: 9
Changed lines of the file:
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@@
 		(in_pos_files yes)
 		(dnp no)
-		(property "Reference" "C?"
+		(property "Reference" "C17"
 			(at 76.2 73.66 0)
 			(show_name no)
@@
 			(project "PS-PrechargeBoard"
 				(path "/74d17fe6-68d4-4bd7-954a-e2bbb58b1f1e/0def18ef-81e8-47ac-b719-2d9f8237a855/b1f43d5a-c322-4586-a0be-8c986728595c"
-					(reference "C?")
+					(reference "C17")
 					(unit 1)
 				)
@@
 			(project "lv"
 				(path "/88356d12-c87f-4bdd-bbd8-756414c90a6d/b1f43d5a-c322-4586-a0be-8c986728595c"
-					(reference "C?")
-					(unit 1)
-				)
-			)
-			(project "PS-PrechargeBoard"
-				(path "/9641192f-df6c-4894-9070-848e3256daf8/b1f43d5a-c322-4586-a0be-8c986728595c"
 					(reference "C?")
 					(unit 1)
@@
 		(in_pos_files yes)
 		(dnp no)
-		(property "Reference" "C?"
+		(property "Reference" "C19"
 			(at 194.564 88.646 0)
 			(show_name no)
@@
 			(project "PS-PrechargeBoard"
 				(path "/74d17fe6-68d4-4bd7-954a-e2bbb58b1f1e/0def18ef-81e8-47ac-b719-2d9f8237a855/b1f43d5a-c322-4586-a0be-8c986728595c"
-					(reference "C?")
+					(reference "C19")
 					(unit 1)
 				)
@@
 			(project "lv"
 				(path "/88356d12-c87f-4bdd-bbd8-756414c90a6d/b1f43d5a-c322-4586-a0be-8c986728595c"
-					(reference "C?")
-					(unit 1)
-				)
-			)
-			(project "PS-PrechargeBoard"
-				(path "/9641192f-df6c-4894-9070-848e3256daf8/b1f43d5a-c322-4586-a0be-8c986728595c"
 					(reference "C?")
 					(unit 1)
@@
 		(dnp no)
 		(fields_autoplaced yes)
-		(property "Reference" "JP?"
+		(property "Reference" "JP1"
 			(at 215.9 78.74 0)
 			(show_name no)
@@
 			(project "PS-PrechargeBoard"
 				(path "/74d17fe6-68d4-4bd7-954a-e2bbb58b1f1e/0def18ef-81e8-47ac-b719-2d9f8237a855/b1f43d5a-c322-4586-a0be-8c986728595c"
-					(reference "JP?")
+					(reference "JP1")
 					(unit 1)
 				)
@@
 			(project "lv"
 				(path "/88356d12-c87f-4bdd-bbd8-756414c90a6d/b1f43d5a-c322-4586-a0be-8c986728595c"
-					(reference "JP?")
-					(unit 1)
-				)
-			)
-			(project "PS-PrechargeBoard"
-				(path "/9641192f-df6c-4894-9070-848e3256daf8/b1f43d5a-c322-4586-a0be-8c986728595c"
 					(reference "JP?")
 					(unit 1)
@@
 		(in_pos_files yes)
 		(dnp no)
-		(property "Reference" "C?"
+		(property "Reference" "C18"
 			(at 88.138 73.66 0)
 			(show_name no)
@@
 			(project "PS-PrechargeBoard"
 				(path "/74d17fe6-68d4-4bd7-954a-e2bbb58b1f1e/0def18ef-81e8-47ac-b719-2d9f8237a855/b1f43d5a-c322-4586-a0be-8c986728595c"
-					(reference "C?")
+					(reference "C18")
 					(unit 1)
 				)
@@
 			(project "lv"
 				(path "/88356d12-c87f-4bdd-bbd8-756414c90a6d/b1f43d5a-c322-4586-a0be-8c986728595c"
-					(reference "C?")
-					(unit 1)
-				)
-			)
-			(project "PS-PrechargeBoard"
-				(path "/9641192f-df6c-4894-9070-848e3256daf8/b1f43d5a-c322-4586-a0be-8c986728595c"
 					(reference "C?")
 					(unit 1)
@@
 		(in_pos_files yes)
 		(dnp no)
-		(property "Reference" "C?"
+		(property "Reference" "C16"
 			(at 65.278 73.66 0)
 			(show_name no)
@@
 			(project "PS-PrechargeBoard"
 				(path "/74d17fe6-68d4-4bd7-954a-e2bbb58b1f1e/0def18ef-81e8-47ac-b719-2d9f8237a855/b1f43d5a-c322-4586-a0be-8c986728595c"
-					(reference "C?")
+					(reference "C16")
 					(unit 1)
 				)
@@
 			(project "lv"
 				(path "/88356d12-c87f-4bdd-bbd8-756414c90a6d/b1f43d5a-c322-4586-a0be-8c986728595c"
-					(reference "C?")
-					(unit 1)
-				)
-			)
-			(project "PS-PrechargeBoard"
-				(path "/9641192f-df6c-4894-9070-848e3256daf8/b1f43d5a-c322-4586-a0be-8c986728595c"
 					(reference "C?")
 					(unit 1)
@@
 		(in_pos_files yes)
 		(dnp no)
-		(property "Reference" "R?"
+		(property "Reference" "R10"
 			(at 201.93 80.01 90)
 			(show_name no)
@@
 			(project "PS-PrechargeBoard"
 				(path "/74d17fe6-68d4-4bd7-954a-e2bbb58b1f1e/0def18ef-81e8-47ac-b719-2d9f8237a855/b1f43d5a-c322-4586-a0be-8c986728595c"
-					(reference "R?")
+					(reference "R10")
 					(unit 1)
 				)
@@
 			(project "lv"
 				(path "/88356d12-c87f-4bdd-bbd8-756414c90a6d/b1f43d5a-c322-4586-a0be-8c986728595c"
-					(reference "R?")
-					(unit 1)
-				)
-			)
-			(project "PS-PrechargeBoard"
-				(path "/9641192f-df6c-4894-9070-848e3256daf8/b1f43d5a-c322-4586-a0be-8c986728595c"
 					(reference "R?")
 					(unit 1)
@@
 		(dnp no)
 		(fields_autoplaced yes)
-		(property "Reference" "D?"
+		(property "Reference" "D4"
 			(at 196.85 46.99 0)
 			(show_name no)
@@
 			(project "PS-PrechargeBoard"
 				(path "/74d17fe6-68d4-4bd7-954a-e2bbb58b1f1e/0def18ef-81e8-47ac-b719-2d9f8237a855/b1f43d5a-c322-4586-a0be-8c986728595c"
-					(reference "D?")
+					(reference "D4")
 					(unit 1)
 				)
@@
 			(project "lv"
 				(path "/88356d12-c87f-4bdd-bbd8-756414c90a6d/b1f43d5a-c322-4586-a0be-8c986728595c"
-					(reference "D?")
-					(unit 1)
-				)
-			)
-			(project "PS-PrechargeBoard"
-				(path "/9641192f-df6c-4894-9070-848e3256daf8/b1f43d5a-c322-4586-a0be-8c986728595c"
 					(reference "D?")
 					(unit 1)
@@
 		(dnp no)
 		(fields_autoplaced yes)
-		(property "Reference" "IC?"
+		(property "Reference" "IC1"
 			(at 128.27 63.5 0)
 			(show_name no)
@@
 			(project "PS-PrechargeBoard"
 				(path "/74d17fe6-68d4-4bd7-954a-e2bbb58b1f1e/0def18ef-81e8-47ac-b719-2d9f8237a855/b1f43d5a-c322-4586-a0be-8c986728595c"
-					(reference "IC?")
+					(reference "IC1")
 					(unit 1)
 				)
@@
 			(project "lv"
 				(path "/88356d12-c87f-4bdd-bbd8-756414c90a6d/b1f43d5a-c322-4586-a0be-8c986728595c"
-					(reference "IC?")
-					(unit 1)
-				)
-			)
-			(project "PS-PrechargeBoard"
-				(path "/9641192f-df6c-4894-9070-848e3256daf8/b1f43d5a-c322-4586-a0be-8c986728595c"
 					(reference "IC?")
 					(unit 1)
@@
 		(in_pos_files yes)
 		(dnp no)
-		(property "Reference" "R?"
+		(property "Reference" "R9"
 			(at 176.53 80.01 90)
 			(show_name no)
@@
 			(project "PS-PrechargeBoard"
 				(path "/74d17fe6-68d4-4bd7-954a-e2bbb58b1f1e/0def18ef-81e8-47ac-b719-2d9f8237a855/b1f43d5a-c322-4586-a0be-8c986728595c"
-					(reference "R?")
+					(reference "R9")
 					(unit 1)
 				)
@@
 					(reference "R?")
 					(unit 1)
-				)
-			)
-			(project "PS-PrechargeBoard"
-				(path "/9641192f-df6c-4894-9070-848e3256daf8/b1f43d5a-c322-4586-a0be-8c986728595c"
-					(reference "R?")
-					(unit 1)

Commit message: battery voltage & motor voltage
Parts:
- renumbered C16 to C44, C17 to C45, C18 to C46, C19 to C47, D4 to D12, IC1 to IC2, R9 to R36, R10 to R37
Changed lines of the file:
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@@
 		(in_pos_files yes)
 		(dnp no)
-		(property "Reference" "C17"
+		(property "Reference" "C45"
 			(at 76.2 73.66 0)
 			(show_name no)
@@
 			(project "PS-PrechargeBoard"
 				(path "/74d17fe6-68d4-4bd7-954a-e2bbb58b1f1e/0def18ef-81e8-47ac-b719-2d9f8237a855/b1f43d5a-c322-4586-a0be-8c986728595c"
-					(reference "C17")
+					(reference "C45")
 					(unit 1)
 				)
@@
 		(in_pos_files yes)
 		(dnp no)
-		(property "Reference" "C19"
+		(property "Reference" "C47"
 			(at 194.564 88.646 0)
 			(show_name no)
@@
 			(project "PS-PrechargeBoard"
 				(path "/74d17fe6-68d4-4bd7-954a-e2bbb58b1f1e/0def18ef-81e8-47ac-b719-2d9f8237a855/b1f43d5a-c322-4586-a0be-8c986728595c"
-					(reference "C19")
+					(reference "C47")
 					(unit 1)
 				)
@@
 		(in_pos_files yes)
 		(dnp no)
-		(property "Reference" "C18"
+		(property "Reference" "C46"
 			(at 88.138 73.66 0)
 			(show_name no)
@@
 			(project "PS-PrechargeBoard"
 				(path "/74d17fe6-68d4-4bd7-954a-e2bbb58b1f1e/0def18ef-81e8-47ac-b719-2d9f8237a855/b1f43d5a-c322-4586-a0be-8c986728595c"
-					(reference "C18")
+					(reference "C46")
 					(unit 1)
 				)
@@
 		(in_pos_files yes)
 		(dnp no)
-		(property "Reference" "C16"
+		(property "Reference" "C44"
 			(at 65.278 73.66 0)
 			(show_name no)
@@
 			(project "PS-PrechargeBoard"
 				(path "/74d17fe6-68d4-4bd7-954a-e2bbb58b1f1e/0def18ef-81e8-47ac-b719-2d9f8237a855/b1f43d5a-c322-4586-a0be-8c986728595c"
-					(reference "C16")
+					(reference "C44")
 					(unit 1)
 				)
@@
 		(in_pos_files yes)
 		(dnp no)
-		(property "Reference" "R10"
+		(property "Reference" "R37"
 			(at 201.93 80.01 90)
 			(show_name no)
@@
 			(project "PS-PrechargeBoard"
 				(path "/74d17fe6-68d4-4bd7-954a-e2bbb58b1f1e/0def18ef-81e8-47ac-b719-2d9f8237a855/b1f43d5a-c322-4586-a0be-8c986728595c"
-					(reference "R10")
+					(reference "R37")
 					(unit 1)
 				)
@@
 		(dnp no)
 		(fields_autoplaced yes)
-		(property "Reference" "D4"
+		(property "Reference" "D12"
 			(at 196.85 46.99 0)
 			(show_name no)
@@
 			(project "PS-PrechargeBoard"
 				(path "/74d17fe6-68d4-4bd7-954a-e2bbb58b1f1e/0def18ef-81e8-47ac-b719-2d9f8237a855/b1f43d5a-c322-4586-a0be-8c986728595c"
-					(reference "D4")
+					(reference "D12")
 					(unit 1)
 				)
@@
 		(dnp no)
 		(fields_autoplaced yes)
-		(property "Reference" "IC1"
+		(property "Reference" "IC2"
 			(at 128.27 63.5 0)
 			(show_name no)
@@
 			(project "PS-PrechargeBoard"
 				(path "/74d17fe6-68d4-4bd7-954a-e2bbb58b1f1e/0def18ef-81e8-47ac-b719-2d9f8237a855/b1f43d5a-c322-4586-a0be-8c986728595c"
-					(reference "IC1")
+					(reference "IC2")
 					(unit 1)
 				)
@@
 		(in_pos_files yes)
 		(dnp no)
-		(property "Reference" "R9"
+		(property "Reference" "R36"
 			(at 176.53 80.01 90)
 			(show_name no)
@@
 			(project "PS-PrechargeBoard"
 				(path "/74d17fe6-68d4-4bd7-954a-e2bbb58b1f1e/0def18ef-81e8-47ac-b719-2d9f8237a855/b1f43d5a-c322-4586-a0be-8c986728595c"
-					(reference "R9")
-					(unit 1)
-				)
+					(reference "R36")
+					(unit 1)
+				)

Commit message: mini review notes
Parts:
- renumbered D12 to D14
Changed lines of the file:
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@@
 		(dnp no)
 		(fields_autoplaced yes)
-		(property "Reference" "D12"
+		(property "Reference" "D14"
 			(at 196.85 46.99 0)
 			(show_name no)
@@
 			(project "PS-PrechargeBoard"
 				(path "/74d17fe6-68d4-4bd7-954a-e2bbb58b1f1e/0def18ef-81e8-47ac-b719-2d9f8237a855/b1f43d5a-c322-4586-a0be-8c986728595c"
-					(reference "D12")
+					(reference "D14")
 					(unit 1)
 				)

Commit message: shifted hierarchical sheets
Parts:
- renumbered C45 to C?, C47 to C?, C46 to C?, C44 to C?, D14 to D?, IC2 to IC?, JP1 to JP?, R37 to R?, R36 to R?
Changed lines of the file:
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@@
 		(in_pos_files yes)
 		(dnp no)
-		(property "Reference" "C45"
+		(property "Reference" "C?"
 			(at 76.2 73.66 0)
 			(show_name no)
@@
 		(instances
 			(project "PS-PrechargeBoard"
-				(path "/74d17fe6-68d4-4bd7-954a-e2bbb58b1f1e/0def18ef-81e8-47ac-b719-2d9f8237a855/b1f43d5a-c322-4586-a0be-8c986728595c"
-					(reference "C45")
-					(unit 1)
-				)
-			)
-			(project "lv"
-				(path "/88356d12-c87f-4bdd-bbd8-756414c90a6d/b1f43d5a-c322-4586-a0be-8c986728595c"
+				(path "/74d17fe6-68d4-4bd7-954a-e2bbb58b1f1e/b145027e-119d-4806-b245-f9ce431b31da"
 					(reference "C?")
 					(unit 1)
@@
 		(in_pos_files yes)
 		(dnp no)
-		(property "Reference" "C47"
+		(property "Reference" "C?"
 			(at 194.564 88.646 0)
 			(show_name no)
@@
 		(instances
 			(project "PS-PrechargeBoard"
-				(path "/74d17fe6-68d4-4bd7-954a-e2bbb58b1f1e/0def18ef-81e8-47ac-b719-2d9f8237a855/b1f43d5a-c322-4586-a0be-8c986728595c"
-					(reference "C47")
-					(unit 1)
-				)
-			)
-			(project "lv"
-				(path "/88356d12-c87f-4bdd-bbd8-756414c90a6d/b1f43d5a-c322-4586-a0be-8c986728595c"
+				(path "/74d17fe6-68d4-4bd7-954a-e2bbb58b1f1e/b145027e-119d-4806-b245-f9ce431b31da"
 					(reference "C?")
 					(unit 1)
@@
 		(dnp no)
 		(fields_autoplaced yes)
-		(property "Reference" "JP1"
+		(property "Reference" "JP?"
 			(at 215.9 78.74 0)
 			(show_name no)
@@
 		(instances
 			(project "PS-PrechargeBoard"
-				(path "/74d17fe6-68d4-4bd7-954a-e2bbb58b1f1e/0def18ef-81e8-47ac-b719-2d9f8237a855/b1f43d5a-c322-4586-a0be-8c986728595c"
-					(reference "JP1")
-					(unit 1)
-				)
-			)
-			(project "lv"
-				(path "/88356d12-c87f-4bdd-bbd8-756414c90a6d/b1f43d5a-c322-4586-a0be-8c986728595c"
+				(path "/74d17fe6-68d4-4bd7-954a-e2bbb58b1f1e/b145027e-119d-4806-b245-f9ce431b31da"
 					(reference "JP?")
 					(unit 1)
@@
 		(in_pos_files yes)
 		(dnp no)
-		(property "Reference" "C46"
+		(property "Reference" "C?"
 			(at 88.138 73.66 0)
 			(show_name no)
@@
 		(instances
 			(project "PS-PrechargeBoard"
-				(path "/74d17fe6-68d4-4bd7-954a-e2bbb58b1f1e/0def18ef-81e8-47ac-b719-2d9f8237a855/b1f43d5a-c322-4586-a0be-8c986728595c"
-					(reference "C46")
-					(unit 1)
-				)
-			)
-			(project "lv"
-				(path "/88356d12-c87f-4bdd-bbd8-756414c90a6d/b1f43d5a-c322-4586-a0be-8c986728595c"
+				(path "/74d17fe6-68d4-4bd7-954a-e2bbb58b1f1e/b145027e-119d-4806-b245-f9ce431b31da"
 					(reference "C?")
 					(unit 1)
@@
 		(in_pos_files yes)
 		(dnp no)
-		(property "Reference" "C44"
+		(property "Reference" "C?"
 			(at 65.278 73.66 0)
 			(show_name no)
@@
 		(instances
 			(project "PS-PrechargeBoard"
-				(path "/74d17fe6-68d4-4bd7-954a-e2bbb58b1f1e/0def18ef-81e8-47ac-b719-2d9f8237a855/b1f43d5a-c322-4586-a0be-8c986728595c"
-					(reference "C44")
-					(unit 1)
-				)
-			)
-			(project "lv"
-				(path "/88356d12-c87f-4bdd-bbd8-756414c90a6d/b1f43d5a-c322-4586-a0be-8c986728595c"
+				(path "/74d17fe6-68d4-4bd7-954a-e2bbb58b1f1e/b145027e-119d-4806-b245-f9ce431b31da"
 					(reference "C?")
 					(unit 1)
@@
 		(in_pos_files yes)
 		(dnp no)
-		(property "Reference" "R37"
+		(property "Reference" "R?"
 			(at 201.93 80.01 90)
 			(show_name no)
@@
 		(instances
 			(project "PS-PrechargeBoard"
-				(path "/74d17fe6-68d4-4bd7-954a-e2bbb58b1f1e/0def18ef-81e8-47ac-b719-2d9f8237a855/b1f43d5a-c322-4586-a0be-8c986728595c"
-					(reference "R37")
-					(unit 1)
-				)
-			)
-			(project "lv"
-				(path "/88356d12-c87f-4bdd-bbd8-756414c90a6d/b1f43d5a-c322-4586-a0be-8c986728595c"
+				(path "/74d17fe6-68d4-4bd7-954a-e2bbb58b1f1e/b145027e-119d-4806-b245-f9ce431b31da"
 					(reference "R?")
 					(unit 1)
@@
 		(dnp no)
 		(fields_autoplaced yes)
-		(property "Reference" "D14"
+		(property "Reference" "D?"
 			(at 196.85 46.99 0)
 			(show_name no)
@@
 		(instances
 			(project "PS-PrechargeBoard"
-				(path "/74d17fe6-68d4-4bd7-954a-e2bbb58b1f1e/0def18ef-81e8-47ac-b719-2d9f8237a855/b1f43d5a-c322-4586-a0be-8c986728595c"
-					(reference "D14")
-					(unit 1)
-				)
-			)
-			(project "lv"
-				(path "/88356d12-c87f-4bdd-bbd8-756414c90a6d/b1f43d5a-c322-4586-a0be-8c986728595c"
+				(path "/74d17fe6-68d4-4bd7-954a-e2bbb58b1f1e/b145027e-119d-4806-b245-f9ce431b31da"
 					(reference "D?")
 					(unit 1)
@@
 		(dnp no)
 		(fields_autoplaced yes)
-		(property "Reference" "IC2"
+		(property "Reference" "IC?"
 			(at 128.27 63.5 0)
 			(show_name no)
@@
 		(instances
 			(project "PS-PrechargeBoard"
-				(path "/74d17fe6-68d4-4bd7-954a-e2bbb58b1f1e/0def18ef-81e8-47ac-b719-2d9f8237a855/b1f43d5a-c322-4586-a0be-8c986728595c"
-					(reference "IC2")
-					(unit 1)
-				)
-			)
-			(project "lv"
-				(path "/88356d12-c87f-4bdd-bbd8-756414c90a6d/b1f43d5a-c322-4586-a0be-8c986728595c"
+				(path "/74d17fe6-68d4-4bd7-954a-e2bbb58b1f1e/b145027e-119d-4806-b245-f9ce431b31da"
 					(reference "IC?")
 					(unit 1)
@@
 		(in_pos_files yes)
 		(dnp no)
-		(property "Reference" "R36"
+		(property "Reference" "R?"
 			(at 176.53 80.01 90)
 			(show_name no)
@@
 		(instances
 			(project "PS-PrechargeBoard"
-				(path "/74d17fe6-68d4-4bd7-954a-e2bbb58b1f1e/0def18ef-81e8-47ac-b719-2d9f8237a855/b1f43d5a-c322-4586-a0be-8c986728595c"
-					(reference "R36")
-					(unit 1)
-				)
-			)
-			(project "lv"
-				(path "/88356d12-c87f-4bdd-bbd8-756414c90a6d/b1f43d5a-c322-4586-a0be-8c986728595c"
+				(path "/74d17fe6-68d4-4bd7-954a-e2bbb58b1f1e/b145027e-119d-4806-b245-f9ce431b31da"
 					(reference "R?")
 					(unit 1)

Commit message: V_OUT_BAT & V_OUT_MOT & PRECHARGE_CTRL to MCU
Parts:
- gave numbers to parts that had none: 9
Changed lines of the file:
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@@
 		(in_pos_files yes)
 		(dnp no)
-		(property "Reference" "C?"
+		(property "Reference" "C44"
 			(at 76.2 73.66 0)
 			(show_name no)
@@
 			(project "PS-PrechargeBoard"
 				(path "/74d17fe6-68d4-4bd7-954a-e2bbb58b1f1e/b145027e-119d-4806-b245-f9ce431b31da"
-					(reference "C?")
+					(reference "C44")
 					(unit 1)
 				)
@@
 		(in_pos_files yes)
 		(dnp no)
-		(property "Reference" "C?"
+		(property "Reference" "C46"
 			(at 194.564 88.646 0)
 			(show_name no)
@@
 			(project "PS-PrechargeBoard"
 				(path "/74d17fe6-68d4-4bd7-954a-e2bbb58b1f1e/b145027e-119d-4806-b245-f9ce431b31da"
-					(reference "C?")
+					(reference "C46")
 					(unit 1)
 				)
@@
 		(dnp no)
 		(fields_autoplaced yes)
-		(property "Reference" "JP?"
+		(property "Reference" "JP1"
 			(at 215.9 78.74 0)
 			(show_name no)
@@
 			(project "PS-PrechargeBoard"
 				(path "/74d17fe6-68d4-4bd7-954a-e2bbb58b1f1e/b145027e-119d-4806-b245-f9ce431b31da"
-					(reference "JP?")
+					(reference "JP1")
 					(unit 1)
 				)
@@
 		(in_pos_files yes)
 		(dnp no)
-		(property "Reference" "C?"
+		(property "Reference" "C45"
 			(at 88.138 73.66 0)
 			(show_name no)
@@
 			(project "PS-PrechargeBoard"
 				(path "/74d17fe6-68d4-4bd7-954a-e2bbb58b1f1e/b145027e-119d-4806-b245-f9ce431b31da"
-					(reference "C?")
+					(reference "C45")
 					(unit 1)
 				)
@@
 		(in_pos_files yes)
 		(dnp no)
-		(property "Reference" "C?"
+		(property "Reference" "C43"
 			(at 65.278 73.66 0)
 			(show_name no)
@@
 			(project "PS-PrechargeBoard"
 				(path "/74d17fe6-68d4-4bd7-954a-e2bbb58b1f1e/b145027e-119d-4806-b245-f9ce431b31da"
-					(reference "C?")
+					(reference "C43")
 					(unit 1)
 				)
@@
 		(in_pos_files yes)
 		(dnp no)
-		(property "Reference" "R?"
+		(property "Reference" "R40"
 			(at 201.93 80.01 90)
 			(show_name no)
@@
 			(project "PS-PrechargeBoard"
 				(path "/74d17fe6-68d4-4bd7-954a-e2bbb58b1f1e/b145027e-119d-4806-b245-f9ce431b31da"
-					(reference "R?")
+					(reference "R40")
 					(unit 1)
 				)
@@
 		(dnp no)
 		(fields_autoplaced yes)
-		(property "Reference" "D?"
+		(property "Reference" "D9"
 			(at 196.85 46.99 0)
 			(show_name no)
@@
 			(project "PS-PrechargeBoard"
 				(path "/74d17fe6-68d4-4bd7-954a-e2bbb58b1f1e/b145027e-119d-4806-b245-f9ce431b31da"
-					(reference "D?")
+					(reference "D9")
 					(unit 1)
 				)
@@
 		(dnp no)
 		(fields_autoplaced yes)
-		(property "Reference" "IC?"
+		(property "Reference" "IC3"
 			(at 128.27 63.5 0)
 			(show_name no)
@@
 			(project "PS-PrechargeBoard"
 				(path "/74d17fe6-68d4-4bd7-954a-e2bbb58b1f1e/b145027e-119d-4806-b245-f9ce431b31da"
-					(reference "IC?")
+					(reference "IC3")
 					(unit 1)
 				)
@@
 		(in_pos_files yes)
 		(dnp no)
-		(property "Reference" "R?"
+		(property "Reference" "R39"
 			(at 176.53 80.01 90)
 			(show_name no)
@@
 			(project "PS-PrechargeBoard"
 				(path "/74d17fe6-68d4-4bd7-954a-e2bbb58b1f1e/b145027e-119d-4806-b245-f9ce431b31da"
-					(reference "R?")
+					(reference "R39")
 					(unit 1)
 				)
