File: LDO.kicad_sch (KiCad schematic)
At the start: 5 parts, among them U1 MCP1826S

Commit message: lv 1.2
Parts:
- renumbered C1 to C19, C2 to C20, D1 to D5, U1 to U3
Changed lines of the file:
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@@
-		)
-	)
-	(hierarchical_label "5V"
-		(shape input)
-		(at 3.835 0.8096 180)
-		(effects
-			(font
-				(size 1.27 1.27)
-			)
-			(justify right)
 		)
 	)
@@
 		(shape input)
 		(at 152.4 76.2 270)
-		(effects
-			(font
-				(size 1.27 1.27)
-			)
-			(justify right)
-		)
-	)
-	(hierarchical_label "5V"
-		(shape input)
-		(at 6.375 3.3496 180)
 		(effects
 			(font
@@
 		(dnp no)
 		(fields_autoplaced yes)
-		(property "Reference" "C2"
+		(property "Reference" "C20"
 			(at 168.275 68.5735 0)
 			(show_name no)
@@
 			(project "PS-PrechargeBoard"
 				(path "/74d17fe6-68d4-4bd7-954a-e2bbb58b1f1e/ac0b82bc-5139-4aa7-86f9-8716cbcedbf0"
-					(reference "C2")
+					(reference "C20")
 					(unit 1)
 				)
@@
 		(dnp no)
 		(fields_autoplaced yes)
-		(property "Reference" "U1"
+		(property "Reference" "U3"
 			(at 152.4 56.515 0)
 			(show_name no)
@@
 			(project "PS-PrechargeBoard"
 				(path "/74d17fe6-68d4-4bd7-954a-e2bbb58b1f1e/ac0b82bc-5139-4aa7-86f9-8716cbcedbf0"
-					(reference "U1")
+					(reference "U3")
 					(unit 1)
 				)
@@
 		(dnp no)
 		(fields_autoplaced yes)
-		(property "Reference" "D1"
+		(property "Reference" "D5"
 			(at 133.604 57.15 0)
 			(show_name no)
@@
 			(project "PS-PrechargeBoard"
 				(path "/74d17fe6-68d4-4bd7-954a-e2bbb58b1f1e/ac0b82bc-5139-4aa7-86f9-8716cbcedbf0"
-					(reference "D1")
+					(reference "D5")
 					(unit 1)
 				)
@@
 		(dnp no)
 		(fields_autoplaced yes)
-		(property "Reference" "C1"
+		(property "Reference" "C19"
 			(at 142.875 68.5735 0)
 			(show_name no)
@@
 			(project "PS-PrechargeBoard"
 				(path "/74d17fe6-68d4-4bd7-954a-e2bbb58b1f1e/ac0b82bc-5139-4aa7-86f9-8716cbcedbf0"
-					(reference "C1")
-					(unit 1)
-				)
+					(reference "C19")
+					(unit 1)
+				)

Commit message: hv 1.0
Parts:
- renumbered C19 to C18, C20 to C19, D5 to D3
Changed lines of the file:
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@@
 		(dnp no)
 		(fields_autoplaced yes)
-		(property "Reference" "C20"
+		(property "Reference" "C19"
 			(at 168.275 68.5735 0)
 			(show_name no)
@@
 			(project "PS-PrechargeBoard"
 				(path "/74d17fe6-68d4-4bd7-954a-e2bbb58b1f1e/ac0b82bc-5139-4aa7-86f9-8716cbcedbf0"
-					(reference "C20")
+					(reference "C19")
 					(unit 1)
 				)
@@
 		(dnp no)
 		(fields_autoplaced yes)
-		(property "Reference" "D5"
+		(property "Reference" "D3"
 			(at 133.604 57.15 0)
 			(show_name no)
@@
 			(project "PS-PrechargeBoard"
 				(path "/74d17fe6-68d4-4bd7-954a-e2bbb58b1f1e/ac0b82bc-5139-4aa7-86f9-8716cbcedbf0"
-					(reference "D5")
+					(reference "D3")
 					(unit 1)
 				)
@@
 		(dnp no)
 		(fields_autoplaced yes)
-		(property "Reference" "C19"
+		(property "Reference" "C18"
 			(at 142.875 68.5735 0)
 			(show_name no)
@@
 			(project "PS-PrechargeBoard"
 				(path "/74d17fe6-68d4-4bd7-954a-e2bbb58b1f1e/ac0b82bc-5139-4aa7-86f9-8716cbcedbf0"
-					(reference "C19")
-					(unit 1)
-				)
+					(reference "C18")
+					(unit 1)
+				)

Commit message: hv 1.3
Parts:
- renumbered C19 to C?, C18 to C?, D3 to D?, TP_3.3V1 to TP_3.3V?, U3 to U?
Changed lines of the file:
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@@
 		(dnp no)
 		(fields_autoplaced yes)
-		(property "Reference" "C19"
+		(property "Reference" "C?"
 			(at 168.275 68.5735 0)
 			(show_name no)
@@
 		(instances
 			(project "PS-PrechargeBoard"
-				(path "/74d17fe6-68d4-4bd7-954a-e2bbb58b1f1e/ac0b82bc-5139-4aa7-86f9-8716cbcedbf0"
-					(reference "C19")
-					(unit 1)
-				)
-			)
-			(project "LDO"
-				(path "/8ff43370-8d10-4d2c-b1a3-81d1c2934a98"
-					(reference "C2")
-					(unit 1)
-				)
-			)
-			(project "LeaderSOMBreakout"
-				(path "/e5b32072-3e3d-42a6-9d41-1a76d538e329/f3053c74-1ac6-4a33-80f3-565e8c4c2c7d"
+				(path "/11743897-1544-4e3c-979c-dcc54ac7093b/d07b4748-03cd-4373-ba6d-42f770522878"
 					(reference "C?")
 					(unit 1)
@@
 		(in_pos_files yes)
 		(dnp no)
-		(property "Reference" "TP_3.3V1"
+		(property "Reference" "TP_3.3V?"
 			(at 166.624 54.356 90)
 			(show_name no)
@@
 		(instances
 			(project "PS-PrechargeBoard"
-				(path "/74d17fe6-68d4-4bd7-954a-e2bbb58b1f1e/ac0b82bc-5139-4aa7-86f9-8716cbcedbf0"
-					(reference "TP_3.3V1")
-					(unit 1)
-				)
-			)
-			(project "LDO"
-				(path "/8ff43370-8d10-4d2c-b1a3-81d1c2934a98"
-					(reference "TP_3.3V1")
+				(path "/11743897-1544-4e3c-979c-dcc54ac7093b/d07b4748-03cd-4373-ba6d-42f770522878"
+					(reference "TP_3.3V?")
 					(unit 1)
 				)
@@
 		(dnp no)
 		(fields_autoplaced yes)
-		(property "Reference" "U3"
+		(property "Reference" "U?"
 			(at 152.4 56.515 0)
 			(show_name no)
@@
 		(instances
 			(project "PS-PrechargeBoard"
-				(path "/74d17fe6-68d4-4bd7-954a-e2bbb58b1f1e/ac0b82bc-5139-4aa7-86f9-8716cbcedbf0"
-					(reference "U3")
-					(unit 1)
-				)
-			)
-			(project ""
-				(path "/8ff43370-8d10-4d2c-b1a3-81d1c2934a98"
-					(reference "U1")
+				(path "/11743897-1544-4e3c-979c-dcc54ac7093b/d07b4748-03cd-4373-ba6d-42f770522878"
+					(reference "U?")
 					(unit 1)
 				)
@@
 		(dnp no)
 		(fields_autoplaced yes)
-		(property "Reference" "D3"
+		(property "Reference" "D?"
 			(at 133.604 57.15 0)
 			(show_name no)
@@
 		(instances
 			(project "PS-PrechargeBoard"
-				(path "/74d17fe6-68d4-4bd7-954a-e2bbb58b1f1e/ac0b82bc-5139-4aa7-86f9-8716cbcedbf0"
-					(reference "D3")
-					(unit 1)
-				)
-			)
-			(project ""
-				(path "/8ff43370-8d10-4d2c-b1a3-81d1c2934a98"
-					(reference "D1")
+				(path "/11743897-1544-4e3c-979c-dcc54ac7093b/d07b4748-03cd-4373-ba6d-42f770522878"
+					(reference "D?")
 					(unit 1)
 				)
@@
 		(dnp no)
 		(fields_autoplaced yes)
-		(property "Reference" "C18"
+		(property "Reference" "C?"
 			(at 142.875 68.5735 0)
 			(show_name no)
@@
 		(instances
 			(project "PS-PrechargeBoard"
-				(path "/74d17fe6-68d4-4bd7-954a-e2bbb58b1f1e/ac0b82bc-5139-4aa7-86f9-8716cbcedbf0"
-					(reference "C18")
-					(unit 1)
-				)
-			)
-			(project "LDO"
-				(path "/8ff43370-8d10-4d2c-b1a3-81d1c2934a98"
-					(reference "C1")
-					(unit 1)
-				)
-			)
-			(project ""
-				(path "/e5b32072-3e3d-42a6-9d41-1a76d538e329/f3053c74-1ac6-4a33-80f3-565e8c4c2c7d"
+				(path "/11743897-1544-4e3c-979c-dcc54ac7093b/d07b4748-03cd-4373-ba6d-42f770522878"
 					(reference "C?")
 					(unit 1)
