File: PowerProtection.kicad_sch (KiCad schematic)
At the start: 18 parts, among them IC1 LM74502DDFR, Q1 PSMN012-100YS, Q2 PSMN012-100YS

Commit message: lv 1.2
Parts:
- renumbered D2 to D1, D1 to D2, R1 to R3, R3 to R4, R4 to R5, R5 to R6, R6 to R8
Changed lines of the file:
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@@
 		(in_pos_files yes)
 		(dnp no)
-		(property "Reference" "D1"
+		(property "Reference" "D2"
 			(at 40.64 82.296 0)
 			(show_name no)
@@
 			(project "PS-PrechargeBoard"
 				(path "/74d17fe6-68d4-4bd7-954a-e2bbb58b1f1e/5dc15275-6052-4c98-bd51-73c91f41d1ab"
-					(reference "D1")
+					(reference "D2")
 					(unit 1)
 				)
@@
 		(in_pos_files yes)
 		(dnp no)
-		(property "Reference" "D2"
+		(property "Reference" "D1"
 			(at 22.606 49.276 0)
 			(show_name no)
@@
 			(project "PS-PrechargeBoard"
 				(path "/74d17fe6-68d4-4bd7-954a-e2bbb58b1f1e/5dc15275-6052-4c98-bd51-73c91f41d1ab"
-					(reference "D2")
+					(reference "D1")
 					(unit 1)
 				)
@@
 		(dnp no)
 		(fields_autoplaced yes)
-		(property "Reference" "R1"
+		(property "Reference" "R3"
 			(at 45.72 60.9599 0)
 			(show_name no)
@@
 			(project "PS-PrechargeBoard"
 				(path "/74d17fe6-68d4-4bd7-954a-e2bbb58b1f1e/5dc15275-6052-4c98-bd51-73c91f41d1ab"
-					(reference "R1")
+					(reference "R3")
 					(unit 1)
 				)
@@
 		(in_pos_files yes)
 		(dnp no)
-		(property "Reference" "R6"
+		(property "Reference" "R8"
 			(at 137.668 90.17 90)
 			(show_name no)
@@
 			(project "PS-PrechargeBoard"
 				(path "/74d17fe6-68d4-4bd7-954a-e2bbb58b1f1e/5dc15275-6052-4c98-bd51-73c91f41d1ab"
-					(reference "R6")
+					(reference "R8")
 					(unit 1)
 				)
@@
 		(in_pos_files yes)
 		(dnp no)
-		(property "Reference" "R3"
+		(property "Reference" "R4"
 			(at 67.31 54.61 90)
 			(show_name no)
@@
 			(project "PS-PrechargeBoard"
 				(path "/74d17fe6-68d4-4bd7-954a-e2bbb58b1f1e/5dc15275-6052-4c98-bd51-73c91f41d1ab"
-					(reference "R3")
+					(reference "R4")
 					(unit 1)
 				)
@@
 		(in_pos_files yes)
 		(dnp no)
-		(property "Reference" "R5"
+		(property "Reference" "R6"
 			(at 118.618 90.424 90)
 			(show_name no)
@@
 			(project "PS-PrechargeBoard"
 				(path "/74d17fe6-68d4-4bd7-954a-e2bbb58b1f1e/5dc15275-6052-4c98-bd51-73c91f41d1ab"
-					(reference "R5")
+					(reference "R6")
 					(unit 1)
 				)
@@
 		(in_pos_files yes)
 		(dnp no)
-		(property "Reference" "R4"
+		(property "Reference" "R5"
 			(at 118.11 78.74 90)
 			(show_name no)
@@
 			(project "PS-PrechargeBoard"
 				(path "/74d17fe6-68d4-4bd7-954a-e2bbb58b1f1e/5dc15275-6052-4c98-bd51-73c91f41d1ab"
-					(reference "R4")
-					(unit 1)
-				)
+					(reference "R5")
+					(unit 1)
+				)

Commit message: hv 1.0
Parts:
- renumbered R6 to R10, R7 to R11, R8 to R12, R3 to R7, R4 to R8, R5 to R9
Changed lines of the file:
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@@
 		(dnp no)
 		(fields_autoplaced yes)
-		(property "Reference" "R3"
+		(property "Reference" "R7"
 			(at 45.72 60.9599 0)
 			(show_name no)
@@
 			(project "PS-PrechargeBoard"
 				(path "/74d17fe6-68d4-4bd7-954a-e2bbb58b1f1e/5dc15275-6052-4c98-bd51-73c91f41d1ab"
-					(reference "R3")
+					(reference "R7")
 					(unit 1)
 				)
@@
 		(in_pos_files yes)
 		(dnp no)
-		(property "Reference" "R8"
+		(property "Reference" "R12"
 			(at 137.668 90.17 90)
 			(show_name no)
@@
 			(project "PS-PrechargeBoard"
 				(path "/74d17fe6-68d4-4bd7-954a-e2bbb58b1f1e/5dc15275-6052-4c98-bd51-73c91f41d1ab"
-					(reference "R8")
+					(reference "R12")
 					(unit 1)
 				)
@@
 		(in_pos_files yes)
 		(dnp no)
-		(property "Reference" "R4"
+		(property "Reference" "R8"
 			(at 67.31 54.61 90)
 			(show_name no)
@@
 			(project "PS-PrechargeBoard"
 				(path "/74d17fe6-68d4-4bd7-954a-e2bbb58b1f1e/5dc15275-6052-4c98-bd51-73c91f41d1ab"
-					(reference "R4")
+					(reference "R8")
 					(unit 1)
 				)
@@
 		(in_pos_files yes)
 		(dnp no)
-		(property "Reference" "R6"
+		(property "Reference" "R10"
 			(at 118.618 90.424 90)
 			(show_name no)
@@
 			(project "PS-PrechargeBoard"
 				(path "/74d17fe6-68d4-4bd7-954a-e2bbb58b1f1e/5dc15275-6052-4c98-bd51-73c91f41d1ab"
-					(reference "R6")
+					(reference "R10")
 					(unit 1)
 				)
@@
 		(in_pos_files yes)
 		(dnp no)
-		(property "Reference" "R5"
+		(property "Reference" "R9"
 			(at 118.11 78.74 90)
 			(show_name no)
@@
 			(project "PS-PrechargeBoard"
 				(path "/74d17fe6-68d4-4bd7-954a-e2bbb58b1f1e/5dc15275-6052-4c98-bd51-73c91f41d1ab"
-					(reference "R5")
+					(reference "R9")
 					(unit 1)
 				)
@@
 		(in_pos_files yes)
 		(dnp no)
-		(property "Reference" "R7"
+		(property "Reference" "R11"
 			(at 137.16 77.47 90)
 			(show_name no)
@@
 			(project "PS-PrechargeBoard"
 				(path "/74d17fe6-68d4-4bd7-954a-e2bbb58b1f1e/5dc15275-6052-4c98-bd51-73c91f41d1ab"
-					(reference "R7")
-					(unit 1)
-				)
+					(reference "R11")
+					(unit 1)
+				)

Commit message: hv 1.1
Parts:
- renumbered R11 to R10, R12 to R11, R7 to R6, R8 to R7, R9 to R8, R10 to R9
Changed lines of the file:
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@@
 		(dnp no)
 		(fields_autoplaced yes)
-		(property "Reference" "R7"
+		(property "Reference" "R6"
 			(at 45.72 60.9599 0)
 			(show_name no)
@@
 			(project "PS-PrechargeBoard"
 				(path "/74d17fe6-68d4-4bd7-954a-e2bbb58b1f1e/5dc15275-6052-4c98-bd51-73c91f41d1ab"
-					(reference "R7")
+					(reference "R6")
 					(unit 1)
 				)
@@
 		(in_pos_files yes)
 		(dnp no)
-		(property "Reference" "R12"
+		(property "Reference" "R11"
 			(at 137.668 90.17 90)
 			(show_name no)
@@
 			(project "PS-PrechargeBoard"
 				(path "/74d17fe6-68d4-4bd7-954a-e2bbb58b1f1e/5dc15275-6052-4c98-bd51-73c91f41d1ab"
-					(reference "R12")
+					(reference "R11")
 					(unit 1)
 				)
@@
 		(in_pos_files yes)
 		(dnp no)
-		(property "Reference" "R8"
+		(property "Reference" "R7"
 			(at 67.31 54.61 90)
 			(show_name no)
@@
 			(project "PS-PrechargeBoard"
 				(path "/74d17fe6-68d4-4bd7-954a-e2bbb58b1f1e/5dc15275-6052-4c98-bd51-73c91f41d1ab"
-					(reference "R8")
+					(reference "R7")
 					(unit 1)
 				)
@@
 		(in_pos_files yes)
 		(dnp no)
-		(property "Reference" "R10"
+		(property "Reference" "R9"
 			(at 118.618 90.424 90)
 			(show_name no)
@@
 			(project "PS-PrechargeBoard"
 				(path "/74d17fe6-68d4-4bd7-954a-e2bbb58b1f1e/5dc15275-6052-4c98-bd51-73c91f41d1ab"
-					(reference "R10")
+					(reference "R9")
 					(unit 1)
 				)
@@
 		(in_pos_files yes)
 		(dnp no)
-		(property "Reference" "R9"
+		(property "Reference" "R8"
 			(at 118.11 78.74 90)
 			(show_name no)
@@
 			(project "PS-PrechargeBoard"
 				(path "/74d17fe6-68d4-4bd7-954a-e2bbb58b1f1e/5dc15275-6052-4c98-bd51-73c91f41d1ab"
-					(reference "R9")
+					(reference "R8")
 					(unit 1)
 				)
@@
 		(in_pos_files yes)
 		(dnp no)
-		(property "Reference" "R11"
+		(property "Reference" "R10"
 			(at 137.16 77.47 90)
 			(show_name no)
@@
 			(project "PS-PrechargeBoard"
 				(path "/74d17fe6-68d4-4bd7-954a-e2bbb58b1f1e/5dc15275-6052-4c98-bd51-73c91f41d1ab"
-					(reference "R11")
-					(unit 1)
-				)
+					(reference "R10")
+					(unit 1)
+				)

Commit message: hv 1.3
Parts:
- renumbered C3 to C?, C1 to C?, C6 to C?, C4 to C?, C5 to C?, C2 to C?, C7 to C?, D2 to D?, D1 to D?, IC1 to IC?, Q1 to Q?, Q2 to Q?, R6 to R?, R11 to R?, R7 to R?, R9 to R?, R8 to R?, R10 to R?
