File: PowerProtection.kicad_sch (KiCad schematic)
At the start: 18 parts

Commit message: CAN nano & CAN debug nano
Parts:
- gave numbers to parts that had none: 18

Commit message: battery voltage & motor voltage
Parts:
- renumbered C21 to C10, C22 to C11, C23 to C12, C24 to C13, C25 to C14, C26 to C15, C20 to C9, D5 to D4, D6 to D5, IC2 to IC1, R11 to R17, R12 to R18, R13 to R19, R14 to R20, R15 to R21, R16 to R22
Changed lines of the file:
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@@
 		(in_pos_files yes)
 		(dnp no)
-		(property "Reference" "D6"
+		(property "Reference" "D5"
 			(at 40.64 82.296 0)
 			(show_name no)
@@
 			(project "PS-PrechargeBoard"
 				(path "/74d17fe6-68d4-4bd7-954a-e2bbb58b1f1e/0def18ef-81e8-47ac-b719-2d9f8237a855/9b47e6f4-7691-492a-9adf-22bd19fd1cb1"
-					(reference "D6")
+					(reference "D5")
 					(unit 1)
 				)
@@
 		(dnp no)
 		(fields_autoplaced yes)
-		(property "Reference" "C22"
+		(property "Reference" "C11"
 			(at 57.785 80.0099 0)
 			(show_name no)
@@
 			(project "PS-PrechargeBoard"
 				(path "/74d17fe6-68d4-4bd7-954a-e2bbb58b1f1e/0def18ef-81e8-47ac-b719-2d9f8237a855/9b47e6f4-7691-492a-9adf-22bd19fd1cb1"
-					(reference "C22")
+					(reference "C11")
 					(unit 1)
 				)
@@
 		(in_pos_files yes)
 		(dnp no)
-		(property "Reference" "D5"
+		(property "Reference" "D4"
 			(at 22.606 49.276 0)
 			(show_name no)
@@
 			(project "PS-PrechargeBoard"
 				(path "/74d17fe6-68d4-4bd7-954a-e2bbb58b1f1e/0def18ef-81e8-47ac-b719-2d9f8237a855/9b47e6f4-7691-492a-9adf-22bd19fd1cb1"
-					(reference "D5")
+					(reference "D4")
 					(unit 1)
 				)
@@
 		(dnp no)
 		(fields_autoplaced yes)
-		(property "Reference" "R11"
+		(property "Reference" "R17"
 			(at 45.72 60.9599 0)
 			(show_name no)
@@
 			(project "PS-PrechargeBoard"
 				(path "/74d17fe6-68d4-4bd7-954a-e2bbb58b1f1e/0def18ef-81e8-47ac-b719-2d9f8237a855/9b47e6f4-7691-492a-9adf-22bd19fd1cb1"
-					(reference "R11")
+					(reference "R17")
 					(unit 1)
 				)
@@
 		(in_pos_files yes)
 		(dnp no)
-		(property "Reference" "R16"
+		(property "Reference" "R22"
 			(at 137.668 90.17 90)
 			(show_name no)
@@
 			(project "PS-PrechargeBoard"
 				(path "/74d17fe6-68d4-4bd7-954a-e2bbb58b1f1e/0def18ef-81e8-47ac-b719-2d9f8237a855/9b47e6f4-7691-492a-9adf-22bd19fd1cb1"
-					(reference "R16")
+					(reference "R22")
 					(unit 1)
 				)
@@
 		(in_pos_files yes)
 		(dnp no)
-		(property "Reference" "C20"
+		(property "Reference" "C9"
 			(at 38.1 49.5299 0)
 			(show_name no)
@@
 			(project "PS-PrechargeBoard"
 				(path "/74d17fe6-68d4-4bd7-954a-e2bbb58b1f1e/0def18ef-81e8-47ac-b719-2d9f8237a855/9b47e6f4-7691-492a-9adf-22bd19fd1cb1"
-					(reference "C20")
+					(reference "C9")
 					(unit 1)
 				)
@@
 		(in_pos_files yes)
 		(dnp no)
-		(property "Reference" "R12"
+		(property "Reference" "R18"
 			(at 67.31 54.61 90)
 			(show_name no)
@@
 			(project "PS-PrechargeBoard"
 				(path "/74d17fe6-68d4-4bd7-954a-e2bbb58b1f1e/0def18ef-81e8-47ac-b719-2d9f8237a855/9b47e6f4-7691-492a-9adf-22bd19fd1cb1"
-					(reference "R12")
+					(reference "R18")
 					(unit 1)
 				)
@@
 		(in_pos_files yes)
 		(dnp no)
-		(property "Reference" "IC2"
+		(property "Reference" "IC1"
 			(at 75.184 73.66 0)
 			(show_name no)
@@
 			(project "PS-PrechargeBoard"
 				(path "/74d17fe6-68d4-4bd7-954a-e2bbb58b1f1e/0def18ef-81e8-47ac-b719-2d9f8237a855/9b47e6f4-7691-492a-9adf-22bd19fd1cb1"
-					(reference "IC2")
+					(reference "IC1")
 					(unit 1)
 				)
@@
 		(in_pos_files yes)
 		(dnp no)
-		(property "Reference" "C25"
+		(property "Reference" "C14"
 			(at 113.284 89.154 0)
 			(show_name no)
@@
 			(project "PS-PrechargeBoard"
 				(path "/74d17fe6-68d4-4bd7-954a-e2bbb58b1f1e/0def18ef-81e8-47ac-b719-2d9f8237a855/9b47e6f4-7691-492a-9adf-22bd19fd1cb1"
-					(reference "C25")
+					(reference "C14")
 					(unit 1)
 				)
@@
 		(in_pos_files yes)
 		(dnp no)
-		(property "Reference" "C23"
+		(property "Reference" "C12"
 			(at 54.864 62.23 0)
 			(show_name no)
@@
 			(project "PS-PrechargeBoard"
 				(path "/74d17fe6-68d4-4bd7-954a-e2bbb58b1f1e/0def18ef-81e8-47ac-b719-2d9f8237a855/9b47e6f4-7691-492a-9adf-22bd19fd1cb1"
-					(reference "C23")
+					(reference "C12")
 					(unit 1)
 				)
@@
 		(in_pos_files yes)
 		(dnp no)
-		(property "Reference" "C24"
+		(property "Reference" "C13"
 			(at 112.395 49.5299 0)
 			(show_name no)
@@
 			(project "PS-PrechargeBoard"
 				(path "/74d17fe6-68d4-4bd7-954a-e2bbb58b1f1e/0def18ef-81e8-47ac-b719-2d9f8237a855/9b47e6f4-7691-492a-9adf-22bd19fd1cb1"
-					(reference "C24")
+					(reference "C13")
 					(unit 1)
 				)
@@
 		(in_pos_files yes)
 		(dnp no)
-		(property "Reference" "R14"
+		(property "Reference" "R20"
 			(at 118.618 90.424 90)
 			(show_name no)
@@
 			(project "PS-PrechargeBoard"
 				(path "/74d17fe6-68d4-4bd7-954a-e2bbb58b1f1e/0def18ef-81e8-47ac-b719-2d9f8237a855/9b47e6f4-7691-492a-9adf-22bd19fd1cb1"
-					(reference "R14")
+					(reference "R20")
 					(unit 1)
 				)
@@
 		(in_pos_files yes)
 		(dnp no)
-		(property "Reference" "C21"
+		(property "Reference" "C10"
 			(at 31.75 82.5499 0)
 			(show_name no)
@@
 			(project "PS-PrechargeBoard"
 				(path "/74d17fe6-68d4-4bd7-954a-e2bbb58b1f1e/0def18ef-81e8-47ac-b719-2d9f8237a855/9b47e6f4-7691-492a-9adf-22bd19fd1cb1"
-					(reference "C21")
+					(reference "C10")
 					(unit 1)
 				)
@@
 		(in_pos_files yes)
 		(dnp no)
-		(property "Reference" "C26"
+		(property "Reference" "C15"
 			(at 132.08 88.9 0)
 			(show_name no)
@@
 			(project "PS-PrechargeBoard"
 				(path "/74d17fe6-68d4-4bd7-954a-e2bbb58b1f1e/0def18ef-81e8-47ac-b719-2d9f8237a855/9b47e6f4-7691-492a-9adf-22bd19fd1cb1"
-					(reference "C26")
+					(reference "C15")
 					(unit 1)
 				)
@@
 		(in_pos_files yes)
 		(dnp no)
-		(property "Reference" "R13"
+		(property "Reference" "R19"
 			(at 118.11 78.74 90)
 			(show_name no)
@@
 			(project "PS-PrechargeBoard"
 				(path "/74d17fe6-68d4-4bd7-954a-e2bbb58b1f1e/0def18ef-81e8-47ac-b719-2d9f8237a855/9b47e6f4-7691-492a-9adf-22bd19fd1cb1"
-					(reference "R13")
+					(reference "R19")
 					(unit 1)
 				)
@@
 		(in_pos_files yes)
 		(dnp no)
-		(property "Reference" "R15"
+		(property "Reference" "R21"
 			(at 137.16 77.47 90)
 			(show_name no)
@@
 			(project "PS-PrechargeBoard"
 				(path "/74d17fe6-68d4-4bd7-954a-e2bbb58b1f1e/0def18ef-81e8-47ac-b719-2d9f8237a855/9b47e6f4-7691-492a-9adf-22bd19fd1cb1"
-					(reference "R15")
-					(unit 1)
-				)
+					(reference "R21")
+					(unit 1)
+				)

Commit message: mini review notes
Parts:
- renumbered D4 to D6, D5 to D7
Changed lines of the file:
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@@
 		(in_pos_files yes)
 		(dnp no)
-		(property "Reference" "D5"
+		(property "Reference" "D7"
 			(at 40.64 82.296 0)
 			(show_name no)
@@
 			(project "PS-PrechargeBoard"
 				(path "/74d17fe6-68d4-4bd7-954a-e2bbb58b1f1e/0def18ef-81e8-47ac-b719-2d9f8237a855/9b47e6f4-7691-492a-9adf-22bd19fd1cb1"
-					(reference "D5")
+					(reference "D7")
 					(unit 1)
 				)
@@
 		(in_pos_files yes)
 		(dnp no)
-		(property "Reference" "D4"
+		(property "Reference" "D6"
 			(at 22.606 49.276 0)
 			(show_name no)
@@
 			(project "PS-PrechargeBoard"
 				(path "/74d17fe6-68d4-4bd7-954a-e2bbb58b1f1e/0def18ef-81e8-47ac-b719-2d9f8237a855/9b47e6f4-7691-492a-9adf-22bd19fd1cb1"
-					(reference "D4")
-					(unit 1)
-				)
+					(reference "D6")
+					(unit 1)
+				)

Commit message: shifted hierarchical sheets
Parts:
- renumbered C11 to C?, C9 to C?, C14 to C?, C12 to C?, C13 to C?, C10 to C?, C15 to C?, D7 to D?, D6 to D?, IC1 to IC?, Q1 to Q?, Q2 to Q?, R17 to R?, R22 to R?, R18 to R?, R20 to R?, R19 to R?, R21 to R?

Commit message: V_OUT_BAT & V_OUT_MOT & PRECHARGE_CTRL to MCU
Parts:
- gave numbers to parts that had none: 18
Changed lines of the file:
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@@
 		(in_pos_files yes)
 		(dnp no)
-		(property "Reference" "D?"
+		(property "Reference" "D12"
 			(at 40.64 82.296 0)
 			(show_name no)
@@
 			(project "PS-PrechargeBoard"
 				(path "/74d17fe6-68d4-4bd7-954a-e2bbb58b1f1e/3c8d3f54-ba9f-4300-800c-08eda88a8ae0"
-					(reference "D?")
+					(reference "D12")
 					(unit 1)
 				)
@@
 		(dnp no)
 		(fields_autoplaced yes)
-		(property "Reference" "C?"
+		(property "Reference" "C51"
 			(at 57.785 80.0099 0)
 			(show_name no)
@@
 			(project "PS-PrechargeBoard"
 				(path "/74d17fe6-68d4-4bd7-954a-e2bbb58b1f1e/3c8d3f54-ba9f-4300-800c-08eda88a8ae0"
-					(reference "C?")
+					(reference "C51")
 					(unit 1)
 				)
@@
 		(in_pos_files yes)
 		(dnp no)
-		(property "Reference" "D?"
+		(property "Reference" "D11"
 			(at 22.606 49.276 0)
 			(show_name no)
@@
 			(project "PS-PrechargeBoard"
 				(path "/74d17fe6-68d4-4bd7-954a-e2bbb58b1f1e/3c8d3f54-ba9f-4300-800c-08eda88a8ae0"
-					(reference "D?")
+					(reference "D11")
 					(unit 1)
 				)
@@
 		(dnp no)
 		(fields_autoplaced yes)
-		(property "Reference" "R?"
+		(property "Reference" "R41"
 			(at 45.72 60.9599 0)
 			(show_name no)
@@
 			(project "PS-PrechargeBoard"
 				(path "/74d17fe6-68d4-4bd7-954a-e2bbb58b1f1e/3c8d3f54-ba9f-4300-800c-08eda88a8ae0"
-					(reference "R?")
+					(reference "R41")
 					(unit 1)
 				)
@@
 		(in_pos_files yes)
 		(dnp no)
-		(property "Reference" "R?"
+		(property "Reference" "R46"
 			(at 137.668 90.17 90)
 			(show_name no)
@@
 			(project "PS-PrechargeBoard"
 				(path "/74d17fe6-68d4-4bd7-954a-e2bbb58b1f1e/3c8d3f54-ba9f-4300-800c-08eda88a8ae0"
-					(reference "R?")
+					(reference "R46")
 					(unit 1)
 				)
@@
 		(in_pos_files yes)
 		(dnp no)
-		(property "Reference" "C?"
+		(property "Reference" "C49"
 			(at 38.1 49.5299 0)
 			(show_name no)
@@
 			(project "PS-PrechargeBoard"
 				(path "/74d17fe6-68d4-4bd7-954a-e2bbb58b1f1e/3c8d3f54-ba9f-4300-800c-08eda88a8ae0"
-					(reference "C?")
+					(reference "C49")
 					(unit 1)
 				)
@@
 		(in_pos_files yes)
 		(dnp no)
-		(property "Reference" "R?"
+		(property "Reference" "R42"
 			(at 67.31 54.61 90)
 			(show_name no)
@@
 			(project "PS-PrechargeBoard"
 				(path "/74d17fe6-68d4-4bd7-954a-e2bbb58b1f1e/3c8d3f54-ba9f-4300-800c-08eda88a8ae0"
-					(reference "R?")
+					(reference "R42")
 					(unit 1)
 				)
@@
 		(in_pos_files yes)
 		(dnp no)
-		(property "Reference" "IC?"
+		(property "Reference" "IC4"
 			(at 75.184 73.66 0)
 			(show_name no)
@@
 			(project "PS-PrechargeBoard"
 				(path "/74d17fe6-68d4-4bd7-954a-e2bbb58b1f1e/3c8d3f54-ba9f-4300-800c-08eda88a8ae0"
-					(reference "IC?")
+					(reference "IC4")
 					(unit 1)
 				)
@@
 		(in_pos_files yes)
 		(dnp no)
-		(property "Reference" "Q?"
+		(property "Reference" "Q2"
 			(at 52.578 38.862 90)
 			(show_name no)
@@
 			(project "PS-PrechargeBoard"
 				(path "/74d17fe6-68d4-4bd7-954a-e2bbb58b1f1e/3c8d3f54-ba9f-4300-800c-08eda88a8ae0"
-					(reference "Q?")
+					(reference "Q2")
 					(unit 1)
 				)
@@
 		(in_pos_files yes)
 		(dnp no)
-		(property "Reference" "C?"
+		(property "Reference" "C54"
 			(at 113.284 89.154 0)
 			(show_name no)
@@
 			(project "PS-PrechargeBoard"
 				(path "/74d17fe6-68d4-4bd7-954a-e2bbb58b1f1e/3c8d3f54-ba9f-4300-800c-08eda88a8ae0"
-					(reference "C?")
+					(reference "C54")
 					(unit 1)
 				)
@@
 		(in_pos_files yes)
 		(dnp no)
-		(property "Reference" "C?"
+		(property "Reference" "C52"
 			(at 54.864 62.23 0)
 			(show_name no)
@@
 			(project "PS-PrechargeBoard"
 				(path "/74d17fe6-68d4-4bd7-954a-e2bbb58b1f1e/3c8d3f54-ba9f-4300-800c-08eda88a8ae0"
-					(reference "C?")
+					(reference "C52")
 					(unit 1)
 				)
@@
 		(in_pos_files yes)
 		(dnp no)
-		(property "Reference" "C?"
+		(property "Reference" "C53"
 			(at 112.395 49.5299 0)
 			(show_name no)
@@
 			(project "PS-PrechargeBoard"
 				(path "/74d17fe6-68d4-4bd7-954a-e2bbb58b1f1e/3c8d3f54-ba9f-4300-800c-08eda88a8ae0"
-					(reference "C?")
+					(reference "C53")
 					(unit 1)
 				)
@@
 		(in_pos_files yes)
 		(dnp no)
-		(property "Reference" "Q?"
+		(property "Reference" "Q3"
 			(at 100.584 38.608 90)
 			(show_name no)
@@
 			(project "PS-PrechargeBoard"
 				(path "/74d17fe6-68d4-4bd7-954a-e2bbb58b1f1e/3c8d3f54-ba9f-4300-800c-08eda88a8ae0"
-					(reference "Q?")
+					(reference "Q3")
 					(unit 1)
 				)
@@
 		(in_pos_files yes)
 		(dnp no)
-		(property "Reference" "R?"
+		(property "Reference" "R44"
 			(at 118.618 90.424 90)
 			(show_name no)
@@
 			(project "PS-PrechargeBoard"
 				(path "/74d17fe6-68d4-4bd7-954a-e2bbb58b1f1e/3c8d3f54-ba9f-4300-800c-08eda88a8ae0"
-					(reference "R?")
+					(reference "R44")
 					(unit 1)
 				)
@@
 		(in_pos_files yes)
 		(dnp no)
-		(property "Reference" "C?"
+		(property "Reference" "C50"
 			(at 31.75 82.5499 0)
 			(show_name no)
@@
 			(project "PS-PrechargeBoard"
 				(path "/74d17fe6-68d4-4bd7-954a-e2bbb58b1f1e/3c8d3f54-ba9f-4300-800c-08eda88a8ae0"
-					(reference "C?")
+					(reference "C50")
 					(unit 1)
 				)
@@
 		(in_pos_files yes)
 		(dnp no)
-		(property "Reference" "C?"
+		(property "Reference" "C55"
 			(at 132.08 88.9 0)
 			(show_name no)
@@
 			(project "PS-PrechargeBoard"
 				(path "/74d17fe6-68d4-4bd7-954a-e2bbb58b1f1e/3c8d3f54-ba9f-4300-800c-08eda88a8ae0"
-					(reference "C?")
+					(reference "C55")
 					(unit 1)
 				)
@@
 		(in_pos_files yes)
 		(dnp no)
-		(property "Reference" "R?"
+		(property "Reference" "R43"
 			(at 118.11 78.74 90)
 			(show_name no)
@@
 			(project "PS-PrechargeBoard"
 				(path "/74d17fe6-68d4-4bd7-954a-e2bbb58b1f1e/3c8d3f54-ba9f-4300-800c-08eda88a8ae0"
-					(reference "R?")
+					(reference "R43")
 					(unit 1)
 				)
@@
 		(in_pos_files yes)
 		(dnp no)
-		(property "Reference" "R?"
+		(property "Reference" "R45"
 			(at 137.16 77.47 90)
 			(show_name no)
@@
 			(project "PS-PrechargeBoard"
 				(path "/74d17fe6-68d4-4bd7-954a-e2bbb58b1f1e/3c8d3f54-ba9f-4300-800c-08eda88a8ae0"
-					(reference "R?")
+					(reference "R45")
 					(unit 1)
 				)

Commit message: precharges & voltage sensors
Parts:
- renumbered C49 to C30, C50 to C31, C51 to C32, C52 to C33, C53 to C34, C54 to C35, C55 to C36, D11 to D3, D12 to D4, IC4 to IC3, Q2 to Q1, Q3 to Q2, R41 to R26, R42 to R27, R43 to R28, R44 to R29, R45 to R30, R46 to R31
Changed lines of the file:
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@@
 		(in_pos_files yes)
 		(dnp no)
-		(property "Reference" "D12"
+		(property "Reference" "D4"
 			(at 40.64 82.296 0)
 			(show_name no)
@@
 		(instances
 			(project "PS-PrechargeBoard"
-				(path "/74d17fe6-68d4-4bd7-954a-e2bbb58b1f1e/3c8d3f54-ba9f-4300-800c-08eda88a8ae0"
-					(reference "D12")
+				(path "/74d17fe6-68d4-4bd7-954a-e2bbb58b1f1e/c6e51092-efec-40a8-afae-63cae62691f2/9aee96ea-fe7f-4344-be59-bff28dc77cb5"
+					(reference "D4")
 					(unit 1)
 				)
@@
 		(dnp no)
 		(fields_autoplaced yes)
-		(property "Reference" "C51"
+		(property "Reference" "C32"
 			(at 57.785 80.0099 0)
 			(show_name no)
@@
 		(instances
 			(project "PS-PrechargeBoard"
-				(path "/74d17fe6-68d4-4bd7-954a-e2bbb58b1f1e/3c8d3f54-ba9f-4300-800c-08eda88a8ae0"
-					(reference "C51")
+				(path "/74d17fe6-68d4-4bd7-954a-e2bbb58b1f1e/c6e51092-efec-40a8-afae-63cae62691f2/9aee96ea-fe7f-4344-be59-bff28dc77cb5"
+					(reference "C32")
 					(unit 1)
 				)
@@
 		(in_pos_files yes)
 		(dnp no)
-		(property "Reference" "D11"
+		(property "Reference" "D3"
 			(at 22.606 49.276 0)
 			(show_name no)
@@
 		(instances
 			(project "PS-PrechargeBoard"
-				(path "/74d17fe6-68d4-4bd7-954a-e2bbb58b1f1e/3c8d3f54-ba9f-4300-800c-08eda88a8ae0"
-					(reference "D11")
+				(path "/74d17fe6-68d4-4bd7-954a-e2bbb58b1f1e/c6e51092-efec-40a8-afae-63cae62691f2/9aee96ea-fe7f-4344-be59-bff28dc77cb5"
+					(reference "D3")
 					(unit 1)
 				)
@@
 		(dnp no)
 		(fields_autoplaced yes)
-		(property "Reference" "R41"
+		(property "Reference" "R26"
 			(at 45.72 60.9599 0)
 			(show_name no)
@@
 		(instances
 			(project "PS-PrechargeBoard"
-				(path "/74d17fe6-68d4-4bd7-954a-e2bbb58b1f1e/3c8d3f54-ba9f-4300-800c-08eda88a8ae0"
-					(reference "R41")
+				(path "/74d17fe6-68d4-4bd7-954a-e2bbb58b1f1e/c6e51092-efec-40a8-afae-63cae62691f2/9aee96ea-fe7f-4344-be59-bff28dc77cb5"
+					(reference "R26")
 					(unit 1)
 				)
@@
 		(in_pos_files yes)
 		(dnp no)
-		(property "Reference" "R46"
+		(property "Reference" "R31"
 			(at 137.668 90.17 90)
 			(show_name no)
@@
 		(instances
 			(project "PS-PrechargeBoard"
-				(path "/74d17fe6-68d4-4bd7-954a-e2bbb58b1f1e/3c8d3f54-ba9f-4300-800c-08eda88a8ae0"
-					(reference "R46")
+				(path "/74d17fe6-68d4-4bd7-954a-e2bbb58b1f1e/c6e51092-efec-40a8-afae-63cae62691f2/9aee96ea-fe7f-4344-be59-bff28dc77cb5"
+					(reference "R31")
 					(unit 1)
 				)
@@
 		(in_pos_files yes)
 		(dnp no)
-		(property "Reference" "C49"
+		(property "Reference" "C30"
 			(at 38.1 49.5299 0)
 			(show_name no)
@@
 		(instances
 			(project "PS-PrechargeBoard"
-				(path "/74d17fe6-68d4-4bd7-954a-e2bbb58b1f1e/3c8d3f54-ba9f-4300-800c-08eda88a8ae0"
-					(reference "C49")
+				(path "/74d17fe6-68d4-4bd7-954a-e2bbb58b1f1e/c6e51092-efec-40a8-afae-63cae62691f2/9aee96ea-fe7f-4344-be59-bff28dc77cb5"
+					(reference "C30")
 					(unit 1)
 				)
@@
 		(in_pos_files yes)
 		(dnp no)
-		(property "Reference" "R42"
+		(property "Reference" "R27"
 			(at 67.31 54.61 90)
 			(show_name no)
@@
 		(instances
 			(project "PS-PrechargeBoard"
-				(path "/74d17fe6-68d4-4bd7-954a-e2bbb58b1f1e/3c8d3f54-ba9f-4300-800c-08eda88a8ae0"
-					(reference "R42")
+				(path "/74d17fe6-68d4-4bd7-954a-e2bbb58b1f1e/c6e51092-efec-40a8-afae-63cae62691f2/9aee96ea-fe7f-4344-be59-bff28dc77cb5"
+					(reference "R27")
 					(unit 1)
 				)
@@
 		(in_pos_files yes)
 		(dnp no)
-		(property "Reference" "IC4"
+		(property "Reference" "IC3"
 			(at 75.184 73.66 0)
 			(show_name no)
@@
 		(instances
 			(project "PS-PrechargeBoard"
-				(path "/74d17fe6-68d4-4bd7-954a-e2bbb58b1f1e/3c8d3f54-ba9f-4300-800c-08eda88a8ae0"
-					(reference "IC4")
+				(path "/74d17fe6-68d4-4bd7-954a-e2bbb58b1f1e/c6e51092-efec-40a8-afae-63cae62691f2/9aee96ea-fe7f-4344-be59-bff28dc77cb5"
+					(reference "IC3")
 					(unit 1)
 				)
@@
 		(in_pos_files yes)
 		(dnp no)
-		(property "Reference" "Q2"
+		(property "Reference" "Q1"
 			(at 52.578 38.862 90)
 			(show_name no)
@@
 		(instances
 			(project "PS-PrechargeBoard"
-				(path "/74d17fe6-68d4-4bd7-954a-e2bbb58b1f1e/3c8d3f54-ba9f-4300-800c-08eda88a8ae0"
-					(reference "Q2")
+				(path "/74d17fe6-68d4-4bd7-954a-e2bbb58b1f1e/c6e51092-efec-40a8-afae-63cae62691f2/9aee96ea-fe7f-4344-be59-bff28dc77cb5"
+					(reference "Q1")
 					(unit 1)
 				)
@@
 		(in_pos_files yes)
 		(dnp no)
-		(property "Reference" "C54"
+		(property "Reference" "C35"
 			(at 113.284 89.154 0)
 			(show_name no)
@@
 		(instances
 			(project "PS-PrechargeBoard"
-				(path "/74d17fe6-68d4-4bd7-954a-e2bbb58b1f1e/3c8d3f54-ba9f-4300-800c-08eda88a8ae0"
-					(reference "C54")
+				(path "/74d17fe6-68d4-4bd7-954a-e2bbb58b1f1e/c6e51092-efec-40a8-afae-63cae62691f2/9aee96ea-fe7f-4344-be59-bff28dc77cb5"
+					(reference "C35")
 					(unit 1)
 				)
@@
 		(in_pos_files yes)
 		(dnp no)
-		(property "Reference" "C52"
+		(property "Reference" "C33"
 			(at 54.864 62.23 0)
 			(show_name no)
@@
 		(instances
 			(project "PS-PrechargeBoard"
-				(path "/74d17fe6-68d4-4bd7-954a-e2bbb58b1f1e/3c8d3f54-ba9f-4300-800c-08eda88a8ae0"
-					(reference "C52")
+				(path "/74d17fe6-68d4-4bd7-954a-e2bbb58b1f1e/c6e51092-efec-40a8-afae-63cae62691f2/9aee96ea-fe7f-4344-be59-bff28dc77cb5"
+					(reference "C33")
 					(unit 1)
 				)
@@
 		(in_pos_files yes)
 		(dnp no)
-		(property "Reference" "C53"
+		(property "Reference" "C34"
 			(at 112.395 49.5299 0)
 			(show_name no)
@@
 		(instances
 			(project "PS-PrechargeBoard"
-				(path "/74d17fe6-68d4-4bd7-954a-e2bbb58b1f1e/3c8d3f54-ba9f-4300-800c-08eda88a8ae0"
-					(reference "C53")
+				(path "/74d17fe6-68d4-4bd7-954a-e2bbb58b1f1e/c6e51092-efec-40a8-afae-63cae62691f2/9aee96ea-fe7f-4344-be59-bff28dc77cb5"
+					(reference "C34")
 					(unit 1)
 				)
@@
 		(in_pos_files yes)
 		(dnp no)
-		(property "Reference" "Q3"
+		(property "Reference" "Q2"
 			(at 100.584 38.608 90)
 			(show_name no)
@@
 		(instances
 			(project "PS-PrechargeBoard"
-				(path "/74d17fe6-68d4-4bd7-954a-e2bbb58b1f1e/3c8d3f54-ba9f-4300-800c-08eda88a8ae0"
-					(reference "Q3")
+				(path "/74d17fe6-68d4-4bd7-954a-e2bbb58b1f1e/c6e51092-efec-40a8-afae-63cae62691f2/9aee96ea-fe7f-4344-be59-bff28dc77cb5"
+					(reference "Q2")
 					(unit 1)
 				)
@@
 		(in_pos_files yes)
 		(dnp no)
-		(property "Reference" "R44"
+		(property "Reference" "R29"
 			(at 118.618 90.424 90)
 			(show_name no)
@@
 		(instances
 			(project "PS-PrechargeBoard"
-				(path "/74d17fe6-68d4-4bd7-954a-e2bbb58b1f1e/3c8d3f54-ba9f-4300-800c-08eda88a8ae0"
-					(reference "R44")
+				(path "/74d17fe6-68d4-4bd7-954a-e2bbb58b1f1e/c6e51092-efec-40a8-afae-63cae62691f2/9aee96ea-fe7f-4344-be59-bff28dc77cb5"
+					(reference "R29")
 					(unit 1)
 				)
@@
 		(in_pos_files yes)
 		(dnp no)
-		(property "Reference" "C50"
+		(property "Reference" "C31"
 			(at 31.75 82.5499 0)
 			(show_name no)
@@
 		(instances
 			(project "PS-PrechargeBoard"
-				(path "/74d17fe6-68d4-4bd7-954a-e2bbb58b1f1e/3c8d3f54-ba9f-4300-800c-08eda88a8ae0"
-					(reference "C50")
+				(path "/74d17fe6-68d4-4bd7-954a-e2bbb58b1f1e/c6e51092-efec-40a8-afae-63cae62691f2/9aee96ea-fe7f-4344-be59-bff28dc77cb5"
+					(reference "C31")
 					(unit 1)
 				)
@@
 		(in_pos_files yes)
 		(dnp no)
-		(property "Reference" "C55"
+		(property "Reference" "C36"
 			(at 132.08 88.9 0)
 			(show_name no)
@@
 		(instances
 			(project "PS-PrechargeBoard"
-				(path "/74d17fe6-68d4-4bd7-954a-e2bbb58b1f1e/3c8d3f54-ba9f-4300-800c-08eda88a8ae0"
-					(reference "C55")
+				(path "/74d17fe6-68d4-4bd7-954a-e2bbb58b1f1e/c6e51092-efec-40a8-afae-63cae62691f2/9aee96ea-fe7f-4344-be59-bff28dc77cb5"
+					(reference "C36")
 					(unit 1)
 				)
@@
 		(in_pos_files yes)
 		(dnp no)
-		(property "Reference" "R43"
+		(property "Reference" "R28"
 			(at 118.11 78.74 90)
 			(show_name no)
@@
 		(instances
 			(project "PS-PrechargeBoard"
-				(path "/74d17fe6-68d4-4bd7-954a-e2bbb58b1f1e/3c8d3f54-ba9f-4300-800c-08eda88a8ae0"
-					(reference "R43")
+				(path "/74d17fe6-68d4-4bd7-954a-e2bbb58b1f1e/c6e51092-efec-40a8-afae-63cae62691f2/9aee96ea-fe7f-4344-be59-bff28dc77cb5"
+					(reference "R28")
 					(unit 1)
 				)
@@
 		(in_pos_files yes)
 		(dnp no)
-		(property "Reference" "R45"
+		(property "Reference" "R30"
 			(at 137.16 77.47 90)
 			(show_name no)
@@
 		(instances
 			(project "PS-PrechargeBoard"
-				(path "/74d17fe6-68d4-4bd7-954a-e2bbb58b1f1e/3c8d3f54-ba9f-4300-800c-08eda88a8ae0"
-					(reference "R45")
+				(path "/74d17fe6-68d4-4bd7-954a-e2bbb58b1f1e/c6e51092-efec-40a8-afae-63cae62691f2/9aee96ea-fe7f-4344-be59-bff28dc77cb5"
+					(reference "R30")
 					(unit 1)
 				)
