File: PowerProtection.kicad_sch (KiCad schematic)
At the start: 18 parts, among them IC3 LM74502DDFR, Q1 PSMN012-100YS, Q2 PSMN012-100YS

Commit message: saving
Parts:
- renumbered C32 to C?, C30 to C?, C35 to C?, C33 to C?, C34 to C?, C31 to C?, C36 to C?, D4 to D?, D3 to D?, IC3 to IC?, Q1 to Q?, Q2 to Q?, R26 to R?, R31 to R?, R27 to R?, R29 to R?, R28 to R?, R30 to R?
Changed lines of the file:
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@@
 		(in_pos_files yes)
 		(dnp no)
-		(property "Reference" "D4"
+		(property "Reference" "D?"
 			(at 40.64 82.296 0)
 			(show_name no)
@@
 		(instances
 			(project "PS-PrechargeBoard"
-				(path "/74d17fe6-68d4-4bd7-954a-e2bbb58b1f1e/c6e51092-efec-40a8-afae-63cae62691f2/9aee96ea-fe7f-4344-be59-bff28dc77cb5"
-					(reference "D4")
+				(path "/74d17fe6-68d4-4bd7-954a-e2bbb58b1f1e/1d9e626a-e7f8-4206-aa73-4d13edd0b32c"
+					(reference "D?")
 					(unit 1)
 				)
@@
 		(dnp no)
 		(fields_autoplaced yes)
-		(property "Reference" "C32"
+		(property "Reference" "C?"
 			(at 57.785 80.0099 0)
 			(show_name no)
@@
 		(instances
 			(project "PS-PrechargeBoard"
-				(path "/74d17fe6-68d4-4bd7-954a-e2bbb58b1f1e/c6e51092-efec-40a8-afae-63cae62691f2/9aee96ea-fe7f-4344-be59-bff28dc77cb5"
-					(reference "C32")
+				(path "/74d17fe6-68d4-4bd7-954a-e2bbb58b1f1e/1d9e626a-e7f8-4206-aa73-4d13edd0b32c"
+					(reference "C?")
 					(unit 1)
 				)
@@
 		(in_pos_files yes)
 		(dnp no)
-		(property "Reference" "D3"
+		(property "Reference" "D?"
 			(at 22.606 49.276 0)
 			(show_name no)
@@
 		(instances
 			(project "PS-PrechargeBoard"
-				(path "/74d17fe6-68d4-4bd7-954a-e2bbb58b1f1e/c6e51092-efec-40a8-afae-63cae62691f2/9aee96ea-fe7f-4344-be59-bff28dc77cb5"
-					(reference "D3")
+				(path "/74d17fe6-68d4-4bd7-954a-e2bbb58b1f1e/1d9e626a-e7f8-4206-aa73-4d13edd0b32c"
+					(reference "D?")
 					(unit 1)
 				)
@@
 		(dnp no)
 		(fields_autoplaced yes)
-		(property "Reference" "R26"
+		(property "Reference" "R?"
 			(at 45.72 60.9599 0)
 			(show_name no)
@@
 		(instances
 			(project "PS-PrechargeBoard"
-				(path "/74d17fe6-68d4-4bd7-954a-e2bbb58b1f1e/c6e51092-efec-40a8-afae-63cae62691f2/9aee96ea-fe7f-4344-be59-bff28dc77cb5"
-					(reference "R26")
+				(path "/74d17fe6-68d4-4bd7-954a-e2bbb58b1f1e/1d9e626a-e7f8-4206-aa73-4d13edd0b32c"
+					(reference "R?")
 					(unit 1)
 				)
@@
 		(in_pos_files yes)
 		(dnp no)
-		(property "Reference" "R31"
+		(property "Reference" "R?"
 			(at 137.668 90.17 90)
 			(show_name no)
@@
 		(instances
 			(project "PS-PrechargeBoard"
-				(path "/74d17fe6-68d4-4bd7-954a-e2bbb58b1f1e/c6e51092-efec-40a8-afae-63cae62691f2/9aee96ea-fe7f-4344-be59-bff28dc77cb5"
-					(reference "R31")
+				(path "/74d17fe6-68d4-4bd7-954a-e2bbb58b1f1e/1d9e626a-e7f8-4206-aa73-4d13edd0b32c"
+					(reference "R?")
 					(unit 1)
 				)
@@
 		(in_pos_files yes)
 		(dnp no)
-		(property "Reference" "C30"
+		(property "Reference" "C?"
 			(at 38.1 49.5299 0)
 			(show_name no)
@@
 		(instances
 			(project "PS-PrechargeBoard"
-				(path "/74d17fe6-68d4-4bd7-954a-e2bbb58b1f1e/c6e51092-efec-40a8-afae-63cae62691f2/9aee96ea-fe7f-4344-be59-bff28dc77cb5"
-					(reference "C30")
+				(path "/74d17fe6-68d4-4bd7-954a-e2bbb58b1f1e/1d9e626a-e7f8-4206-aa73-4d13edd0b32c"
+					(reference "C?")
 					(unit 1)
 				)
@@
 		(in_pos_files yes)
 		(dnp no)
-		(property "Reference" "R27"
+		(property "Reference" "R?"
 			(at 67.31 54.61 90)
 			(show_name no)
@@
 		(instances
 			(project "PS-PrechargeBoard"
-				(path "/74d17fe6-68d4-4bd7-954a-e2bbb58b1f1e/c6e51092-efec-40a8-afae-63cae62691f2/9aee96ea-fe7f-4344-be59-bff28dc77cb5"
-					(reference "R27")
+				(path "/74d17fe6-68d4-4bd7-954a-e2bbb58b1f1e/1d9e626a-e7f8-4206-aa73-4d13edd0b32c"
+					(reference "R?")
 					(unit 1)
 				)
@@
 		(in_pos_files yes)
 		(dnp no)
-		(property "Reference" "IC3"
+		(property "Reference" "IC?"
 			(at 75.184 73.66 0)
 			(show_name no)
@@
 		(instances
 			(project "PS-PrechargeBoard"
-				(path "/74d17fe6-68d4-4bd7-954a-e2bbb58b1f1e/c6e51092-efec-40a8-afae-63cae62691f2/9aee96ea-fe7f-4344-be59-bff28dc77cb5"
-					(reference "IC3")
+				(path "/74d17fe6-68d4-4bd7-954a-e2bbb58b1f1e/1d9e626a-e7f8-4206-aa73-4d13edd0b32c"
+					(reference "IC?")
 					(unit 1)
 				)
@@
 		(in_pos_files yes)
 		(dnp no)
-		(property "Reference" "Q1"
+		(property "Reference" "Q?"
 			(at 52.578 38.862 90)
 			(show_name no)
@@
 		(instances
 			(project "PS-PrechargeBoard"
-				(path "/74d17fe6-68d4-4bd7-954a-e2bbb58b1f1e/c6e51092-efec-40a8-afae-63cae62691f2/9aee96ea-fe7f-4344-be59-bff28dc77cb5"
-					(reference "Q1")
+				(path "/74d17fe6-68d4-4bd7-954a-e2bbb58b1f1e/1d9e626a-e7f8-4206-aa73-4d13edd0b32c"
+					(reference "Q?")
 					(unit 1)
 				)
@@
 		(in_pos_files yes)
 		(dnp no)
-		(property "Reference" "C35"
+		(property "Reference" "C?"
 			(at 113.284 89.154 0)
 			(show_name no)
@@
 		(instances
 			(project "PS-PrechargeBoard"
-				(path "/74d17fe6-68d4-4bd7-954a-e2bbb58b1f1e/c6e51092-efec-40a8-afae-63cae62691f2/9aee96ea-fe7f-4344-be59-bff28dc77cb5"
-					(reference "C35")
+				(path "/74d17fe6-68d4-4bd7-954a-e2bbb58b1f1e/1d9e626a-e7f8-4206-aa73-4d13edd0b32c"
+					(reference "C?")
 					(unit 1)
 				)
@@
 		(in_pos_files yes)
 		(dnp no)
-		(property "Reference" "C33"
+		(property "Reference" "C?"
 			(at 54.864 62.23 0)
 			(show_name no)
@@
 		(instances
 			(project "PS-PrechargeBoard"
-				(path "/74d17fe6-68d4-4bd7-954a-e2bbb58b1f1e/c6e51092-efec-40a8-afae-63cae62691f2/9aee96ea-fe7f-4344-be59-bff28dc77cb5"
-					(reference "C33")
+				(path "/74d17fe6-68d4-4bd7-954a-e2bbb58b1f1e/1d9e626a-e7f8-4206-aa73-4d13edd0b32c"
+					(reference "C?")
 					(unit 1)
 				)
@@
 		(in_pos_files yes)
 		(dnp no)
-		(property "Reference" "C34"
+		(property "Reference" "C?"
 			(at 112.395 49.5299 0)
 			(show_name no)
@@
 		(instances
 			(project "PS-PrechargeBoard"
-				(path "/74d17fe6-68d4-4bd7-954a-e2bbb58b1f1e/c6e51092-efec-40a8-afae-63cae62691f2/9aee96ea-fe7f-4344-be59-bff28dc77cb5"
-					(reference "C34")
+				(path "/74d17fe6-68d4-4bd7-954a-e2bbb58b1f1e/1d9e626a-e7f8-4206-aa73-4d13edd0b32c"
+					(reference "C?")
 					(unit 1)
 				)
@@
 		(in_pos_files yes)
 		(dnp no)
-		(property "Reference" "Q2"
+		(property "Reference" "Q?"
 			(at 100.584 38.608 90)
 			(show_name no)
@@
 		(instances
 			(project "PS-PrechargeBoard"
-				(path "/74d17fe6-68d4-4bd7-954a-e2bbb58b1f1e/c6e51092-efec-40a8-afae-63cae62691f2/9aee96ea-fe7f-4344-be59-bff28dc77cb5"
-					(reference "Q2")
+				(path "/74d17fe6-68d4-4bd7-954a-e2bbb58b1f1e/1d9e626a-e7f8-4206-aa73-4d13edd0b32c"
+					(reference "Q?")
 					(unit 1)
 				)
@@
 		(in_pos_files yes)
 		(dnp no)
-		(property "Reference" "R29"
+		(property "Reference" "R?"
 			(at 118.618 90.424 90)
 			(show_name no)
@@
 		(instances
 			(project "PS-PrechargeBoard"
-				(path "/74d17fe6-68d4-4bd7-954a-e2bbb58b1f1e/c6e51092-efec-40a8-afae-63cae62691f2/9aee96ea-fe7f-4344-be59-bff28dc77cb5"
-					(reference "R29")
+				(path "/74d17fe6-68d4-4bd7-954a-e2bbb58b1f1e/1d9e626a-e7f8-4206-aa73-4d13edd0b32c"
+					(reference "R?")
 					(unit 1)
 				)
@@
 		(in_pos_files yes)
 		(dnp no)
-		(property "Reference" "C31"
+		(property "Reference" "C?"
 			(at 31.75 82.5499 0)
 			(show_name no)
@@
 		(instances
 			(project "PS-PrechargeBoard"
-				(path "/74d17fe6-68d4-4bd7-954a-e2bbb58b1f1e/c6e51092-efec-40a8-afae-63cae62691f2/9aee96ea-fe7f-4344-be59-bff28dc77cb5"
-					(reference "C31")
+				(path "/74d17fe6-68d4-4bd7-954a-e2bbb58b1f1e/1d9e626a-e7f8-4206-aa73-4d13edd0b32c"
+					(reference "C?")
 					(unit 1)
 				)
@@
 		(in_pos_files yes)
 		(dnp no)
-		(property "Reference" "C36"
+		(property "Reference" "C?"
 			(at 132.08 88.9 0)
 			(show_name no)
@@
 		(instances
 			(project "PS-PrechargeBoard"
-				(path "/74d17fe6-68d4-4bd7-954a-e2bbb58b1f1e/c6e51092-efec-40a8-afae-63cae62691f2/9aee96ea-fe7f-4344-be59-bff28dc77cb5"
-					(reference "C36")
+				(path "/74d17fe6-68d4-4bd7-954a-e2bbb58b1f1e/1d9e626a-e7f8-4206-aa73-4d13edd0b32c"
+					(reference "C?")
 					(unit 1)
 				)
@@
 		(in_pos_files yes)
 		(dnp no)
-		(property "Reference" "R28"
+		(property "Reference" "R?"
 			(at 118.11 78.74 90)
 			(show_name no)
@@
 		(instances
 			(project "PS-PrechargeBoard"
-				(path "/74d17fe6-68d4-4bd7-954a-e2bbb58b1f1e/c6e51092-efec-40a8-afae-63cae62691f2/9aee96ea-fe7f-4344-be59-bff28dc77cb5"
-					(reference "R28")
+				(path "/74d17fe6-68d4-4bd7-954a-e2bbb58b1f1e/1d9e626a-e7f8-4206-aa73-4d13edd0b32c"
+					(reference "R?")
 					(unit 1)
 				)
@@
 		(in_pos_files yes)
 		(dnp no)
-		(property "Reference" "R30"
+		(property "Reference" "R?"
 			(at 137.16 77.47 90)
 			(show_name no)
@@
 		(instances
 			(project "PS-PrechargeBoard"
-				(path "/74d17fe6-68d4-4bd7-954a-e2bbb58b1f1e/c6e51092-efec-40a8-afae-63cae62691f2/9aee96ea-fe7f-4344-be59-bff28dc77cb5"
-					(reference "R30")
+				(path "/74d17fe6-68d4-4bd7-954a-e2bbb58b1f1e/1d9e626a-e7f8-4206-aa73-4d13edd0b32c"
+					(reference "R?")
 					(unit 1)
 				)

Commit message: final schematic REV-A?
Parts:
- gave numbers to parts that had none: 18
Changed lines of the file:
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@@
 		(in_pos_files yes)
 		(dnp no)
-		(property "Reference" "D?"
+		(property "Reference" "D12"
 			(at 40.64 82.296 0)
 			(show_name no)
@@
 		(instances
 			(project "PS-PrechargeBoard"
-				(path "/74d17fe6-68d4-4bd7-954a-e2bbb58b1f1e/1d9e626a-e7f8-4206-aa73-4d13edd0b32c"
-					(reference "D?")
+				(path "/74d17fe6-68d4-4bd7-954a-e2bbb58b1f1e/2ca150cf-fbe5-4d5b-a7dc-f2dc5c6024d0/f8c7dce2-42c7-4aa0-bec7-e504fb9f435f"
+					(reference "D12")
 					(unit 1)
 				)
@@
 		(dnp no)
 		(fields_autoplaced yes)
-		(property "Reference" "C?"
+		(property "Reference" "C41"
 			(at 57.785 80.0099 0)
 			(show_name no)
@@
 		(instances
 			(project "PS-PrechargeBoard"
-				(path "/74d17fe6-68d4-4bd7-954a-e2bbb58b1f1e/1d9e626a-e7f8-4206-aa73-4d13edd0b32c"
-					(reference "C?")
+				(path "/74d17fe6-68d4-4bd7-954a-e2bbb58b1f1e/2ca150cf-fbe5-4d5b-a7dc-f2dc5c6024d0/f8c7dce2-42c7-4aa0-bec7-e504fb9f435f"
+					(reference "C41")
 					(unit 1)
 				)
@@
 		(in_pos_files yes)
 		(dnp no)
-		(property "Reference" "D?"
+		(property "Reference" "D11"
 			(at 22.606 49.276 0)
 			(show_name no)
@@
 		(instances
 			(project "PS-PrechargeBoard"
-				(path "/74d17fe6-68d4-4bd7-954a-e2bbb58b1f1e/1d9e626a-e7f8-4206-aa73-4d13edd0b32c"
-					(reference "D?")
+				(path "/74d17fe6-68d4-4bd7-954a-e2bbb58b1f1e/2ca150cf-fbe5-4d5b-a7dc-f2dc5c6024d0/f8c7dce2-42c7-4aa0-bec7-e504fb9f435f"
+					(reference "D11")
 					(unit 1)
 				)
@@
 		(dnp no)
 		(fields_autoplaced yes)
-		(property "Reference" "R?"
+		(property "Reference" "R54"
 			(at 45.72 60.9599 0)
 			(show_name no)
@@
 		(instances
 			(project "PS-PrechargeBoard"
-				(path "/74d17fe6-68d4-4bd7-954a-e2bbb58b1f1e/1d9e626a-e7f8-4206-aa73-4d13edd0b32c"
-					(reference "R?")
+				(path "/74d17fe6-68d4-4bd7-954a-e2bbb58b1f1e/2ca150cf-fbe5-4d5b-a7dc-f2dc5c6024d0/f8c7dce2-42c7-4aa0-bec7-e504fb9f435f"
+					(reference "R54")
 					(unit 1)
 				)
@@
 		(in_pos_files yes)
 		(dnp no)
-		(property "Reference" "R?"
+		(property "Reference" "R59"
 			(at 137.668 90.17 90)
 			(show_name no)
@@
 		(instances
 			(project "PS-PrechargeBoard"
-				(path "/74d17fe6-68d4-4bd7-954a-e2bbb58b1f1e/1d9e626a-e7f8-4206-aa73-4d13edd0b32c"
-					(reference "R?")
+				(path "/74d17fe6-68d4-4bd7-954a-e2bbb58b1f1e/2ca150cf-fbe5-4d5b-a7dc-f2dc5c6024d0/f8c7dce2-42c7-4aa0-bec7-e504fb9f435f"
+					(reference "R59")
 					(unit 1)
 				)
@@
 		(in_pos_files yes)
 		(dnp no)
-		(property "Reference" "C?"
+		(property "Reference" "C39"
 			(at 38.1 49.5299 0)
 			(show_name no)
@@
 		(instances
 			(project "PS-PrechargeBoard"
-				(path "/74d17fe6-68d4-4bd7-954a-e2bbb58b1f1e/1d9e626a-e7f8-4206-aa73-4d13edd0b32c"
-					(reference "C?")
+				(path "/74d17fe6-68d4-4bd7-954a-e2bbb58b1f1e/2ca150cf-fbe5-4d5b-a7dc-f2dc5c6024d0/f8c7dce2-42c7-4aa0-bec7-e504fb9f435f"
+					(reference "C39")
 					(unit 1)
 				)
@@
 		(in_pos_files yes)
 		(dnp no)
-		(property "Reference" "R?"
+		(property "Reference" "R55"
 			(at 67.31 54.61 90)
 			(show_name no)
@@
 		(instances
 			(project "PS-PrechargeBoard"
-				(path "/74d17fe6-68d4-4bd7-954a-e2bbb58b1f1e/1d9e626a-e7f8-4206-aa73-4d13edd0b32c"
-					(reference "R?")
+				(path "/74d17fe6-68d4-4bd7-954a-e2bbb58b1f1e/2ca150cf-fbe5-4d5b-a7dc-f2dc5c6024d0/f8c7dce2-42c7-4aa0-bec7-e504fb9f435f"
+					(reference "R55")
 					(unit 1)
 				)
@@
 		(in_pos_files yes)
 		(dnp no)
-		(property "Reference" "IC?"
+		(property "Reference" "IC6"
 			(at 75.184 73.66 0)
 			(show_name no)
@@
 		(instances
 			(project "PS-PrechargeBoard"
-				(path "/74d17fe6-68d4-4bd7-954a-e2bbb58b1f1e/1d9e626a-e7f8-4206-aa73-4d13edd0b32c"
-					(reference "IC?")
+				(path "/74d17fe6-68d4-4bd7-954a-e2bbb58b1f1e/2ca150cf-fbe5-4d5b-a7dc-f2dc5c6024d0/f8c7dce2-42c7-4aa0-bec7-e504fb9f435f"
+					(reference "IC6")
 					(unit 1)
 				)
@@
 		(in_pos_files yes)
 		(dnp no)
-		(property "Reference" "Q?"
+		(property "Reference" "Q3"
 			(at 52.578 38.862 90)
 			(show_name no)
@@
 		(instances
 			(project "PS-PrechargeBoard"
-				(path "/74d17fe6-68d4-4bd7-954a-e2bbb58b1f1e/1d9e626a-e7f8-4206-aa73-4d13edd0b32c"
-					(reference "Q?")
+				(path "/74d17fe6-68d4-4bd7-954a-e2bbb58b1f1e/2ca150cf-fbe5-4d5b-a7dc-f2dc5c6024d0/f8c7dce2-42c7-4aa0-bec7-e504fb9f435f"
+					(reference "Q3")
 					(unit 1)
 				)
@@
 		(in_pos_files yes)
 		(dnp no)
-		(property "Reference" "C?"
+		(property "Reference" "C44"
 			(at 113.284 89.154 0)
 			(show_name no)
@@
 		(instances
 			(project "PS-PrechargeBoard"
-				(path "/74d17fe6-68d4-4bd7-954a-e2bbb58b1f1e/1d9e626a-e7f8-4206-aa73-4d13edd0b32c"
-					(reference "C?")
+				(path "/74d17fe6-68d4-4bd7-954a-e2bbb58b1f1e/2ca150cf-fbe5-4d5b-a7dc-f2dc5c6024d0/f8c7dce2-42c7-4aa0-bec7-e504fb9f435f"
+					(reference "C44")
 					(unit 1)
 				)
@@
 		(in_pos_files yes)
 		(dnp no)
-		(property "Reference" "C?"
+		(property "Reference" "C42"
 			(at 54.864 62.23 0)
 			(show_name no)
@@
 		(instances
 			(project "PS-PrechargeBoard"
-				(path "/74d17fe6-68d4-4bd7-954a-e2bbb58b1f1e/1d9e626a-e7f8-4206-aa73-4d13edd0b32c"
-					(reference "C?")
+				(path "/74d17fe6-68d4-4bd7-954a-e2bbb58b1f1e/2ca150cf-fbe5-4d5b-a7dc-f2dc5c6024d0/f8c7dce2-42c7-4aa0-bec7-e504fb9f435f"
+					(reference "C42")
 					(unit 1)
 				)
@@
 		(in_pos_files yes)
 		(dnp no)
-		(property "Reference" "C?"
+		(property "Reference" "C43"
 			(at 112.395 49.5299 0)
 			(show_name no)
@@
 		(instances
 			(project "PS-PrechargeBoard"
-				(path "/74d17fe6-68d4-4bd7-954a-e2bbb58b1f1e/1d9e626a-e7f8-4206-aa73-4d13edd0b32c"
-					(reference "C?")
+				(path "/74d17fe6-68d4-4bd7-954a-e2bbb58b1f1e/2ca150cf-fbe5-4d5b-a7dc-f2dc5c6024d0/f8c7dce2-42c7-4aa0-bec7-e504fb9f435f"
+					(reference "C43")
 					(unit 1)
 				)
@@
 		(in_pos_files yes)
 		(dnp no)
-		(property "Reference" "Q?"
+		(property "Reference" "Q4"
 			(at 100.584 38.608 90)
 			(show_name no)
@@
 		(instances
 			(project "PS-PrechargeBoard"
-				(path "/74d17fe6-68d4-4bd7-954a-e2bbb58b1f1e/1d9e626a-e7f8-4206-aa73-4d13edd0b32c"
-					(reference "Q?")
+				(path "/74d17fe6-68d4-4bd7-954a-e2bbb58b1f1e/2ca150cf-fbe5-4d5b-a7dc-f2dc5c6024d0/f8c7dce2-42c7-4aa0-bec7-e504fb9f435f"
+					(reference "Q4")
 					(unit 1)
 				)
@@
 		(in_pos_files yes)
 		(dnp no)
-		(property "Reference" "R?"
+		(property "Reference" "R57"
 			(at 118.618 90.424 90)
 			(show_name no)
@@
 		(instances
 			(project "PS-PrechargeBoard"
-				(path "/74d17fe6-68d4-4bd7-954a-e2bbb58b1f1e/1d9e626a-e7f8-4206-aa73-4d13edd0b32c"
-					(reference "R?")
+				(path "/74d17fe6-68d4-4bd7-954a-e2bbb58b1f1e/2ca150cf-fbe5-4d5b-a7dc-f2dc5c6024d0/f8c7dce2-42c7-4aa0-bec7-e504fb9f435f"
+					(reference "R57")
 					(unit 1)
 				)
@@
 		(in_pos_files yes)
 		(dnp no)
-		(property "Reference" "C?"
+		(property "Reference" "C40"
 			(at 31.75 82.5499 0)
 			(show_name no)
@@
 		(instances
 			(project "PS-PrechargeBoard"
-				(path "/74d17fe6-68d4-4bd7-954a-e2bbb58b1f1e/1d9e626a-e7f8-4206-aa73-4d13edd0b32c"
-					(reference "C?")
+				(path "/74d17fe6-68d4-4bd7-954a-e2bbb58b1f1e/2ca150cf-fbe5-4d5b-a7dc-f2dc5c6024d0/f8c7dce2-42c7-4aa0-bec7-e504fb9f435f"
+					(reference "C40")
 					(unit 1)
 				)
@@
 		(in_pos_files yes)
 		(dnp no)
-		(property "Reference" "C?"
+		(property "Reference" "C45"
 			(at 132.08 88.9 0)
 			(show_name no)
@@
 		(instances
 			(project "PS-PrechargeBoard"
-				(path "/74d17fe6-68d4-4bd7-954a-e2bbb58b1f1e/1d9e626a-e7f8-4206-aa73-4d13edd0b32c"
-					(reference "C?")
+				(path "/74d17fe6-68d4-4bd7-954a-e2bbb58b1f1e/2ca150cf-fbe5-4d5b-a7dc-f2dc5c6024d0/f8c7dce2-42c7-4aa0-bec7-e504fb9f435f"
+					(reference "C45")
 					(unit 1)
 				)
@@
 		(in_pos_files yes)
 		(dnp no)
-		(property "Reference" "R?"
+		(property "Reference" "R56"
 			(at 118.11 78.74 90)
 			(show_name no)
@@
 		(instances
 			(project "PS-PrechargeBoard"
-				(path "/74d17fe6-68d4-4bd7-954a-e2bbb58b1f1e/1d9e626a-e7f8-4206-aa73-4d13edd0b32c"
-					(reference "R?")
+				(path "/74d17fe6-68d4-4bd7-954a-e2bbb58b1f1e/2ca150cf-fbe5-4d5b-a7dc-f2dc5c6024d0/f8c7dce2-42c7-4aa0-bec7-e504fb9f435f"
+					(reference "R56")
 					(unit 1)
 				)
@@
 		(in_pos_files yes)
 		(dnp no)
-		(property "Reference" "R?"
+		(property "Reference" "R58"
 			(at 137.16 77.47 90)
 			(show_name no)
@@
 		(instances
 			(project "PS-PrechargeBoard"
-				(path "/74d17fe6-68d4-4bd7-954a-e2bbb58b1f1e/1d9e626a-e7f8-4206-aa73-4d13edd0b32c"
-					(reference "R?")
+				(path "/74d17fe6-68d4-4bd7-954a-e2bbb58b1f1e/2ca150cf-fbe5-4d5b-a7dc-f2dc5c6024d0/f8c7dce2-42c7-4aa0-bec7-e504fb9f435f"
+					(reference "R58")
 					(unit 1)
 				)
