File: PowerProtection.kicad_sch (KiCad schematic)
At the start: 18 parts, among them IC1 LM74502DDFR, Q3 PSMN012-100YS, Q4 PSMN012-100YS

Commit message: restored pp placement
Other:
- title: Power Protection -> (none)
Changed lines of the file:
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@@
 	(generator "eeschema")
 	(generator_version "10.0")
-	(paper "A5")
-	(title_block
-		(title "Power Protection")
-	)
+	(paper "A4")
 	(text "4.84ms = 75us + 220nF * 6.5V/300uA\n6.5V recommended on datasheet\n4.84ms power up delay"
 		(exclude_from_sim no)
