File: Power_Mux.kicad_sch (KiCad schematic)
At the start: 6 parts, among them U1 TPS2117DRLR

Commit message: lv 1.2
Parts:
- renumbered C1 to C14, C2 to C15, C3 to C16, C4 to C17, R1 to R11, U1 to U2
Changed lines of the file:
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@@
 		(in_pos_files yes)
 		(dnp no)
-		(property "Reference" "C4"
+		(property "Reference" "C17"
 			(at 91.8972 57.2516 0)
 			(show_name no)
@@
 			(project "PS-PrechargeBoard"
 				(path "/74d17fe6-68d4-4bd7-954a-e2bbb58b1f1e/6c9f9146-fe47-479e-b844-c090447a528f"
-					(reference "C4")
+					(reference "C17")
 					(unit 1)
 				)
@@
 		(in_pos_files yes)
 		(dnp no)
-		(property "Reference" "R1"
+		(property "Reference" "R11"
 			(at 78.994 67.564 0)
 			(show_name no)
@@
 			(project "PS-PrechargeBoard"
 				(path "/74d17fe6-68d4-4bd7-954a-e2bbb58b1f1e/6c9f9146-fe47-479e-b844-c090447a528f"
-					(reference "R1")
+					(reference "R11")
 					(unit 1)
 				)
@@
 		(in_pos_files yes)
 		(dnp no)
-		(property "Reference" "C1"
+		(property "Reference" "C14"
 			(at 24.5872 44.5516 0)
 			(show_name no)
@@
 			(project "PS-PrechargeBoard"
 				(path "/74d17fe6-68d4-4bd7-954a-e2bbb58b1f1e/6c9f9146-fe47-479e-b844-c090447a528f"
-					(reference "C1")
+					(reference "C14")
 					(unit 1)
 				)
@@
 		(dnp no)
 		(fields_autoplaced yes)
-		(property "Reference" "U1"
+		(property "Reference" "U2"
 			(at 60.96 44.45 0)
 			(show_name no)
@@
 			(project "PS-PrechargeBoard"
 				(path "/74d17fe6-68d4-4bd7-954a-e2bbb58b1f1e/6c9f9146-fe47-479e-b844-c090447a528f"
-					(reference "U1")
+					(reference "U2")
 					(unit 1)
 				)
@@
 		(in_pos_files yes)
 		(dnp no)
-		(property "Reference" "C3"
+		(property "Reference" "C16"
 			(at 42.3672 67.4116 0)
 			(show_name no)
@@
 			(project "PS-PrechargeBoard"
 				(path "/74d17fe6-68d4-4bd7-954a-e2bbb58b1f1e/6c9f9146-fe47-479e-b844-c090447a528f"
-					(reference "C3")
+					(reference "C16")
 					(unit 1)
 				)
@@
 		(in_pos_files yes)
 		(dnp no)
-		(property "Reference" "C2"
+		(property "Reference" "C15"
 			(at 38.5572 44.5516 0)
 			(show_name no)
@@
 			(project "PS-PrechargeBoard"
 				(path "/74d17fe6-68d4-4bd7-954a-e2bbb58b1f1e/6c9f9146-fe47-479e-b844-c090447a528f"
-					(reference "C2")
-					(unit 1)
-				)
+					(reference "C15")
+					(unit 1)
+				)

Commit message: hv 1.0
Parts:
- renumbered R11 to R15
Changed lines of the file:
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@@
 		(in_pos_files yes)
 		(dnp no)
-		(property "Reference" "R11"
+		(property "Reference" "R15"
 			(at 78.994 67.564 0)
 			(show_name no)
@@
 			(project "PS-PrechargeBoard"
 				(path "/74d17fe6-68d4-4bd7-954a-e2bbb58b1f1e/6c9f9146-fe47-479e-b844-c090447a528f"
-					(reference "R11")
+					(reference "R15")
 					(unit 1)
 				)

Commit message: hv 1.1
Parts:
- renumbered R15 to R14
Changed lines of the file:
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@@
 		(in_pos_files yes)
 		(dnp no)
-		(property "Reference" "R15"
+		(property "Reference" "R14"
 			(at 78.994 67.564 0)
 			(show_name no)
@@
 			(project "PS-PrechargeBoard"
 				(path "/74d17fe6-68d4-4bd7-954a-e2bbb58b1f1e/6c9f9146-fe47-479e-b844-c090447a528f"
-					(reference "R15")
+					(reference "R14")
 					(unit 1)
 				)

Commit message: hv 1.3
Parts:
- renumbered C17 to C?, C14 to C?, C16 to C?, C15 to C?, R14 to R?, U2 to U?
Changed lines of the file:
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@@
 		(in_pos_files yes)
 		(dnp no)
-		(property "Reference" "C17"
+		(property "Reference" "C?"
 			(at 91.8972 57.2516 0)
 			(show_name no)
@@
 		(instances
 			(project "PS-PrechargeBoard"
-				(path "/74d17fe6-68d4-4bd7-954a-e2bbb58b1f1e/6c9f9146-fe47-479e-b844-c090447a528f"
-					(reference "C17")
-					(unit 1)
-				)
-			)
-			(project "power-mux-block"
-				(path "/c8207045-8aef-4538-bcc4-1e380c549c2c"
-					(reference "C4")
+				(path "/11743897-1544-4e3c-979c-dcc54ac7093b/47a0820e-ddb4-4652-9c69-8d106132f60e"
+					(reference "C?")
 					(unit 1)
 				)
@@
 		(in_pos_files yes)
 		(dnp no)
-		(property "Reference" "R14"
+		(property "Reference" "R?"
 			(at 78.994 67.564 0)
 			(show_name no)
@@
 		(instances
 			(project "PS-PrechargeBoard"
-				(path "/74d17fe6-68d4-4bd7-954a-e2bbb58b1f1e/6c9f9146-fe47-479e-b844-c090447a528f"
-					(reference "R14")
-					(unit 1)
-				)
-			)
-			(project "power-mux-block"
-				(path "/c8207045-8aef-4538-bcc4-1e380c549c2c"
-					(reference "R1")
+				(path "/11743897-1544-4e3c-979c-dcc54ac7093b/47a0820e-ddb4-4652-9c69-8d106132f60e"
+					(reference "R?")
 					(unit 1)
 				)
@@
 		(in_pos_files yes)
 		(dnp no)
-		(property "Reference" "C14"
+		(property "Reference" "C?"
 			(at 24.5872 44.5516 0)
 			(show_name no)
@@
 		(instances
 			(project "PS-PrechargeBoard"
-				(path "/74d17fe6-68d4-4bd7-954a-e2bbb58b1f1e/6c9f9146-fe47-479e-b844-c090447a528f"
-					(reference "C14")
-					(unit 1)
-				)
-			)
-			(project "power-mux-block"
-				(path "/c8207045-8aef-4538-bcc4-1e380c549c2c"
-					(reference "C1")
+				(path "/11743897-1544-4e3c-979c-dcc54ac7093b/47a0820e-ddb4-4652-9c69-8d106132f60e"
+					(reference "C?")
 					(unit 1)
 				)
@@
 		(dnp no)
 		(fields_autoplaced yes)
-		(property "Reference" "U2"
+		(property "Reference" "U?"
 			(at 60.96 44.45 0)
 			(show_name no)
@@
 		(instances
 			(project "PS-PrechargeBoard"
-				(path "/74d17fe6-68d4-4bd7-954a-e2bbb58b1f1e/6c9f9146-fe47-479e-b844-c090447a528f"
-					(reference "U2")
-					(unit 1)
-				)
-			)
-			(project ""
-				(path "/c8207045-8aef-4538-bcc4-1e380c549c2c"
-					(reference "U1")
+				(path "/11743897-1544-4e3c-979c-dcc54ac7093b/47a0820e-ddb4-4652-9c69-8d106132f60e"
+					(reference "U?")
 					(unit 1)
 				)
@@
 		(in_pos_files yes)
 		(dnp no)
-		(property "Reference" "C16"
+		(property "Reference" "C?"
 			(at 42.3672 67.4116 0)
 			(show_name no)
@@
 		(instances
 			(project "PS-PrechargeBoard"
-				(path "/74d17fe6-68d4-4bd7-954a-e2bbb58b1f1e/6c9f9146-fe47-479e-b844-c090447a528f"
-					(reference "C16")
-					(unit 1)
-				)
-			)
-			(project "power-mux-block"
-				(path "/c8207045-8aef-4538-bcc4-1e380c549c2c"
-					(reference "C3")
+				(path "/11743897-1544-4e3c-979c-dcc54ac7093b/47a0820e-ddb4-4652-9c69-8d106132f60e"
+					(reference "C?")
 					(unit 1)
 				)
@@
 		(in_pos_files yes)
 		(dnp no)
-		(property "Reference" "C15"
+		(property "Reference" "C?"
 			(at 38.5572 44.5516 0)
 			(show_name no)
@@
 		(instances
 			(project "PS-PrechargeBoard"
-				(path "/74d17fe6-68d4-4bd7-954a-e2bbb58b1f1e/6c9f9146-fe47-479e-b844-c090447a528f"
-					(reference "C15")
+				(path "/11743897-1544-4e3c-979c-dcc54ac7093b/47a0820e-ddb4-4652-9c69-8d106132f60e"
+					(reference "C?")
 					(unit 1)
 				)
-			)
-			(project "power-mux-block"
-				(path "/c8207045-8aef-4538-bcc4-1e380c549c2c"
-					(reference "C2")
-					(unit 1)
-				)
