File: Power_Mux.kicad_sch (KiCad schematic)
At the start: 6 parts

Commit message: CAN nano & CAN debug nano
Parts:
- gave numbers to parts that had none: 6
Changed lines of the file:
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@@
 		(in_pos_files yes)
 		(dnp no)
-		(property "Reference" "C?"
+		(property "Reference" "C37"
 			(at 91.8972 57.2516 0)
 			(show_name no)
@@
 			(project "PS-PrechargeBoard"
 				(path "/74d17fe6-68d4-4bd7-954a-e2bbb58b1f1e/0def18ef-81e8-47ac-b719-2d9f8237a855/47a0820e-ddb4-4652-9c69-8d106132f60e"
-					(reference "C?")
+					(reference "C37")
 					(unit 1)
 				)
@@
 			(project "lv"
 				(path "/88356d12-c87f-4bdd-bbd8-756414c90a6d/47a0820e-ddb4-4652-9c69-8d106132f60e"
-					(reference "C?")
-					(unit 1)
-				)
-			)
-			(project "PS-PrechargeBoard"
-				(path "/9641192f-df6c-4894-9070-848e3256daf8/47a0820e-ddb4-4652-9c69-8d106132f60e"
 					(reference "C?")
 					(unit 1)
@@
 		(in_pos_files yes)
 		(dnp no)
-		(property "Reference" "R?"
+		(property "Reference" "R21"
 			(at 78.994 67.564 0)
 			(show_name no)
@@
 			(project "PS-PrechargeBoard"
 				(path "/74d17fe6-68d4-4bd7-954a-e2bbb58b1f1e/0def18ef-81e8-47ac-b719-2d9f8237a855/47a0820e-ddb4-4652-9c69-8d106132f60e"
-					(reference "R?")
+					(reference "R21")
 					(unit 1)
 				)
@@
 			(project "lv"
 				(path "/88356d12-c87f-4bdd-bbd8-756414c90a6d/47a0820e-ddb4-4652-9c69-8d106132f60e"
-					(reference "R?")
-					(unit 1)
-				)
-			)
-			(project "PS-PrechargeBoard"
-				(path "/9641192f-df6c-4894-9070-848e3256daf8/47a0820e-ddb4-4652-9c69-8d106132f60e"
 					(reference "R?")
 					(unit 1)
@@
 		(in_pos_files yes)
 		(dnp no)
-		(property "Reference" "C?"
+		(property "Reference" "C34"
 			(at 24.5872 44.5516 0)
 			(show_name no)
@@
 			(project "PS-PrechargeBoard"
 				(path "/74d17fe6-68d4-4bd7-954a-e2bbb58b1f1e/0def18ef-81e8-47ac-b719-2d9f8237a855/47a0820e-ddb4-4652-9c69-8d106132f60e"
-					(reference "C?")
+					(reference "C34")
 					(unit 1)
 				)
@@
 			(project "lv"
 				(path "/88356d12-c87f-4bdd-bbd8-756414c90a6d/47a0820e-ddb4-4652-9c69-8d106132f60e"
-					(reference "C?")
-					(unit 1)
-				)
-			)
-			(project "PS-PrechargeBoard"
-				(path "/9641192f-df6c-4894-9070-848e3256daf8/47a0820e-ddb4-4652-9c69-8d106132f60e"
 					(reference "C?")
 					(unit 1)
@@
 		(dnp no)
 		(fields_autoplaced yes)
-		(property "Reference" "U?"
+		(property "Reference" "U3"
 			(at 60.96 44.45 0)
 			(show_name no)
@@
 			(project "PS-PrechargeBoard"
 				(path "/74d17fe6-68d4-4bd7-954a-e2bbb58b1f1e/0def18ef-81e8-47ac-b719-2d9f8237a855/47a0820e-ddb4-4652-9c69-8d106132f60e"
-					(reference "U?")
+					(reference "U3")
 					(unit 1)
 				)
@@
 			(project "lv"
 				(path "/88356d12-c87f-4bdd-bbd8-756414c90a6d/47a0820e-ddb4-4652-9c69-8d106132f60e"
-					(reference "U?")
-					(unit 1)
-				)
-			)
-			(project "PS-PrechargeBoard"
-				(path "/9641192f-df6c-4894-9070-848e3256daf8/47a0820e-ddb4-4652-9c69-8d106132f60e"
 					(reference "U?")
 					(unit 1)
@@
 		(in_pos_files yes)
 		(dnp no)
-		(property "Reference" "C?"
+		(property "Reference" "C36"
 			(at 42.3672 67.4116 0)
 			(show_name no)
@@
 			(project "PS-PrechargeBoard"
 				(path "/74d17fe6-68d4-4bd7-954a-e2bbb58b1f1e/0def18ef-81e8-47ac-b719-2d9f8237a855/47a0820e-ddb4-4652-9c69-8d106132f60e"
-					(reference "C?")
+					(reference "C36")
 					(unit 1)
 				)
@@
 			(project "lv"
 				(path "/88356d12-c87f-4bdd-bbd8-756414c90a6d/47a0820e-ddb4-4652-9c69-8d106132f60e"
-					(reference "C?")
-					(unit 1)
-				)
-			)
-			(project "PS-PrechargeBoard"
-				(path "/9641192f-df6c-4894-9070-848e3256daf8/47a0820e-ddb4-4652-9c69-8d106132f60e"
 					(reference "C?")
 					(unit 1)
@@
 		(in_pos_files yes)
 		(dnp no)
-		(property "Reference" "C?"
+		(property "Reference" "C35"
 			(at 38.5572 44.5516 0)
 			(show_name no)
@@
 			(project "PS-PrechargeBoard"
 				(path "/74d17fe6-68d4-4bd7-954a-e2bbb58b1f1e/0def18ef-81e8-47ac-b719-2d9f8237a855/47a0820e-ddb4-4652-9c69-8d106132f60e"
-					(reference "C?")
+					(reference "C35")
 					(unit 1)
 				)
@@
 					(reference "C?")
 					(unit 1)
-				)
-			)
-			(project "PS-PrechargeBoard"
-				(path "/9641192f-df6c-4894-9070-848e3256daf8/47a0820e-ddb4-4652-9c69-8d106132f60e"
-					(reference "C?")
-					(unit 1)

Commit message: battery voltage & motor voltage
Parts:
- renumbered C34 to C22, C35 to C23, C36 to C24, C37 to C25, R21 to R25, U3 to U5
Changed lines of the file:
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@@
 		(in_pos_files yes)
 		(dnp no)
-		(property "Reference" "C37"
+		(property "Reference" "C25"
 			(at 91.8972 57.2516 0)
 			(show_name no)
@@
 			(project "PS-PrechargeBoard"
 				(path "/74d17fe6-68d4-4bd7-954a-e2bbb58b1f1e/0def18ef-81e8-47ac-b719-2d9f8237a855/47a0820e-ddb4-4652-9c69-8d106132f60e"
-					(reference "C37")
+					(reference "C25")
 					(unit 1)
 				)
@@
 		(in_pos_files yes)
 		(dnp no)
-		(property "Reference" "R21"
+		(property "Reference" "R25"
 			(at 78.994 67.564 0)
 			(show_name no)
@@
 			(project "PS-PrechargeBoard"
 				(path "/74d17fe6-68d4-4bd7-954a-e2bbb58b1f1e/0def18ef-81e8-47ac-b719-2d9f8237a855/47a0820e-ddb4-4652-9c69-8d106132f60e"
-					(reference "R21")
+					(reference "R25")
 					(unit 1)
 				)
@@
 		(in_pos_files yes)
 		(dnp no)
-		(property "Reference" "C34"
+		(property "Reference" "C22"
 			(at 24.5872 44.5516 0)
 			(show_name no)
@@
 			(project "PS-PrechargeBoard"
 				(path "/74d17fe6-68d4-4bd7-954a-e2bbb58b1f1e/0def18ef-81e8-47ac-b719-2d9f8237a855/47a0820e-ddb4-4652-9c69-8d106132f60e"
-					(reference "C34")
+					(reference "C22")
 					(unit 1)
 				)
@@
 		(dnp no)
 		(fields_autoplaced yes)
-		(property "Reference" "U3"
+		(property "Reference" "U5"
 			(at 60.96 44.45 0)
 			(show_name no)
@@
 			(project "PS-PrechargeBoard"
 				(path "/74d17fe6-68d4-4bd7-954a-e2bbb58b1f1e/0def18ef-81e8-47ac-b719-2d9f8237a855/47a0820e-ddb4-4652-9c69-8d106132f60e"
-					(reference "U3")
+					(reference "U5")
 					(unit 1)
 				)
@@
 		(in_pos_files yes)
 		(dnp no)
-		(property "Reference" "C36"
+		(property "Reference" "C24"
 			(at 42.3672 67.4116 0)
 			(show_name no)
@@
 			(project "PS-PrechargeBoard"
 				(path "/74d17fe6-68d4-4bd7-954a-e2bbb58b1f1e/0def18ef-81e8-47ac-b719-2d9f8237a855/47a0820e-ddb4-4652-9c69-8d106132f60e"
-					(reference "C36")
+					(reference "C24")
 					(unit 1)
 				)
@@
 		(in_pos_files yes)
 		(dnp no)
-		(property "Reference" "C35"
+		(property "Reference" "C23"
 			(at 38.5572 44.5516 0)
 			(show_name no)
@@
 			(project "PS-PrechargeBoard"
 				(path "/74d17fe6-68d4-4bd7-954a-e2bbb58b1f1e/0def18ef-81e8-47ac-b719-2d9f8237a855/47a0820e-ddb4-4652-9c69-8d106132f60e"
-					(reference "C35")
-					(unit 1)
-				)
+					(reference "C23")
+					(unit 1)
+				)

Commit message: fixed battery voltage & motor voltage
Parts:
- U5: now not fitted
Changed lines of the file:
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@@
 		(on_board yes)
 		(in_pos_files yes)
-		(dnp no)
+		(dnp yes)
 		(fields_autoplaced yes)
 		(property "Reference" "U5"

Commit message: shifted hierarchical sheets
Parts:
- renumbered C25 to C?, C22 to C?, C24 to C?, C23 to C?, R25 to R?, U5 to U?
Changed lines of the file:
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@@
 		(in_pos_files yes)
 		(dnp no)
-		(property "Reference" "C25"
+		(property "Reference" "C?"
 			(at 91.8972 57.2516 0)
 			(show_name no)
@@
 		(instances
 			(project "PS-PrechargeBoard"
-				(path "/74d17fe6-68d4-4bd7-954a-e2bbb58b1f1e/0def18ef-81e8-47ac-b719-2d9f8237a855/47a0820e-ddb4-4652-9c69-8d106132f60e"
-					(reference "C25")
-					(unit 1)
-				)
-			)
-			(project "lv"
-				(path "/88356d12-c87f-4bdd-bbd8-756414c90a6d/47a0820e-ddb4-4652-9c69-8d106132f60e"
+				(path "/74d17fe6-68d4-4bd7-954a-e2bbb58b1f1e/5e9f1eea-2df2-42e3-8b3e-de31498eaece"
 					(reference "C?")
 					(unit 1)
@@
 		(in_pos_files yes)
 		(dnp no)
-		(property "Reference" "R25"
+		(property "Reference" "R?"
 			(at 78.994 67.564 0)
 			(show_name no)
@@
 		(instances
 			(project "PS-PrechargeBoard"
-				(path "/74d17fe6-68d4-4bd7-954a-e2bbb58b1f1e/0def18ef-81e8-47ac-b719-2d9f8237a855/47a0820e-ddb4-4652-9c69-8d106132f60e"
-					(reference "R25")
-					(unit 1)
-				)
-			)
-			(project "lv"
-				(path "/88356d12-c87f-4bdd-bbd8-756414c90a6d/47a0820e-ddb4-4652-9c69-8d106132f60e"
+				(path "/74d17fe6-68d4-4bd7-954a-e2bbb58b1f1e/5e9f1eea-2df2-42e3-8b3e-de31498eaece"
 					(reference "R?")
 					(unit 1)
@@
 		(in_pos_files yes)
 		(dnp no)
-		(property "Reference" "C22"
+		(property "Reference" "C?"
 			(at 24.5872 44.5516 0)
 			(show_name no)
@@
 		(instances
 			(project "PS-PrechargeBoard"
-				(path "/74d17fe6-68d4-4bd7-954a-e2bbb58b1f1e/0def18ef-81e8-47ac-b719-2d9f8237a855/47a0820e-ddb4-4652-9c69-8d106132f60e"
-					(reference "C22")
-					(unit 1)
-				)
-			)
-			(project "lv"
-				(path "/88356d12-c87f-4bdd-bbd8-756414c90a6d/47a0820e-ddb4-4652-9c69-8d106132f60e"
+				(path "/74d17fe6-68d4-4bd7-954a-e2bbb58b1f1e/5e9f1eea-2df2-42e3-8b3e-de31498eaece"
 					(reference "C?")
 					(unit 1)
@@
 		(dnp yes)
 		(fields_autoplaced yes)
-		(property "Reference" "U5"
+		(property "Reference" "U?"
 			(at 60.96 44.45 0)
 			(show_name no)
@@
 		(instances
 			(project "PS-PrechargeBoard"
-				(path "/74d17fe6-68d4-4bd7-954a-e2bbb58b1f1e/0def18ef-81e8-47ac-b719-2d9f8237a855/47a0820e-ddb4-4652-9c69-8d106132f60e"
-					(reference "U5")
-					(unit 1)
-				)
-			)
-			(project "lv"
-				(path "/88356d12-c87f-4bdd-bbd8-756414c90a6d/47a0820e-ddb4-4652-9c69-8d106132f60e"
+				(path "/74d17fe6-68d4-4bd7-954a-e2bbb58b1f1e/5e9f1eea-2df2-42e3-8b3e-de31498eaece"
 					(reference "U?")
 					(unit 1)
@@
 		(in_pos_files yes)
 		(dnp no)
-		(property "Reference" "C24"
+		(property "Reference" "C?"
 			(at 42.3672 67.4116 0)
 			(show_name no)
@@
 		(instances
 			(project "PS-PrechargeBoard"
-				(path "/74d17fe6-68d4-4bd7-954a-e2bbb58b1f1e/0def18ef-81e8-47ac-b719-2d9f8237a855/47a0820e-ddb4-4652-9c69-8d106132f60e"
-					(reference "C24")
-					(unit 1)
-				)
-			)
-			(project "lv"
-				(path "/88356d12-c87f-4bdd-bbd8-756414c90a6d/47a0820e-ddb4-4652-9c69-8d106132f60e"
+				(path "/74d17fe6-68d4-4bd7-954a-e2bbb58b1f1e/5e9f1eea-2df2-42e3-8b3e-de31498eaece"
 					(reference "C?")
 					(unit 1)
@@
 		(in_pos_files yes)
 		(dnp no)
-		(property "Reference" "C23"
+		(property "Reference" "C?"
 			(at 38.5572 44.5516 0)
 			(show_name no)
@@
 		(instances
 			(project "PS-PrechargeBoard"
-				(path "/74d17fe6-68d4-4bd7-954a-e2bbb58b1f1e/0def18ef-81e8-47ac-b719-2d9f8237a855/47a0820e-ddb4-4652-9c69-8d106132f60e"
-					(reference "C23")
-					(unit 1)
-				)
-			)
-			(project "lv"
-				(path "/88356d12-c87f-4bdd-bbd8-756414c90a6d/47a0820e-ddb4-4652-9c69-8d106132f60e"
+				(path "/74d17fe6-68d4-4bd7-954a-e2bbb58b1f1e/5e9f1eea-2df2-42e3-8b3e-de31498eaece"
 					(reference "C?")
 					(unit 1)

Commit message: V_OUT_BAT & V_OUT_MOT & PRECHARGE_CTRL to MCU
Parts:
- gave numbers to parts that had none: 6
Changed lines of the file:
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@@
 		(in_pos_files yes)
 		(dnp no)
-		(property "Reference" "C?"
+		(property "Reference" "C59"
 			(at 91.8972 57.2516 0)
 			(show_name no)
@@
 			(project "PS-PrechargeBoard"
 				(path "/74d17fe6-68d4-4bd7-954a-e2bbb58b1f1e/5e9f1eea-2df2-42e3-8b3e-de31498eaece"
-					(reference "C?")
+					(reference "C59")
 					(unit 1)
 				)
@@
 		(in_pos_files yes)
 		(dnp no)
-		(property "Reference" "R?"
+		(property "Reference" "R47"
 			(at 78.994 67.564 0)
 			(show_name no)
@@
 			(project "PS-PrechargeBoard"
 				(path "/74d17fe6-68d4-4bd7-954a-e2bbb58b1f1e/5e9f1eea-2df2-42e3-8b3e-de31498eaece"
-					(reference "R?")
+					(reference "R47")
 					(unit 1)
 				)
@@
 		(in_pos_files yes)
 		(dnp no)
-		(property "Reference" "C?"
+		(property "Reference" "C56"
 			(at 24.5872 44.5516 0)
 			(show_name no)
@@
 			(project "PS-PrechargeBoard"
 				(path "/74d17fe6-68d4-4bd7-954a-e2bbb58b1f1e/5e9f1eea-2df2-42e3-8b3e-de31498eaece"
-					(reference "C?")
+					(reference "C56")
 					(unit 1)
 				)
@@
 		(dnp yes)
 		(fields_autoplaced yes)
-		(property "Reference" "U?"
+		(property "Reference" "U7"
 			(at 60.96 44.45 0)
 			(show_name no)
@@
 			(project "PS-PrechargeBoard"
 				(path "/74d17fe6-68d4-4bd7-954a-e2bbb58b1f1e/5e9f1eea-2df2-42e3-8b3e-de31498eaece"
-					(reference "U?")
+					(reference "U7")
 					(unit 1)
 				)
@@
 		(in_pos_files yes)
 		(dnp no)
-		(property "Reference" "C?"
+		(property "Reference" "C58"
 			(at 42.3672 67.4116 0)
 			(show_name no)
@@
 			(project "PS-PrechargeBoard"
 				(path "/74d17fe6-68d4-4bd7-954a-e2bbb58b1f1e/5e9f1eea-2df2-42e3-8b3e-de31498eaece"
-					(reference "C?")
+					(reference "C58")
 					(unit 1)
 				)
@@
 		(in_pos_files yes)
 		(dnp no)
-		(property "Reference" "C?"
+		(property "Reference" "C57"
 			(at 38.5572 44.5516 0)
 			(show_name no)
@@
 			(project "PS-PrechargeBoard"
 				(path "/74d17fe6-68d4-4bd7-954a-e2bbb58b1f1e/5e9f1eea-2df2-42e3-8b3e-de31498eaece"
-					(reference "C?")
+					(reference "C57")
 					(unit 1)
 				)

Commit message: precharges & voltage sensors
Parts:
- renumbered C56 to C37, C57 to C38, C58 to C39, C59 to C40, R47 to R32
Changed lines of the file:
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@@
 		(in_pos_files yes)
 		(dnp no)
-		(property "Reference" "C59"
+		(property "Reference" "C40"
 			(at 91.8972 57.2516 0)
 			(show_name no)
@@
 		(instances
 			(project "PS-PrechargeBoard"
-				(path "/74d17fe6-68d4-4bd7-954a-e2bbb58b1f1e/5e9f1eea-2df2-42e3-8b3e-de31498eaece"
-					(reference "C59")
+				(path "/74d17fe6-68d4-4bd7-954a-e2bbb58b1f1e/c6e51092-efec-40a8-afae-63cae62691f2/c3c1aad2-e774-4d45-973c-7509c3ed46d5"
+					(reference "C40")
 					(unit 1)
 				)
@@
 		(in_pos_files yes)
 		(dnp no)
-		(property "Reference" "R47"
+		(property "Reference" "R32"
 			(at 78.994 67.564 0)
 			(show_name no)
@@
 		(instances
 			(project "PS-PrechargeBoard"
-				(path "/74d17fe6-68d4-4bd7-954a-e2bbb58b1f1e/5e9f1eea-2df2-42e3-8b3e-de31498eaece"
-					(reference "R47")
+				(path "/74d17fe6-68d4-4bd7-954a-e2bbb58b1f1e/c6e51092-efec-40a8-afae-63cae62691f2/c3c1aad2-e774-4d45-973c-7509c3ed46d5"
+					(reference "R32")
 					(unit 1)
 				)
@@
 		(in_pos_files yes)
 		(dnp no)
-		(property "Reference" "C56"
+		(property "Reference" "C37"
 			(at 24.5872 44.5516 0)
 			(show_name no)
@@
 		(instances
 			(project "PS-PrechargeBoard"
-				(path "/74d17fe6-68d4-4bd7-954a-e2bbb58b1f1e/5e9f1eea-2df2-42e3-8b3e-de31498eaece"
-					(reference "C56")
+				(path "/74d17fe6-68d4-4bd7-954a-e2bbb58b1f1e/c6e51092-efec-40a8-afae-63cae62691f2/c3c1aad2-e774-4d45-973c-7509c3ed46d5"
+					(reference "C37")
 					(unit 1)
 				)
@@
 		(instances
 			(project "PS-PrechargeBoard"
-				(path "/74d17fe6-68d4-4bd7-954a-e2bbb58b1f1e/5e9f1eea-2df2-42e3-8b3e-de31498eaece"
+				(path "/74d17fe6-68d4-4bd7-954a-e2bbb58b1f1e/c6e51092-efec-40a8-afae-63cae62691f2/c3c1aad2-e774-4d45-973c-7509c3ed46d5"
 					(reference "U7")
 					(unit 1)
@@
 		(in_pos_files yes)
 		(dnp no)
-		(property "Reference" "C58"
+		(property "Reference" "C39"
 			(at 42.3672 67.4116 0)
 			(show_name no)
@@
 		(instances
 			(project "PS-PrechargeBoard"
-				(path "/74d17fe6-68d4-4bd7-954a-e2bbb58b1f1e/5e9f1eea-2df2-42e3-8b3e-de31498eaece"
-					(reference "C58")
+				(path "/74d17fe6-68d4-4bd7-954a-e2bbb58b1f1e/c6e51092-efec-40a8-afae-63cae62691f2/c3c1aad2-e774-4d45-973c-7509c3ed46d5"
+					(reference "C39")
 					(unit 1)
 				)
@@
 		(in_pos_files yes)
 		(dnp no)
-		(property "Reference" "C57"
+		(property "Reference" "C38"
 			(at 38.5572 44.5516 0)
 			(show_name no)
@@
 		(instances
 			(project "PS-PrechargeBoard"
-				(path "/74d17fe6-68d4-4bd7-954a-e2bbb58b1f1e/5e9f1eea-2df2-42e3-8b3e-de31498eaece"
-					(reference "C57")
+				(path "/74d17fe6-68d4-4bd7-954a-e2bbb58b1f1e/c6e51092-efec-40a8-afae-63cae62691f2/c3c1aad2-e774-4d45-973c-7509c3ed46d5"
+					(reference "C38")
 					(unit 1)
 				)
