File: USB-C_Connector.kicad_sch (KiCad schematic)
At the start: 6 parts, among them J1 USB_C_Receptacle_USB2.0_16P

Commit message: lv 1.2
Parts:
- renumbered C1 to C18, D1 to D3, D2 to D4, J1 to J2, R1 to R12, R2 to R13
Changed lines of the file:
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@@
 		(in_pos_files yes)
 		(dnp no)
-		(property "Reference" "R1"
+		(property "Reference" "R12"
 			(at 86.106 48.26 90)
 			(show_name no)
@@
 			(project "PS-PrechargeBoard"
 				(path "/74d17fe6-68d4-4bd7-954a-e2bbb58b1f1e/d871e5fa-d64d-4178-a9ac-7b40bce44e34"
-					(reference "R1")
+					(reference "R12")
 					(unit 1)
 				)
@@
 		(in_pos_files yes)
 		(dnp no)
-		(property "Reference" "R2"
+		(property "Reference" "R13"
 			(at 93.726 48.26 90)
 			(show_name no)
@@
 			(project "PS-PrechargeBoard"
 				(path "/74d17fe6-68d4-4bd7-954a-e2bbb58b1f1e/d871e5fa-d64d-4178-a9ac-7b40bce44e34"
-					(reference "R2")
+					(reference "R13")
 					(unit 1)
 				)
@@
 		(dnp no)
 		(fields_autoplaced yes)
-		(property "Reference" "J1"
+		(property "Reference" "J2"
 			(at 35.56 22.86 0)
 			(show_name no)
@@
 			(project "PS-PrechargeBoard"
 				(path "/74d17fe6-68d4-4bd7-954a-e2bbb58b1f1e/d871e5fa-d64d-4178-a9ac-7b40bce44e34"
-					(reference "J1")
+					(reference "J2")
 					(unit 1)
 				)
@@
 		(dnp no)
 		(fields_autoplaced yes)
-		(property "Reference" "#FLG05"
+		(property "Reference" "#FLG07"
 			(at 71.755 30.48 0)
 			(hide yes)
@@
 			(project "PS-PrechargeBoard"
 				(path "/74d17fe6-68d4-4bd7-954a-e2bbb58b1f1e/d871e5fa-d64d-4178-a9ac-7b40bce44e34"
-					(reference "#FLG05")
+					(reference "#FLG07")
 					(unit 1)
 				)
@@
 		(in_pos_files yes)
 		(dnp no)
-		(property "Reference" "D1"
+		(property "Reference" "D3"
 			(at 59.69 24.765 0)
 			(show_name no)
@@
 			(project "PS-PrechargeBoard"
 				(path "/74d17fe6-68d4-4bd7-954a-e2bbb58b1f1e/d871e5fa-d64d-4178-a9ac-7b40bce44e34"
-					(reference "D1")
+					(reference "D3")
 					(unit 1)
 				)
@@
 		(in_pos_files yes)
 		(dnp no)
-		(property "Reference" "C1"
+		(property "Reference" "C18"
 			(at 64.3128 37.9984 0)
 			(show_name no)
@@
 			(project "PS-PrechargeBoard"
 				(path "/74d17fe6-68d4-4bd7-954a-e2bbb58b1f1e/d871e5fa-d64d-4178-a9ac-7b40bce44e34"
-					(reference "C1")
+					(reference "C18")
 					(unit 1)
 				)
@@
 		(in_pos_files yes)
 		(dnp no)
-		(property "Reference" "D2"
+		(property "Reference" "D4"
 			(at 82.55 71.12 0)
 			(show_name no)
@@
 			(project "PS-PrechargeBoard"
 				(path "/74d17fe6-68d4-4bd7-954a-e2bbb58b1f1e/d871e5fa-d64d-4178-a9ac-7b40bce44e34"
-					(reference "D2")
-					(unit 1)
-				)
+					(reference "D4")
+					(unit 1)
+				)

Commit message: lv 1.3
Parts:
- renumbered J2 to J3
Changed lines of the file:
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@@
 		(dnp no)
 		(fields_autoplaced yes)
-		(property "Reference" "J2"
+		(property "Reference" "J3"
 			(at 35.56 22.86 0)
 			(show_name no)
@@
 			(project "PS-PrechargeBoard"
 				(path "/74d17fe6-68d4-4bd7-954a-e2bbb58b1f1e/d871e5fa-d64d-4178-a9ac-7b40bce44e34"
-					(reference "J2")
+					(reference "J3")
 					(unit 1)
 				)

Commit message: hv 1.0
Parts:
- renumbered C18 to C35, D3 to D7, D4 to D8, J3 to J6, R12 to R24, R13 to R25
Changed lines of the file:
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@@
 		(in_pos_files yes)
 		(dnp no)
-		(property "Reference" "R12"
+		(property "Reference" "R24"
 			(at 86.106 48.26 90)
 			(show_name no)
@@
 			(project "PS-PrechargeBoard"
 				(path "/74d17fe6-68d4-4bd7-954a-e2bbb58b1f1e/d871e5fa-d64d-4178-a9ac-7b40bce44e34"
-					(reference "R12")
+					(reference "R24")
 					(unit 1)
 				)
@@
 		(in_pos_files yes)
 		(dnp no)
-		(property "Reference" "R13"
+		(property "Reference" "R25"
 			(at 93.726 48.26 90)
 			(show_name no)
@@
 			(project "PS-PrechargeBoard"
 				(path "/74d17fe6-68d4-4bd7-954a-e2bbb58b1f1e/d871e5fa-d64d-4178-a9ac-7b40bce44e34"
-					(reference "R13")
+					(reference "R25")
 					(unit 1)
 				)
@@
 		(dnp no)
 		(fields_autoplaced yes)
-		(property "Reference" "J3"
+		(property "Reference" "J6"
 			(at 35.56 22.86 0)
 			(show_name no)
@@
 			(project "PS-PrechargeBoard"
 				(path "/74d17fe6-68d4-4bd7-954a-e2bbb58b1f1e/d871e5fa-d64d-4178-a9ac-7b40bce44e34"
-					(reference "J3")
+					(reference "J6")
 					(unit 1)
 				)
@@
 		(dnp no)
 		(fields_autoplaced yes)
-		(property "Reference" "#FLG07"
+		(property "Reference" "#FLG09"
 			(at 71.755 30.48 0)
 			(hide yes)
@@
 			(project "PS-PrechargeBoard"
 				(path "/74d17fe6-68d4-4bd7-954a-e2bbb58b1f1e/d871e5fa-d64d-4178-a9ac-7b40bce44e34"
-					(reference "#FLG07")
+					(reference "#FLG09")
 					(unit 1)
 				)
@@
 		(in_pos_files yes)
 		(dnp no)
-		(property "Reference" "D3"
+		(property "Reference" "D7"
 			(at 59.69 24.765 0)
 			(show_name no)
@@
 			(project "PS-PrechargeBoard"
 				(path "/74d17fe6-68d4-4bd7-954a-e2bbb58b1f1e/d871e5fa-d64d-4178-a9ac-7b40bce44e34"
-					(reference "D3")
+					(reference "D7")
 					(unit 1)
 				)
@@
 		(in_pos_files yes)
 		(dnp no)
-		(property "Reference" "C18"
+		(property "Reference" "C35"
 			(at 64.3128 37.9984 0)
 			(show_name no)
@@
 			(project "PS-PrechargeBoard"
 				(path "/74d17fe6-68d4-4bd7-954a-e2bbb58b1f1e/d871e5fa-d64d-4178-a9ac-7b40bce44e34"
-					(reference "C18")
+					(reference "C35")
 					(unit 1)
 				)
@@
 		(in_pos_files yes)
 		(dnp no)
-		(property "Reference" "D4"
+		(property "Reference" "D8"
 			(at 82.55 71.12 0)
 			(show_name no)
@@
 			(project "PS-PrechargeBoard"
 				(path "/74d17fe6-68d4-4bd7-954a-e2bbb58b1f1e/d871e5fa-d64d-4178-a9ac-7b40bce44e34"
-					(reference "D4")
-					(unit 1)
-				)
+					(reference "D8")
+					(unit 1)
+				)

Commit message: hv 1.1
Parts:
- renumbered R24 to R23, R25 to R24
Changed lines of the file:
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@@
 		(in_pos_files yes)
 		(dnp no)
-		(property "Reference" "R24"
+		(property "Reference" "R23"
 			(at 86.106 48.26 90)
 			(show_name no)
@@
 			(project "PS-PrechargeBoard"
 				(path "/74d17fe6-68d4-4bd7-954a-e2bbb58b1f1e/d871e5fa-d64d-4178-a9ac-7b40bce44e34"
-					(reference "R24")
+					(reference "R23")
 					(unit 1)
 				)
@@
 		(in_pos_files yes)
 		(dnp no)
-		(property "Reference" "R25"
+		(property "Reference" "R24"
 			(at 93.726 48.26 90)
 			(show_name no)
@@
 			(project "PS-PrechargeBoard"
 				(path "/74d17fe6-68d4-4bd7-954a-e2bbb58b1f1e/d871e5fa-d64d-4178-a9ac-7b40bce44e34"
-					(reference "R25")
+					(reference "R24")
 					(unit 1)
 				)

Commit message: hv 1.2
Parts:
- renumbered J6 to J7
Changed lines of the file:
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@@
 		(dnp no)
 		(fields_autoplaced yes)
-		(property "Reference" "J6"
+		(property "Reference" "J7"
 			(at 35.56 22.86 0)
 			(show_name no)
@@
 			(project "PS-PrechargeBoard"
 				(path "/74d17fe6-68d4-4bd7-954a-e2bbb58b1f1e/d871e5fa-d64d-4178-a9ac-7b40bce44e34"
-					(reference "J6")
+					(reference "J7")
 					(unit 1)
 				)

Commit message: hv 1.3
Parts:
- renumbered C35 to C?, D7 to D?, D8 to D?, J7 to J?, R23 to R?, R24 to R?
Changed lines of the file:
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@@
 		(in_pos_files yes)
 		(dnp no)
-		(property "Reference" "R23"
+		(property "Reference" "R?"
 			(at 86.106 48.26 90)
 			(show_name no)
@@
 		)
 		(instances
-			(project "usb_conn"
-				(path "/64d5c21e-b85c-41ec-b08c-3556f1a0ecf2"
-					(reference "R1")
-					(unit 1)
-				)
-			)
 			(project "PS-PrechargeBoard"
-				(path "/74d17fe6-68d4-4bd7-954a-e2bbb58b1f1e/d871e5fa-d64d-4178-a9ac-7b40bce44e34"
-					(reference "R23")
+				(path "/11743897-1544-4e3c-979c-dcc54ac7093b/341b12dc-4ba7-44e5-bada-7052e6453482"
+					(reference "R?")
 					(unit 1)
 				)
@@
 		(in_pos_files yes)
 		(dnp no)
-		(property "Reference" "R24"
+		(property "Reference" "R?"
 			(at 93.726 48.26 90)
 			(show_name no)
@@
 		)
 		(instances
-			(project "usb_conn"
-				(path "/64d5c21e-b85c-41ec-b08c-3556f1a0ecf2"
-					(reference "R2")
-					(unit 1)
-				)
-			)
 			(project "PS-PrechargeBoard"
-				(path "/74d17fe6-68d4-4bd7-954a-e2bbb58b1f1e/d871e5fa-d64d-4178-a9ac-7b40bce44e34"
-					(reference "R24")
+				(path "/11743897-1544-4e3c-979c-dcc54ac7093b/341b12dc-4ba7-44e5-bada-7052e6453482"
+					(reference "R?")
 					(unit 1)
 				)
@@
 		(dnp no)
 		(fields_autoplaced yes)
-		(property "Reference" "J7"
+		(property "Reference" "J?"
 			(at 35.56 22.86 0)
 			(show_name no)
@@
 		)
 		(instances
-			(project "usb_conn"
-				(path "/64d5c21e-b85c-41ec-b08c-3556f1a0ecf2"
-					(reference "J1")
-					(unit 1)
-				)
-			)
 			(project "PS-PrechargeBoard"
-				(path "/74d17fe6-68d4-4bd7-954a-e2bbb58b1f1e/d871e5fa-d64d-4178-a9ac-7b40bce44e34"
-					(reference "J7")
+				(path "/11743897-1544-4e3c-979c-dcc54ac7093b/341b12dc-4ba7-44e5-bada-7052e6453482"
+					(reference "J?")
 					(unit 1)
 				)
@@
 		(dnp no)
 		(fields_autoplaced yes)
-		(property "Reference" "#FLG09"
+		(property "Reference" "#FLG05"
 			(at 71.755 30.48 0)
 			(hide yes)
@@
 		)
 		(instances
-			(project "usb_conn"
-				(path "/64d5c21e-b85c-41ec-b08c-3556f1a0ecf2"
-					(reference "#FLG01")
-					(unit 1)
-				)
-			)
 			(project "PS-PrechargeBoard"
-				(path "/74d17fe6-68d4-4bd7-954a-e2bbb58b1f1e/d871e5fa-d64d-4178-a9ac-7b40bce44e34"
-					(reference "#FLG09")
+				(path "/11743897-1544-4e3c-979c-dcc54ac7093b/341b12dc-4ba7-44e5-bada-7052e6453482"
+					(reference "#FLG05")
 					(unit 1)
 				)
@@
 		(in_pos_files yes)
 		(dnp no)
-		(property "Reference" "D7"
+		(property "Reference" "D?"
 			(at 59.69 24.765 0)
 			(show_name no)
@@
 		)
 		(instances
-			(project "usb_conn"
-				(path "/64d5c21e-b85c-41ec-b08c-3556f1a0ecf2"
-					(reference "D1")
-					(unit 1)
-				)
-			)
 			(project "PS-PrechargeBoard"
-				(path "/74d17fe6-68d4-4bd7-954a-e2bbb58b1f1e/d871e5fa-d64d-4178-a9ac-7b40bce44e34"
-					(reference "D7")
+				(path "/11743897-1544-4e3c-979c-dcc54ac7093b/341b12dc-4ba7-44e5-bada-7052e6453482"
+					(reference "D?")
 					(unit 1)
 				)
@@
 		(in_pos_files yes)
 		(dnp no)
-		(property "Reference" "C35"
+		(property "Reference" "C?"
 			(at 64.3128 37.9984 0)
 			(show_name no)
@@
 		)
 		(instances
-			(project "usb_conn"
-				(path "/64d5c21e-b85c-41ec-b08c-3556f1a0ecf2"
-					(reference "C1")
-					(unit 1)
-				)
-			)
 			(project "PS-PrechargeBoard"
-				(path "/74d17fe6-68d4-4bd7-954a-e2bbb58b1f1e/d871e5fa-d64d-4178-a9ac-7b40bce44e34"
-					(reference "C35")
+				(path "/11743897-1544-4e3c-979c-dcc54ac7093b/341b12dc-4ba7-44e5-bada-7052e6453482"
+					(reference "C?")
 					(unit 1)
 				)
@@
 		(in_pos_files yes)
 		(dnp no)
-		(property "Reference" "D8"
+		(property "Reference" "D?"
 			(at 82.55 71.12 0)
 			(show_name no)
@@
 		)
 		(instances
-			(project "usb_conn"
-				(path "/64d5c21e-b85c-41ec-b08c-3556f1a0ecf2"
-					(reference "D2")
+			(project "PS-PrechargeBoard"
+				(path "/11743897-1544-4e3c-979c-dcc54ac7093b/341b12dc-4ba7-44e5-bada-7052e6453482"
+					(reference "D?")
 					(unit 1)
 				)
-			)
-			(project "PS-PrechargeBoard"
-				(path "/74d17fe6-68d4-4bd7-954a-e2bbb58b1f1e/d871e5fa-d64d-4178-a9ac-7b40bce44e34"
-					(reference "D8")
-					(unit 1)
-				)
