File: USB-C_Connector.kicad_sch (KiCad schematic)
At the start: 6 parts

Commit message: CAN nano & CAN debug nano
Parts:
- gave numbers to parts that had none: 6
Changed lines of the file:
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@@
 		(in_pos_files yes)
 		(dnp no)
-		(property "Reference" "R?"
+		(property "Reference" "R17"
 			(at 86.106 48.26 90)
 			(show_name no)
@@
 			(project "PS-PrechargeBoard"
 				(path "/74d17fe6-68d4-4bd7-954a-e2bbb58b1f1e/0def18ef-81e8-47ac-b719-2d9f8237a855/341b12dc-4ba7-44e5-bada-7052e6453482"
-					(reference "R?")
+					(reference "R17")
 					(unit 1)
 				)
@@
 			(project "lv"
 				(path "/88356d12-c87f-4bdd-bbd8-756414c90a6d/341b12dc-4ba7-44e5-bada-7052e6453482"
-					(reference "R?")
-					(unit 1)
-				)
-			)
-			(project "PS-PrechargeBoard"
-				(path "/9641192f-df6c-4894-9070-848e3256daf8/341b12dc-4ba7-44e5-bada-7052e6453482"
 					(reference "R?")
 					(unit 1)
@@
 		(in_pos_files yes)
 		(dnp no)
-		(property "Reference" "R?"
+		(property "Reference" "R18"
 			(at 93.726 48.26 90)
 			(show_name no)
@@
 			(project "PS-PrechargeBoard"
 				(path "/74d17fe6-68d4-4bd7-954a-e2bbb58b1f1e/0def18ef-81e8-47ac-b719-2d9f8237a855/341b12dc-4ba7-44e5-bada-7052e6453482"
-					(reference "R?")
+					(reference "R18")
 					(unit 1)
 				)
@@
 			(project "lv"
 				(path "/88356d12-c87f-4bdd-bbd8-756414c90a6d/341b12dc-4ba7-44e5-bada-7052e6453482"
-					(reference "R?")
-					(unit 1)
-				)
-			)
-			(project "PS-PrechargeBoard"
-				(path "/9641192f-df6c-4894-9070-848e3256daf8/341b12dc-4ba7-44e5-bada-7052e6453482"
 					(reference "R?")
 					(unit 1)
@@
 		(dnp no)
 		(fields_autoplaced yes)
-		(property "Reference" "J?"
+		(property "Reference" "J3"
 			(at 35.56 22.86 0)
 			(show_name no)
@@
 			(project "PS-PrechargeBoard"
 				(path "/74d17fe6-68d4-4bd7-954a-e2bbb58b1f1e/0def18ef-81e8-47ac-b719-2d9f8237a855/341b12dc-4ba7-44e5-bada-7052e6453482"
-					(reference "J?")
+					(reference "J3")
 					(unit 1)
 				)
@@
 			(project "lv"
 				(path "/88356d12-c87f-4bdd-bbd8-756414c90a6d/341b12dc-4ba7-44e5-bada-7052e6453482"
-					(reference "J?")
-					(unit 1)
-				)
-			)
-			(project "PS-PrechargeBoard"
-				(path "/9641192f-df6c-4894-9070-848e3256daf8/341b12dc-4ba7-44e5-bada-7052e6453482"
 					(reference "J?")
 					(unit 1)
@@
 		(dnp no)
 		(fields_autoplaced yes)
-		(property "Reference" "#FLG05"
+		(property "Reference" "#FLG01"
 			(at 71.755 30.48 0)
 			(hide yes)
@@
 			(project "PS-PrechargeBoard"
 				(path "/74d17fe6-68d4-4bd7-954a-e2bbb58b1f1e/0def18ef-81e8-47ac-b719-2d9f8237a855/341b12dc-4ba7-44e5-bada-7052e6453482"
-					(reference "#FLG05")
+					(reference "#FLG01")
 					(unit 1)
 				)
@@
 			(project "lv"
 				(path "/88356d12-c87f-4bdd-bbd8-756414c90a6d/341b12dc-4ba7-44e5-bada-7052e6453482"
-					(reference "#FLG05")
-					(unit 1)
-				)
-			)
-			(project "PS-PrechargeBoard"
-				(path "/9641192f-df6c-4894-9070-848e3256daf8/341b12dc-4ba7-44e5-bada-7052e6453482"
 					(reference "#FLG05")
 					(unit 1)
@@
 		(in_pos_files yes)
 		(dnp no)
-		(property "Reference" "D?"
+		(property "Reference" "D7"
 			(at 59.69 24.765 0)
 			(show_name no)
@@
 			(project "PS-PrechargeBoard"
 				(path "/74d17fe6-68d4-4bd7-954a-e2bbb58b1f1e/0def18ef-81e8-47ac-b719-2d9f8237a855/341b12dc-4ba7-44e5-bada-7052e6453482"
-					(reference "D?")
+					(reference "D7")
 					(unit 1)
 				)
@@
 			(project "lv"
 				(path "/88356d12-c87f-4bdd-bbd8-756414c90a6d/341b12dc-4ba7-44e5-bada-7052e6453482"
-					(reference "D?")
-					(unit 1)
-				)
-			)
-			(project "PS-PrechargeBoard"
-				(path "/9641192f-df6c-4894-9070-848e3256daf8/341b12dc-4ba7-44e5-bada-7052e6453482"
 					(reference "D?")
 					(unit 1)
@@
 		(in_pos_files yes)
 		(dnp no)
-		(property "Reference" "C?"
+		(property "Reference" "C27"
 			(at 64.3128 37.9984 0)
 			(show_name no)
@@
 			(project "PS-PrechargeBoard"
 				(path "/74d17fe6-68d4-4bd7-954a-e2bbb58b1f1e/0def18ef-81e8-47ac-b719-2d9f8237a855/341b12dc-4ba7-44e5-bada-7052e6453482"
-					(reference "C?")
+					(reference "C27")
 					(unit 1)
 				)
@@
 			(project "lv"
 				(path "/88356d12-c87f-4bdd-bbd8-756414c90a6d/341b12dc-4ba7-44e5-bada-7052e6453482"
-					(reference "C?")
-					(unit 1)
-				)
-			)
-			(project "PS-PrechargeBoard"
-				(path "/9641192f-df6c-4894-9070-848e3256daf8/341b12dc-4ba7-44e5-bada-7052e6453482"
 					(reference "C?")
 					(unit 1)
@@
 		(in_pos_files yes)
 		(dnp no)
-		(property "Reference" "D?"
+		(property "Reference" "D8"
 			(at 82.55 71.12 0)
 			(show_name no)
@@
 			(project "PS-PrechargeBoard"
 				(path "/74d17fe6-68d4-4bd7-954a-e2bbb58b1f1e/0def18ef-81e8-47ac-b719-2d9f8237a855/341b12dc-4ba7-44e5-bada-7052e6453482"
-					(reference "D?")
+					(reference "D8")
 					(unit 1)
 				)
@@
 					(reference "D?")
 					(unit 1)
-				)
-			)
-			(project "PS-PrechargeBoard"
-				(path "/9641192f-df6c-4894-9070-848e3256daf8/341b12dc-4ba7-44e5-bada-7052e6453482"
-					(reference "D?")
-					(unit 1)

Commit message: battery voltage & motor voltage
Parts:
- renumbered C27 to C43, D7 to D10, D8 to D11, J3 to J11, R17 to R34, R18 to R35
Changed lines of the file:
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@@
 		(in_pos_files yes)
 		(dnp no)
-		(property "Reference" "R17"
+		(property "Reference" "R34"
 			(at 86.106 48.26 90)
 			(show_name no)
@@
 			(project "PS-PrechargeBoard"
 				(path "/74d17fe6-68d4-4bd7-954a-e2bbb58b1f1e/0def18ef-81e8-47ac-b719-2d9f8237a855/341b12dc-4ba7-44e5-bada-7052e6453482"
-					(reference "R17")
+					(reference "R34")
 					(unit 1)
 				)
@@
 		(in_pos_files yes)
 		(dnp no)
-		(property "Reference" "R18"
+		(property "Reference" "R35"
 			(at 93.726 48.26 90)
 			(show_name no)
@@
 			(project "PS-PrechargeBoard"
 				(path "/74d17fe6-68d4-4bd7-954a-e2bbb58b1f1e/0def18ef-81e8-47ac-b719-2d9f8237a855/341b12dc-4ba7-44e5-bada-7052e6453482"
-					(reference "R18")
+					(reference "R35")
 					(unit 1)
 				)
@@
 		(dnp no)
 		(fields_autoplaced yes)
-		(property "Reference" "J3"
+		(property "Reference" "J11"
 			(at 35.56 22.86 0)
 			(show_name no)
@@
 			(project "PS-PrechargeBoard"
 				(path "/74d17fe6-68d4-4bd7-954a-e2bbb58b1f1e/0def18ef-81e8-47ac-b719-2d9f8237a855/341b12dc-4ba7-44e5-bada-7052e6453482"
-					(reference "J3")
+					(reference "J11")
 					(unit 1)
 				)
@@
 		(dnp no)
 		(fields_autoplaced yes)
-		(property "Reference" "#FLG01"
+		(property "Reference" "#FLG011"
 			(at 71.755 30.48 0)
 			(hide yes)
@@
 			(project "PS-PrechargeBoard"
 				(path "/74d17fe6-68d4-4bd7-954a-e2bbb58b1f1e/0def18ef-81e8-47ac-b719-2d9f8237a855/341b12dc-4ba7-44e5-bada-7052e6453482"
-					(reference "#FLG01")
+					(reference "#FLG011")
 					(unit 1)
 				)
@@
 		(in_pos_files yes)
 		(dnp no)
-		(property "Reference" "D7"
+		(property "Reference" "D10"
 			(at 59.69 24.765 0)
 			(show_name no)
@@
 			(project "PS-PrechargeBoard"
 				(path "/74d17fe6-68d4-4bd7-954a-e2bbb58b1f1e/0def18ef-81e8-47ac-b719-2d9f8237a855/341b12dc-4ba7-44e5-bada-7052e6453482"
-					(reference "D7")
+					(reference "D10")
 					(unit 1)
 				)
@@
 		(in_pos_files yes)
 		(dnp no)
-		(property "Reference" "C27"
+		(property "Reference" "C43"
 			(at 64.3128 37.9984 0)
 			(show_name no)
@@
 			(project "PS-PrechargeBoard"
 				(path "/74d17fe6-68d4-4bd7-954a-e2bbb58b1f1e/0def18ef-81e8-47ac-b719-2d9f8237a855/341b12dc-4ba7-44e5-bada-7052e6453482"
-					(reference "C27")
+					(reference "C43")
 					(unit 1)
 				)
@@
 		(in_pos_files yes)
 		(dnp no)
-		(property "Reference" "D8"
+		(property "Reference" "D11"
 			(at 82.55 71.12 0)
 			(show_name no)
@@
 			(project "PS-PrechargeBoard"
 				(path "/74d17fe6-68d4-4bd7-954a-e2bbb58b1f1e/0def18ef-81e8-47ac-b719-2d9f8237a855/341b12dc-4ba7-44e5-bada-7052e6453482"
-					(reference "D8")
-					(unit 1)
-				)
+					(reference "D11")
+					(unit 1)
+				)

Commit message: mini review notes
Parts:
- renumbered D10 to D12, D11 to D13
Changed lines of the file:
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@@
 		(dnp no)
 		(fields_autoplaced yes)
-		(property "Reference" "#FLG011"
+		(property "Reference" "#FLG09"
 			(at 71.755 30.48 0)
 			(hide yes)
@@
 			(project "PS-PrechargeBoard"
 				(path "/74d17fe6-68d4-4bd7-954a-e2bbb58b1f1e/0def18ef-81e8-47ac-b719-2d9f8237a855/341b12dc-4ba7-44e5-bada-7052e6453482"
-					(reference "#FLG011")
+					(reference "#FLG09")
 					(unit 1)
 				)
@@
 		(in_pos_files yes)
 		(dnp no)
-		(property "Reference" "D10"
+		(property "Reference" "D12"
 			(at 59.69 24.765 0)
 			(show_name no)
@@
 			(project "PS-PrechargeBoard"
 				(path "/74d17fe6-68d4-4bd7-954a-e2bbb58b1f1e/0def18ef-81e8-47ac-b719-2d9f8237a855/341b12dc-4ba7-44e5-bada-7052e6453482"
-					(reference "D10")
+					(reference "D12")
 					(unit 1)
 				)
@@
 		(in_pos_files yes)
 		(dnp no)
-		(property "Reference" "D11"
+		(property "Reference" "D13"
 			(at 82.55 71.12 0)
 			(show_name no)
@@
 			(project "PS-PrechargeBoard"
 				(path "/74d17fe6-68d4-4bd7-954a-e2bbb58b1f1e/0def18ef-81e8-47ac-b719-2d9f8237a855/341b12dc-4ba7-44e5-bada-7052e6453482"
-					(reference "D11")
-					(unit 1)
-				)
+					(reference "D13")
+					(unit 1)
+				)

Commit message: shifted hierarchical sheets
Parts:
- renumbered C43 to C?, D12 to D?, D13 to D?, J11 to J?, R34 to R?, R35 to R?
Changed lines of the file:
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@@
 		(in_pos_files yes)
 		(dnp no)
-		(property "Reference" "R34"
+		(property "Reference" "R?"
 			(at 86.106 48.26 90)
 			(show_name no)
@@
 		(instances
 			(project "PS-PrechargeBoard"
-				(path "/74d17fe6-68d4-4bd7-954a-e2bbb58b1f1e/0def18ef-81e8-47ac-b719-2d9f8237a855/341b12dc-4ba7-44e5-bada-7052e6453482"
-					(reference "R34")
-					(unit 1)
-				)
-			)
-			(project "lv"
-				(path "/88356d12-c87f-4bdd-bbd8-756414c90a6d/341b12dc-4ba7-44e5-bada-7052e6453482"
+				(path "/74d17fe6-68d4-4bd7-954a-e2bbb58b1f1e/fc3b8ec8-73b6-403d-a70a-e3464732b3c3"
 					(reference "R?")
 					(unit 1)
@@
 		(in_pos_files yes)
 		(dnp no)
-		(property "Reference" "R35"
+		(property "Reference" "R?"
 			(at 93.726 48.26 90)
 			(show_name no)
@@
 		(instances
 			(project "PS-PrechargeBoard"
-				(path "/74d17fe6-68d4-4bd7-954a-e2bbb58b1f1e/0def18ef-81e8-47ac-b719-2d9f8237a855/341b12dc-4ba7-44e5-bada-7052e6453482"
-					(reference "R35")
-					(unit 1)
-				)
-			)
-			(project "lv"
-				(path "/88356d12-c87f-4bdd-bbd8-756414c90a6d/341b12dc-4ba7-44e5-bada-7052e6453482"
+				(path "/74d17fe6-68d4-4bd7-954a-e2bbb58b1f1e/fc3b8ec8-73b6-403d-a70a-e3464732b3c3"
 					(reference "R?")
 					(unit 1)
@@
 		(dnp no)
 		(fields_autoplaced yes)
-		(property "Reference" "J11"
+		(property "Reference" "J?"
 			(at 35.56 22.86 0)
 			(show_name no)
@@
 		(instances
 			(project "PS-PrechargeBoard"
-				(path "/74d17fe6-68d4-4bd7-954a-e2bbb58b1f1e/0def18ef-81e8-47ac-b719-2d9f8237a855/341b12dc-4ba7-44e5-bada-7052e6453482"
-					(reference "J11")
-					(unit 1)
-				)
-			)
-			(project "lv"
-				(path "/88356d12-c87f-4bdd-bbd8-756414c90a6d/341b12dc-4ba7-44e5-bada-7052e6453482"
+				(path "/74d17fe6-68d4-4bd7-954a-e2bbb58b1f1e/fc3b8ec8-73b6-403d-a70a-e3464732b3c3"
 					(reference "J?")
 					(unit 1)
@@
 		(dnp no)
 		(fields_autoplaced yes)
-		(property "Reference" "#FLG09"
+		(property "Reference" "#FLG015"
 			(at 71.755 30.48 0)
 			(hide yes)
@@
 		(instances
 			(project "PS-PrechargeBoard"
-				(path "/74d17fe6-68d4-4bd7-954a-e2bbb58b1f1e/0def18ef-81e8-47ac-b719-2d9f8237a855/341b12dc-4ba7-44e5-bada-7052e6453482"
-					(reference "#FLG09")
-					(unit 1)
-				)
-			)
-			(project "lv"
-				(path "/88356d12-c87f-4bdd-bbd8-756414c90a6d/341b12dc-4ba7-44e5-bada-7052e6453482"
-					(reference "#FLG05")
+				(path "/74d17fe6-68d4-4bd7-954a-e2bbb58b1f1e/fc3b8ec8-73b6-403d-a70a-e3464732b3c3"
+					(reference "#FLG015")
 					(unit 1)
 				)
@@
 		(in_pos_files yes)
 		(dnp no)
-		(property "Reference" "D12"
+		(property "Reference" "D?"
 			(at 59.69 24.765 0)
 			(show_name no)
@@
 		(instances
 			(project "PS-PrechargeBoard"
-				(path "/74d17fe6-68d4-4bd7-954a-e2bbb58b1f1e/0def18ef-81e8-47ac-b719-2d9f8237a855/341b12dc-4ba7-44e5-bada-7052e6453482"
-					(reference "D12")
-					(unit 1)
-				)
-			)
-			(project "lv"
-				(path "/88356d12-c87f-4bdd-bbd8-756414c90a6d/341b12dc-4ba7-44e5-bada-7052e6453482"
+				(path "/74d17fe6-68d4-4bd7-954a-e2bbb58b1f1e/fc3b8ec8-73b6-403d-a70a-e3464732b3c3"
 					(reference "D?")
 					(unit 1)
@@
 		(in_pos_files yes)
 		(dnp no)
-		(property "Reference" "C43"
+		(property "Reference" "C?"
 			(at 64.3128 37.9984 0)
 			(show_name no)
@@
 		(instances
 			(project "PS-PrechargeBoard"
-				(path "/74d17fe6-68d4-4bd7-954a-e2bbb58b1f1e/0def18ef-81e8-47ac-b719-2d9f8237a855/341b12dc-4ba7-44e5-bada-7052e6453482"
-					(reference "C43")
-					(unit 1)
-				)
-			)
-			(project "lv"
-				(path "/88356d12-c87f-4bdd-bbd8-756414c90a6d/341b12dc-4ba7-44e5-bada-7052e6453482"
+				(path "/74d17fe6-68d4-4bd7-954a-e2bbb58b1f1e/fc3b8ec8-73b6-403d-a70a-e3464732b3c3"
 					(reference "C?")
 					(unit 1)
@@
 		(in_pos_files yes)
 		(dnp no)
-		(property "Reference" "D13"
+		(property "Reference" "D?"
 			(at 82.55 71.12 0)
 			(show_name no)
@@
 		(instances
 			(project "PS-PrechargeBoard"
-				(path "/74d17fe6-68d4-4bd7-954a-e2bbb58b1f1e/0def18ef-81e8-47ac-b719-2d9f8237a855/341b12dc-4ba7-44e5-bada-7052e6453482"
-					(reference "D13")
-					(unit 1)
-				)
-			)
-			(project "lv"
-				(path "/88356d12-c87f-4bdd-bbd8-756414c90a6d/341b12dc-4ba7-44e5-bada-7052e6453482"
+				(path "/74d17fe6-68d4-4bd7-954a-e2bbb58b1f1e/fc3b8ec8-73b6-403d-a70a-e3464732b3c3"
 					(reference "D?")
 					(unit 1)

Commit message: V_OUT_BAT & V_OUT_MOT & PRECHARGE_CTRL to MCU
Parts:
- gave numbers to parts that had none: 6
Changed lines of the file:
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@@
 		(in_pos_files yes)
 		(dnp no)
-		(property "Reference" "R?"
+		(property "Reference" "R48"
 			(at 86.106 48.26 90)
 			(show_name no)
@@
 			(project "PS-PrechargeBoard"
 				(path "/74d17fe6-68d4-4bd7-954a-e2bbb58b1f1e/fc3b8ec8-73b6-403d-a70a-e3464732b3c3"
-					(reference "R?")
+					(reference "R48")
 					(unit 1)
 				)
@@
 		(in_pos_files yes)
 		(dnp no)
-		(property "Reference" "R?"
+		(property "Reference" "R49"
 			(at 93.726 48.26 90)
 			(show_name no)
@@
 			(project "PS-PrechargeBoard"
 				(path "/74d17fe6-68d4-4bd7-954a-e2bbb58b1f1e/fc3b8ec8-73b6-403d-a70a-e3464732b3c3"
-					(reference "R?")
+					(reference "R49")
 					(unit 1)
 				)
@@
 		(dnp no)
 		(fields_autoplaced yes)
-		(property "Reference" "J?"
+		(property "Reference" "J8"
 			(at 35.56 22.86 0)
 			(show_name no)
@@
 			(project "PS-PrechargeBoard"
 				(path "/74d17fe6-68d4-4bd7-954a-e2bbb58b1f1e/fc3b8ec8-73b6-403d-a70a-e3464732b3c3"
-					(reference "J?")
+					(reference "J8")
 					(unit 1)
 				)
@@
 		(dnp no)
 		(fields_autoplaced yes)
-		(property "Reference" "#FLG015"
+		(property "Reference" "#FLG09"
 			(at 71.755 30.48 0)
 			(hide yes)
@@
 			(project "PS-PrechargeBoard"
 				(path "/74d17fe6-68d4-4bd7-954a-e2bbb58b1f1e/fc3b8ec8-73b6-403d-a70a-e3464732b3c3"
-					(reference "#FLG015")
+					(reference "#FLG09")
 					(unit 1)
 				)
@@
 		(in_pos_files yes)
 		(dnp no)
-		(property "Reference" "D?"
+		(property "Reference" "D13"
 			(at 59.69 24.765 0)
 			(show_name no)
@@
 			(project "PS-PrechargeBoard"
 				(path "/74d17fe6-68d4-4bd7-954a-e2bbb58b1f1e/fc3b8ec8-73b6-403d-a70a-e3464732b3c3"
-					(reference "D?")
+					(reference "D13")
 					(unit 1)
 				)
@@
 		(in_pos_files yes)
 		(dnp no)
-		(property "Reference" "C?"
+		(property "Reference" "C60"
 			(at 64.3128 37.9984 0)
 			(show_name no)
@@
 			(project "PS-PrechargeBoard"
 				(path "/74d17fe6-68d4-4bd7-954a-e2bbb58b1f1e/fc3b8ec8-73b6-403d-a70a-e3464732b3c3"
-					(reference "C?")
+					(reference "C60")
 					(unit 1)
 				)
@@
 		(in_pos_files yes)
 		(dnp no)
-		(property "Reference" "D?"
+		(property "Reference" "D14"
 			(at 82.55 71.12 0)
 			(show_name no)
@@
 			(project "PS-PrechargeBoard"
 				(path "/74d17fe6-68d4-4bd7-954a-e2bbb58b1f1e/fc3b8ec8-73b6-403d-a70a-e3464732b3c3"
-					(reference "D?")
+					(reference "D14")
 					(unit 1)
 				)

Commit message: precharges & voltage sensors
Parts:
- renumbered C60 to C76, D13 to D17, D14 to D18, J8 to J9, R48 to R67, R49 to R68
Changed lines of the file:
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@@
 		(in_pos_files yes)
 		(dnp no)
-		(property "Reference" "R48"
+		(property "Reference" "R67"
 			(at 86.106 48.26 90)
 			(show_name no)
@@
 			(project "PS-PrechargeBoard"
 				(path "/74d17fe6-68d4-4bd7-954a-e2bbb58b1f1e/fc3b8ec8-73b6-403d-a70a-e3464732b3c3"
-					(reference "R48")
+					(reference "R67")
 					(unit 1)
 				)
@@
 		(in_pos_files yes)
 		(dnp no)
-		(property "Reference" "R49"
+		(property "Reference" "R68"
 			(at 93.726 48.26 90)
 			(show_name no)
@@
 			(project "PS-PrechargeBoard"
 				(path "/74d17fe6-68d4-4bd7-954a-e2bbb58b1f1e/fc3b8ec8-73b6-403d-a70a-e3464732b3c3"
-					(reference "R49")
+					(reference "R68")
 					(unit 1)
 				)
@@
 		(dnp no)
 		(fields_autoplaced yes)
-		(property "Reference" "J8"
+		(property "Reference" "J9"
 			(at 35.56 22.86 0)
 			(show_name no)
@@
 			(project "PS-PrechargeBoard"
 				(path "/74d17fe6-68d4-4bd7-954a-e2bbb58b1f1e/fc3b8ec8-73b6-403d-a70a-e3464732b3c3"
-					(reference "J8")
+					(reference "J9")
 					(unit 1)
 				)
@@
 		(dnp no)
 		(fields_autoplaced yes)
-		(property "Reference" "#FLG09"
+		(property "Reference" "#FLG011"
 			(at 71.755 30.48 0)
 			(hide yes)
@@
 			(project "PS-PrechargeBoard"
 				(path "/74d17fe6-68d4-4bd7-954a-e2bbb58b1f1e/fc3b8ec8-73b6-403d-a70a-e3464732b3c3"
-					(reference "#FLG09")
+					(reference "#FLG011")
 					(unit 1)
 				)
@@
 		(in_pos_files yes)
 		(dnp no)
-		(property "Reference" "D13"
+		(property "Reference" "D17"
 			(at 59.69 24.765 0)
 			(show_name no)
@@
 			(project "PS-PrechargeBoard"
 				(path "/74d17fe6-68d4-4bd7-954a-e2bbb58b1f1e/fc3b8ec8-73b6-403d-a70a-e3464732b3c3"
-					(reference "D13")
+					(reference "D17")
 					(unit 1)
 				)
@@
 		(in_pos_files yes)
 		(dnp no)
-		(property "Reference" "C60"
+		(property "Reference" "C76"
 			(at 64.3128 37.9984 0)
 			(show_name no)
@@
 			(project "PS-PrechargeBoard"
 				(path "/74d17fe6-68d4-4bd7-954a-e2bbb58b1f1e/fc3b8ec8-73b6-403d-a70a-e3464732b3c3"
-					(reference "C60")
+					(reference "C76")
 					(unit 1)
 				)
@@
 		(in_pos_files yes)
 		(dnp no)
-		(property "Reference" "D14"
+		(property "Reference" "D18"
 			(at 82.55 71.12 0)
 			(show_name no)
@@
 			(project "PS-PrechargeBoard"
 				(path "/74d17fe6-68d4-4bd7-954a-e2bbb58b1f1e/fc3b8ec8-73b6-403d-a70a-e3464732b3c3"
-					(reference "D14")
+					(reference "D18")
 					(unit 1)
 				)

Commit message: final schematic REV-A?
Parts:
- renumbered C76 to C46, D17 to D13, D18 to D14, J9 to J6, R67 to R60, R68 to R61
Changed lines of the file:
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@@
 		(in_pos_files yes)
 		(dnp no)
-		(property "Reference" "R67"
+		(property "Reference" "R60"
 			(at 86.106 48.26 90)
 			(show_name no)
@@
 		(instances
 			(project "PS-PrechargeBoard"
-				(path "/74d17fe6-68d4-4bd7-954a-e2bbb58b1f1e/fc3b8ec8-73b6-403d-a70a-e3464732b3c3"
-					(reference "R67")
+				(path "/74d17fe6-68d4-4bd7-954a-e2bbb58b1f1e/2ca150cf-fbe5-4d5b-a7dc-f2dc5c6024d0/2a3ef9c4-dfbd-4c37-804f-440ab95d2b69"
+					(reference "R60")
 					(unit 1)
 				)
@@
 		(in_pos_files yes)
 		(dnp no)
-		(property "Reference" "R68"
+		(property "Reference" "R61"
 			(at 93.726 48.26 90)
 			(show_name no)
@@
 		(instances
 			(project "PS-PrechargeBoard"
-				(path "/74d17fe6-68d4-4bd7-954a-e2bbb58b1f1e/fc3b8ec8-73b6-403d-a70a-e3464732b3c3"
-					(reference "R68")
+				(path "/74d17fe6-68d4-4bd7-954a-e2bbb58b1f1e/2ca150cf-fbe5-4d5b-a7dc-f2dc5c6024d0/2a3ef9c4-dfbd-4c37-804f-440ab95d2b69"
+					(reference "R61")
 					(unit 1)
 				)
@@
 		(dnp no)
 		(fields_autoplaced yes)
-		(property "Reference" "J9"
+		(property "Reference" "J6"
 			(at 35.56 22.86 0)
 			(show_name no)
@@
 		(instances
 			(project "PS-PrechargeBoard"
-				(path "/74d17fe6-68d4-4bd7-954a-e2bbb58b1f1e/fc3b8ec8-73b6-403d-a70a-e3464732b3c3"
-					(reference "J9")
+				(path "/74d17fe6-68d4-4bd7-954a-e2bbb58b1f1e/2ca150cf-fbe5-4d5b-a7dc-f2dc5c6024d0/2a3ef9c4-dfbd-4c37-804f-440ab95d2b69"
+					(reference "J6")
 					(unit 1)
 				)
@@
 		(dnp no)
 		(fields_autoplaced yes)
-		(property "Reference" "#FLG011"
+		(property "Reference" "#FLG06"
 			(at 71.755 30.48 0)
 			(hide yes)
@@
 		(instances
 			(project "PS-PrechargeBoard"
-				(path "/74d17fe6-68d4-4bd7-954a-e2bbb58b1f1e/fc3b8ec8-73b6-403d-a70a-e3464732b3c3"
-					(reference "#FLG011")
+				(path "/74d17fe6-68d4-4bd7-954a-e2bbb58b1f1e/2ca150cf-fbe5-4d5b-a7dc-f2dc5c6024d0/2a3ef9c4-dfbd-4c37-804f-440ab95d2b69"
+					(reference "#FLG06")
 					(unit 1)
 				)
@@
 		(in_pos_files yes)
 		(dnp no)
-		(property "Reference" "D17"
+		(property "Reference" "D13"
 			(at 59.69 24.765 0)
 			(show_name no)
@@
 		(instances
 			(project "PS-PrechargeBoard"
-				(path "/74d17fe6-68d4-4bd7-954a-e2bbb58b1f1e/fc3b8ec8-73b6-403d-a70a-e3464732b3c3"
-					(reference "D17")
+				(path "/74d17fe6-68d4-4bd7-954a-e2bbb58b1f1e/2ca150cf-fbe5-4d5b-a7dc-f2dc5c6024d0/2a3ef9c4-dfbd-4c37-804f-440ab95d2b69"
+					(reference "D13")
 					(unit 1)
 				)
@@
 		(in_pos_files yes)
 		(dnp no)
-		(property "Reference" "C76"
+		(property "Reference" "C46"
 			(at 64.3128 37.9984 0)
 			(show_name no)
@@
 		(instances
 			(project "PS-PrechargeBoard"
-				(path "/74d17fe6-68d4-4bd7-954a-e2bbb58b1f1e/fc3b8ec8-73b6-403d-a70a-e3464732b3c3"
-					(reference "C76")
+				(path "/74d17fe6-68d4-4bd7-954a-e2bbb58b1f1e/2ca150cf-fbe5-4d5b-a7dc-f2dc5c6024d0/2a3ef9c4-dfbd-4c37-804f-440ab95d2b69"
+					(reference "C46")
 					(unit 1)
 				)
@@
 		(in_pos_files yes)
 		(dnp no)
-		(property "Reference" "D18"
+		(property "Reference" "D14"
 			(at 82.55 71.12 0)
 			(show_name no)
@@
 		(instances
 			(project "PS-PrechargeBoard"
-				(path "/74d17fe6-68d4-4bd7-954a-e2bbb58b1f1e/fc3b8ec8-73b6-403d-a70a-e3464732b3c3"
-					(reference "D18")
+				(path "/74d17fe6-68d4-4bd7-954a-e2bbb58b1f1e/2ca150cf-fbe5-4d5b-a7dc-f2dc5c6024d0/2a3ef9c4-dfbd-4c37-804f-440ab95d2b69"
+					(reference "D14")
 					(unit 1)
 				)
