File: USB-C_Connector.kicad_sch (KiCad schematic)
At the start: 6 parts, among them J15 USB_C_Receptacle_USB2.0_16P

Commit message: isolated precharge from fuse
Parts:
- renumbered C55 to C57, J15 to J10
Changed lines of the file:
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@@
 		(dnp no)
 		(fields_autoplaced yes)
-		(property "Reference" "J15"
+		(property "Reference" "J10"
 			(at 35.56 22.86 0)
 			(show_name no)
@@
 			(project "PS-PrechargeBoard"
 				(path "/74d17fe6-68d4-4bd7-954a-e2bbb58b1f1e/2ca150cf-fbe5-4d5b-a7dc-f2dc5c6024d0/2a3ef9c4-dfbd-4c37-804f-440ab95d2b69"
-					(reference "J15")
+					(reference "J10")
 					(unit 1)
 				)
@@
 		(in_pos_files yes)
 		(dnp no)
-		(property "Reference" "C55"
+		(property "Reference" "C57"
 			(at 64.3128 37.9984 0)
 			(show_name no)
@@
 			(project "PS-PrechargeBoard"
 				(path "/74d17fe6-68d4-4bd7-954a-e2bbb58b1f1e/2ca150cf-fbe5-4d5b-a7dc-f2dc5c6024d0/2a3ef9c4-dfbd-4c37-804f-440ab95d2b69"
-					(reference "C55")
+					(reference "C57")
 					(unit 1)
 				)

Commit message: voltage sensor cleanup
Parts:
- renumbered D16 to D14, D17 to D15, R73 to R74, R74 to R75
Changed lines of the file:
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@@
 		(in_pos_files yes)
 		(dnp no)
-		(property "Reference" "R73"
+		(property "Reference" "R74"
 			(at 86.106 48.26 90)
 			(show_name no)
@@
 			(project "PS-PrechargeBoard"
 				(path "/74d17fe6-68d4-4bd7-954a-e2bbb58b1f1e/2ca150cf-fbe5-4d5b-a7dc-f2dc5c6024d0/2a3ef9c4-dfbd-4c37-804f-440ab95d2b69"
-					(reference "R73")
+					(reference "R74")
 					(unit 1)
 				)
@@
 		(in_pos_files yes)
 		(dnp no)
-		(property "Reference" "R74"
+		(property "Reference" "R75"
 			(at 93.726 48.26 90)
 			(show_name no)
@@
 			(project "PS-PrechargeBoard"
 				(path "/74d17fe6-68d4-4bd7-954a-e2bbb58b1f1e/2ca150cf-fbe5-4d5b-a7dc-f2dc5c6024d0/2a3ef9c4-dfbd-4c37-804f-440ab95d2b69"
-					(reference "R74")
+					(reference "R75")
 					(unit 1)
 				)
@@
 		(in_pos_files yes)
 		(dnp no)
-		(property "Reference" "D16"
+		(property "Reference" "D14"
 			(at 59.69 24.765 0)
 			(show_name no)
@@
 			(project "PS-PrechargeBoard"
 				(path "/74d17fe6-68d4-4bd7-954a-e2bbb58b1f1e/2ca150cf-fbe5-4d5b-a7dc-f2dc5c6024d0/2a3ef9c4-dfbd-4c37-804f-440ab95d2b69"
-					(reference "D16")
+					(reference "D14")
 					(unit 1)
 				)
@@
 		(in_pos_files yes)
 		(dnp no)
-		(property "Reference" "D17"
+		(property "Reference" "D15"
 			(at 82.55 71.12 0)
 			(show_name no)
@@
 			(project "PS-PrechargeBoard"
 				(path "/74d17fe6-68d4-4bd7-954a-e2bbb58b1f1e/2ca150cf-fbe5-4d5b-a7dc-f2dc5c6024d0/2a3ef9c4-dfbd-4c37-804f-440ab95d2b69"
-					(reference "D17")
+					(reference "D15")
 					(unit 1)
 				)

Commit message: updated usb-c connector
Parts:
- J8: renamed from J10; footprint LHRS_ICs:USB_C_Receptacle_GCT_USB4105-xx-A_16P_TopMnt_Horizontal -> LHRS_Connectors:USB_C_Receptacle_GCT_USB4105-xx-A_16P_TopMnt_Horizontal
- renumbered C57 to C50, D14 to D11, D15 to D12, R74 to R70, R75 to R71
Changed lines of the file:
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@@
 		(in_pos_files yes)
 		(dnp no)
-		(property "Reference" "R74"
+		(property "Reference" "R70"
 			(at 86.106 48.26 90)
 			(show_name no)
@@
 		(instances
 			(project "PS-PrechargeBoard"
-				(path "/74d17fe6-68d4-4bd7-954a-e2bbb58b1f1e/2ca150cf-fbe5-4d5b-a7dc-f2dc5c6024d0/2a3ef9c4-dfbd-4c37-804f-440ab95d2b69"
-					(reference "R74")
+				(path "/74d17fe6-68d4-4bd7-954a-e2bbb58b1f1e/2ca150cf-fbe5-4d5b-a7dc-f2dc5c6024d0/278d3e71-a9d8-40e3-a9e7-673513fdd902"
+					(reference "R70")
 					(unit 1)
 				)
@@
 		(in_pos_files yes)
 		(dnp no)
-		(property "Reference" "R75"
+		(property "Reference" "R71"
 			(at 93.726 48.26 90)
 			(show_name no)
@@
 		(instances
 			(project "PS-PrechargeBoard"
-				(path "/74d17fe6-68d4-4bd7-954a-e2bbb58b1f1e/2ca150cf-fbe5-4d5b-a7dc-f2dc5c6024d0/2a3ef9c4-dfbd-4c37-804f-440ab95d2b69"
-					(reference "R75")
+				(path "/74d17fe6-68d4-4bd7-954a-e2bbb58b1f1e/2ca150cf-fbe5-4d5b-a7dc-f2dc5c6024d0/278d3e71-a9d8-40e3-a9e7-673513fdd902"
+					(reference "R71")
 					(unit 1)
 				)
@@
 		(dnp no)
 		(fields_autoplaced yes)
-		(property "Reference" "J10"
+		(property "Reference" "J8"
 			(at 35.56 22.86 0)
 			(show_name no)
@@
 			)
 		)
-		(property "Footprint" "LHRS_ICs:USB_C_Receptacle_GCT_USB4105-xx-A_16P_TopMnt_Horizontal"
+		(property "Footprint" "LHRS_Connectors:USB_C_Receptacle_GCT_USB4105-xx-A_16P_TopMnt_Horizontal"
 			(at 39.37 45.72 0)
 			(hide yes)
@@
 		(instances
 			(project "PS-PrechargeBoard"
-				(path "/74d17fe6-68d4-4bd7-954a-e2bbb58b1f1e/2ca150cf-fbe5-4d5b-a7dc-f2dc5c6024d0/2a3ef9c4-dfbd-4c37-804f-440ab95d2b69"
-					(reference "J10")
+				(path "/74d17fe6-68d4-4bd7-954a-e2bbb58b1f1e/2ca150cf-fbe5-4d5b-a7dc-f2dc5c6024d0/278d3e71-a9d8-40e3-a9e7-673513fdd902"
+					(reference "J8")
 					(unit 1)
 				)
@@
 		(dnp no)
 		(fields_autoplaced yes)
-		(property "Reference" "#FLG02"
+		(property "Reference" "#FLG03"
 			(at 71.755 30.48 0)
 			(hide yes)
@@
 		(instances
 			(project "PS-PrechargeBoard"
-				(path "/74d17fe6-68d4-4bd7-954a-e2bbb58b1f1e/2ca150cf-fbe5-4d5b-a7dc-f2dc5c6024d0/2a3ef9c4-dfbd-4c37-804f-440ab95d2b69"
-					(reference "#FLG02")
+				(path "/74d17fe6-68d4-4bd7-954a-e2bbb58b1f1e/2ca150cf-fbe5-4d5b-a7dc-f2dc5c6024d0/278d3e71-a9d8-40e3-a9e7-673513fdd902"
+					(reference "#FLG03")
 					(unit 1)
 				)
@@
 		(in_pos_files yes)
 		(dnp no)
-		(property "Reference" "D14"
+		(property "Reference" "D11"
 			(at 59.69 24.765 0)
 			(show_name no)
@@
 		(instances
 			(project "PS-PrechargeBoard"
-				(path "/74d17fe6-68d4-4bd7-954a-e2bbb58b1f1e/2ca150cf-fbe5-4d5b-a7dc-f2dc5c6024d0/2a3ef9c4-dfbd-4c37-804f-440ab95d2b69"
-					(reference "D14")
+				(path "/74d17fe6-68d4-4bd7-954a-e2bbb58b1f1e/2ca150cf-fbe5-4d5b-a7dc-f2dc5c6024d0/278d3e71-a9d8-40e3-a9e7-673513fdd902"
+					(reference "D11")
 					(unit 1)
 				)
@@
 		(in_pos_files yes)
 		(dnp no)
-		(property "Reference" "C57"
+		(property "Reference" "C50"
 			(at 64.3128 37.9984 0)
 			(show_name no)
@@
 		(instances
 			(project "PS-PrechargeBoard"
-				(path "/74d17fe6-68d4-4bd7-954a-e2bbb58b1f1e/2ca150cf-fbe5-4d5b-a7dc-f2dc5c6024d0/2a3ef9c4-dfbd-4c37-804f-440ab95d2b69"
-					(reference "C57")
+				(path "/74d17fe6-68d4-4bd7-954a-e2bbb58b1f1e/2ca150cf-fbe5-4d5b-a7dc-f2dc5c6024d0/278d3e71-a9d8-40e3-a9e7-673513fdd902"
+					(reference "C50")
 					(unit 1)
 				)
@@
 		(in_pos_files yes)
 		(dnp no)
-		(property "Reference" "D15"
+		(property "Reference" "D12"
 			(at 82.55 71.12 0)
 			(show_name no)
@@
 		(instances
 			(project "PS-PrechargeBoard"
-				(path "/74d17fe6-68d4-4bd7-954a-e2bbb58b1f1e/2ca150cf-fbe5-4d5b-a7dc-f2dc5c6024d0/2a3ef9c4-dfbd-4c37-804f-440ab95d2b69"
-					(reference "D15")
+				(path "/74d17fe6-68d4-4bd7-954a-e2bbb58b1f1e/2ca150cf-fbe5-4d5b-a7dc-f2dc5c6024d0/278d3e71-a9d8-40e3-a9e7-673513fdd902"
+					(reference "D12")
 					(unit 1)
 				)

Commit message: footprints & schematic cute-ification
Parts:
- C50: value 10uF -> 10u
Changed lines of the file:
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@@
 		(dnp no)
 		(fields_autoplaced yes)
-		(property "Reference" "#FLG03"
+		(property "Reference" "#FLG02"
 			(at 71.755 30.48 0)
 			(hide yes)
@@
 			(project "PS-PrechargeBoard"
 				(path "/74d17fe6-68d4-4bd7-954a-e2bbb58b1f1e/2ca150cf-fbe5-4d5b-a7dc-f2dc5c6024d0/278d3e71-a9d8-40e3-a9e7-673513fdd902"
-					(reference "#FLG03")
+					(reference "#FLG02")
 					(unit 1)
 				)
@@
 			)
 		)
-		(property "Value" "10uF"
+		(property "Value" "10u"
 			(at 64.3128 35.687 0)
 			(show_name no)

Commit message: finished schematic & footprint
Parts:
- renumbered R70 to R69, R71 to R70
Changed lines of the file:
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@@
 		(in_pos_files yes)
 		(dnp no)
-		(property "Reference" "R70"
+		(property "Reference" "R69"
 			(at 86.106 48.26 90)
 			(show_name no)
@@
 			(project "PS-PrechargeBoard"
 				(path "/74d17fe6-68d4-4bd7-954a-e2bbb58b1f1e/2ca150cf-fbe5-4d5b-a7dc-f2dc5c6024d0/278d3e71-a9d8-40e3-a9e7-673513fdd902"
-					(reference "R70")
+					(reference "R69")
 					(unit 1)
 				)
@@
 		(in_pos_files yes)
 		(dnp no)
-		(property "Reference" "R71"
+		(property "Reference" "R70"
 			(at 93.726 48.26 90)
 			(show_name no)
@@
 			(project "PS-PrechargeBoard"
 				(path "/74d17fe6-68d4-4bd7-954a-e2bbb58b1f1e/2ca150cf-fbe5-4d5b-a7dc-f2dc5c6024d0/278d3e71-a9d8-40e3-a9e7-673513fdd902"
-					(reference "R71")
+					(reference "R70")
 					(unit 1)
 				)
@@
 		(dnp no)
 		(fields_autoplaced yes)
-		(property "Reference" "#FLG02"
+		(property "Reference" "#FLG01"
 			(at 71.755 30.48 0)
 			(hide yes)
@@
 			(project "PS-PrechargeBoard"
 				(path "/74d17fe6-68d4-4bd7-954a-e2bbb58b1f1e/2ca150cf-fbe5-4d5b-a7dc-f2dc5c6024d0/278d3e71-a9d8-40e3-a9e7-673513fdd902"
-					(reference "#FLG02")
+					(reference "#FLG01")
 					(unit 1)
 				)

Commit message: updated voltage divider to amc3311
Parts:
- renumbered R69 to R71, R70 to R72
Changed lines of the file:
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@@
 		(in_pos_files yes)
 		(dnp no)
-		(property "Reference" "R69"
+		(property "Reference" "R71"
 			(at 86.106 48.26 90)
 			(show_name no)
@@
 			(project "PS-PrechargeBoard"
 				(path "/74d17fe6-68d4-4bd7-954a-e2bbb58b1f1e/2ca150cf-fbe5-4d5b-a7dc-f2dc5c6024d0/278d3e71-a9d8-40e3-a9e7-673513fdd902"
-					(reference "R69")
+					(reference "R71")
 					(unit 1)
 				)
@@
 		(in_pos_files yes)
 		(dnp no)
-		(property "Reference" "R70"
+		(property "Reference" "R72"
 			(at 93.726 48.26 90)
 			(show_name no)
@@
 			(project "PS-PrechargeBoard"
 				(path "/74d17fe6-68d4-4bd7-954a-e2bbb58b1f1e/2ca150cf-fbe5-4d5b-a7dc-f2dc5c6024d0/278d3e71-a9d8-40e3-a9e7-673513fdd902"
-					(reference "R70")
+					(reference "R72")
 					(unit 1)
 				)

Commit message: fixed hv placement
Parts:
- removed D12: TPD2EUSB30DRTR, LHRS_ICs:TPD2EUSB30DRTR, symbol lhrs_ics:TPD2EUSB30DRTR
- added D12: SP0503BAHT, Package_TO_SOT_SMD:SOT-143, symbol lhrs_ics:SP0503BAH
Connections:
- net GND: now also D12.1 (A)
- net VBUS_IN: now also D12.4 (K)
- net USB_DM renamed USB_D-
- net USB_D-: now also D12.3 (K)
- net USB_DP renamed USB_D+
- net USB_D+: now also D12.2 (K)
Other:
- note removed: "5.5V working 7V breakdown 8V clamping"
