File: lv.kicad_sch (KiCad schematic)
At the start: 6 parts, among them J2 CAN_DEBUG_NANO_01x04, J3 CarLVPowerConnector, J4 CAN_NANO_01x05

Commit message: CAN nano & CAN debug nano
Parts:
- added J11: CAN_NANO_01x05, LHRS_Connectors:Molex_Nano-Fit_105309-xx05_1x05_P2.50mm_Vertical, symbol lhrs_connectors:CAN_NANO_01x05
- added R39: 0, Package_DIP:DIP-8_W7.62mm, symbol Device:R
- renumbered F3 to F4, J4 to J10, J3 to J8, J2 to J9, R8 to R40, R9 to R41
Connections:
- net 12V: now also J10.1 (12V), J9.1 (12V), J11.1 (12V)
- net CAN_H: now also J10.2 (CAN_H), J9.2 (CAN_H), J11.2 (CAN_H)
- net CAN_L: now also J10.3 (CAN_L), J9.3 (CAN_L), J11.3 (CAN_L)
- net GND: now also J10.4 (GND), J9.4 (GND), J11.4 (GND), R39.2
- net SHIELD: now reaches J10.5 (SHIELD)
- net SHIELD: now also J11.5 (SHIELD), R39.1
- no-connect marks 2 -> 31
Other:
- sheet 48PinMCU ports: added BOOT0, GNDA, NRST, PA10, PA15, PA3, PA4, PA5, PA6, PA7, PA8, PA9, PB0, PB1, PB10, PB11, PB12, PB13, PB14, PB15, PB2, PB3, PB4, PB7, PB9, PC13, PC14, PC15, VDDA; removed none
- note added: "CAN Nanos"
- note added: "CAN debug nano connector: passive bus monitor, powered from VIN_PROT"
- note added: "MCU"
- note removed: "MCU (test fixture) takes 3.3V"
- moved on the sheet: J10, J9

Commit message: reorganized lv
Other:
- moved on the sheet: J10, J11, J9, R39, R40, R41

Commit message: battery voltage & motor voltage
Parts:
- renumbered J10 to J5, J11 to J6, J8 to J7, J9 to J8, R39 to R14, R40 to R15, R41 to R16
Changed lines of the file:
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@@
 		(in_pos_files yes)
 		(dnp no)
-		(property "Reference" "#PWR036"
+		(property "Reference" "#PWR029"
 			(at 108.585 55.88 0)
 			(hide yes)
@@
 			(project "PS-PrechargeBoard"
 				(path "/74d17fe6-68d4-4bd7-954a-e2bbb58b1f1e/0def18ef-81e8-47ac-b719-2d9f8237a855"
-					(reference "#PWR036")
+					(reference "#PWR029")
 					(unit 1)
 				)
@@
 		(in_pos_files yes)
 		(dnp no)
-		(property "Reference" "J10"
+		(property "Reference" "J5"
 			(at 38.1 55.88 0)
 			(show_name no)
@@
 			(project "PS-PrechargeBoard"
 				(path "/74d17fe6-68d4-4bd7-954a-e2bbb58b1f1e/0def18ef-81e8-47ac-b719-2d9f8237a855"
-					(reference "J10")
+					(reference "J5")
 					(unit 1)
 				)
@@
 		(in_pos_files yes)
 		(dnp yes)
-		(property "Reference" "R39"
+		(property "Reference" "R14"
 			(at 33.02 95.25 90)
 			(show_name no)
@@
 			(project "PS-PrechargeBoard"
 				(path "/74d17fe6-68d4-4bd7-954a-e2bbb58b1f1e/0def18ef-81e8-47ac-b719-2d9f8237a855"
-					(reference "R39")
+					(reference "R14")
 					(unit 1)
 				)
@@
 		(in_pos_files yes)
 		(dnp no)
-		(property "Reference" "R40"
+		(property "Reference" "R15"
 			(at 197.485 30.48 0)
 			(show_name no)
@@
 			(project "PS-PrechargeBoard"
 				(path "/74d17fe6-68d4-4bd7-954a-e2bbb58b1f1e/0def18ef-81e8-47ac-b719-2d9f8237a855"
-					(reference "R40")
+					(reference "R15")
 					(unit 1)
 				)
@@
 		(in_pos_files yes)
 		(dnp no)
-		(property "Reference" "#PWR050"
+		(property "Reference" "#PWR035"
 			(at 210.82 41.91 0)
 			(hide yes)
@@
 			(project "PS-PrechargeBoard"
 				(path "/74d17fe6-68d4-4bd7-954a-e2bbb58b1f1e/0def18ef-81e8-47ac-b719-2d9f8237a855"
-					(reference "#PWR050")
+					(reference "#PWR035")
 					(unit 1)
 				)
@@
 		(in_pos_files yes)
 		(dnp no)
-		(property "Reference" "#PWR044"
+		(property "Reference" "#PWR021"
 			(at 17.78 71.12 0)
 			(hide yes)
@@
 			(project "PS-PrechargeBoard"
 				(path "/74d17fe6-68d4-4bd7-954a-e2bbb58b1f1e/0def18ef-81e8-47ac-b719-2d9f8237a855"
-					(reference "#PWR044")
+					(reference "#PWR021")
 					(unit 1)
 				)
@@
 		(in_pos_files yes)
 		(dnp no)
-		(property "Reference" "#FLG010"
+		(property "Reference" "#FLG05"
 			(at 57.785 24.765 0)
 			(hide yes)
@@
 			(project "PS-PrechargeBoard"
 				(path "/74d17fe6-68d4-4bd7-954a-e2bbb58b1f1e/0def18ef-81e8-47ac-b719-2d9f8237a855"
-					(reference "#FLG010")
+					(reference "#FLG05")
 					(unit 1)
 				)
@@
 		(in_pos_files yes)
 		(dnp no)
-		(property "Reference" "J9"
+		(property "Reference" "J8"
 			(at 40.64 120.65 0)
 			(show_name no)
@@
 			(project "PS-PrechargeBoard"
 				(path "/74d17fe6-68d4-4bd7-954a-e2bbb58b1f1e/0def18ef-81e8-47ac-b719-2d9f8237a855"
-					(reference "J9")
+					(reference "J8")
 					(unit 1)
 				)
@@
 		(in_pos_files yes)
 		(dnp no)
-		(property "Reference" "#PWR043"
+		(property "Reference" "#PWR024"
 			(at 60.96 137.795 0)
 			(hide yes)
@@
 			(project "PS-PrechargeBoard"
 				(path "/74d17fe6-68d4-4bd7-954a-e2bbb58b1f1e/0def18ef-81e8-47ac-b719-2d9f8237a855"
-					(reference "#PWR043")
+					(reference "#PWR024")
 					(unit 1)
 				)
@@
 		(in_pos_files yes)
 		(dnp no)
-		(property "Reference" "J8"
+		(property "Reference" "J7"
 			(at 43.815 24.765 0)
 			(show_name no)
@@
 			(project "PS-PrechargeBoard"
 				(path "/74d17fe6-68d4-4bd7-954a-e2bbb58b1f1e/0def18ef-81e8-47ac-b719-2d9f8237a855"
-					(reference "J8")
+					(reference "J7")
 					(unit 1)
 				)
@@
 		(in_pos_files yes)
 		(dnp no)
-		(property "Reference" "#FLG011"
+		(property "Reference" "#FLG06"
 			(at 57.785 30.48 0)
 			(hide yes)
@@
 			(project "PS-PrechargeBoard"
 				(path "/74d17fe6-68d4-4bd7-954a-e2bbb58b1f1e/0def18ef-81e8-47ac-b719-2d9f8237a855"
-					(reference "#FLG011")
+					(reference "#FLG06")
 					(unit 1)
 				)
@@
 		(in_pos_files yes)
 		(dnp no)
-		(property "Reference" "#PWR041"
+		(property "Reference" "#PWR031"
 			(at 134.62 27.94 0)
 			(hide yes)
@@
 			(project "PS-PrechargeBoard"
 				(path "/74d17fe6-68d4-4bd7-954a-e2bbb58b1f1e/0def18ef-81e8-47ac-b719-2d9f8237a855"
-					(reference "#PWR041")
+					(reference "#PWR031")
 					(unit 1)
 				)
@@
 		(in_pos_files yes)
 		(dnp no)
-		(property "Reference" "#PWR048"
+		(property "Reference" "#PWR027"
 			(at 64.135 73.025 0)
 			(hide yes)
@@
 			(project "PS-PrechargeBoard"
 				(path "/74d17fe6-68d4-4bd7-954a-e2bbb58b1f1e/0def18ef-81e8-47ac-b719-2d9f8237a855"
-					(reference "#PWR048")
+					(reference "#PWR027")
 					(unit 1)
 				)
@@
 		(in_pos_files yes)
 		(dnp no)
-		(property "Reference" "#PWR046"
+		(property "Reference" "#PWR023"
 			(at 38.1 105.41 0)
 			(hide yes)
@@
 			(project "PS-PrechargeBoard"
 				(path "/74d17fe6-68d4-4bd7-954a-e2bbb58b1f1e/0def18ef-81e8-47ac-b719-2d9f8237a855"
-					(reference "#PWR046")
+					(reference "#PWR023")
 					(unit 1)
 				)
@@
 		(in_pos_files yes)
 		(dnp no)
-		(property "Reference" "#PWR040"
+		(property "Reference" "#PWR033"
 			(at 164.592 83.312 0)
 			(hide yes)
@@
 			(project "PS-PrechargeBoard"
 				(path "/74d17fe6-68d4-4bd7-954a-e2bbb58b1f1e/0def18ef-81e8-47ac-b719-2d9f8237a855"
-					(reference "#PWR040")
+					(reference "#PWR033")
 					(unit 1)
 				)
@@
 		(in_pos_files yes)
 		(dnp no)
-		(property "Reference" "#PWR034"
+		(property "Reference" "#PWR036"
 			(at 252.095 41.275 0)
 			(hide yes)
@@
 			(project "PS-PrechargeBoard"
 				(path "/74d17fe6-68d4-4bd7-954a-e2bbb58b1f1e/0def18ef-81e8-47ac-b719-2d9f8237a855"
-					(reference "#PWR034")
+					(reference "#PWR036")
 					(unit 1)
 				)
@@
 		(in_pos_files yes)
 		(dnp no)
-		(property "Reference" "#PWR042"
+		(property "Reference" "#PWR032"
 			(at 153.67 40.64 0)
 			(hide yes)
@@
 			(project "PS-PrechargeBoard"
 				(path "/74d17fe6-68d4-4bd7-954a-e2bbb58b1f1e/0def18ef-81e8-47ac-b719-2d9f8237a855"
-					(reference "#PWR042")
+					(reference "#PWR032")
 					(unit 1)
 				)
@@
 		(in_pos_files yes)
 		(dnp no)
-		(property "Reference" "#PWR045"
+		(property "Reference" "#PWR022"
 			(at 17.78 95.25 0)
 			(hide yes)
@@
 			(project "PS-PrechargeBoard"
 				(path "/74d17fe6-68d4-4bd7-954a-e2bbb58b1f1e/0def18ef-81e8-47ac-b719-2d9f8237a855"
-					(reference "#PWR045")
+					(reference "#PWR022")
 					(unit 1)
 				)
@@
 		(in_pos_files yes)
 		(dnp no)
-		(property "Reference" "#PWR039"
+		(property "Reference" "#PWR028"
 			(at 100.33 40.64 0)
 			(hide yes)
@@
 			(project "PS-PrechargeBoard"
 				(path "/74d17fe6-68d4-4bd7-954a-e2bbb58b1f1e/0def18ef-81e8-47ac-b719-2d9f8237a855"
-					(reference "#PWR039")
+					(reference "#PWR028")
 					(unit 1)
 				)
@@
 		(in_pos_files yes)
 		(dnp no)
-		(property "Reference" "#PWR037"
+		(property "Reference" "#PWR030"
 			(at 108.585 112.395 0)
 			(hide yes)
@@
 			(project "PS-PrechargeBoard"
 				(path "/74d17fe6-68d4-4bd7-954a-e2bbb58b1f1e/0def18ef-81e8-47ac-b719-2d9f8237a855"
-					(reference "#PWR037")
+					(reference "#PWR030")
 					(unit 1)
 				)
@@
 		(in_pos_files yes)
 		(dnp no)
-		(property "Reference" "#PWR038"
+		(property "Reference" "#PWR025"
 			(at 63.5 40.005 0)
 			(hide yes)
@@
 			(project "PS-PrechargeBoard"
 				(path "/74d17fe6-68d4-4bd7-954a-e2bbb58b1f1e/0def18ef-81e8-47ac-b719-2d9f8237a855"
-					(reference "#PWR038")
+					(reference "#PWR025")
 					(unit 1)
 				)
@@
 		(in_pos_files yes)
 		(dnp no)
-		(property "Reference" "#PWR035"
+		(property "Reference" "#PWR037"
 			(at 278.765 35.56 0)
 			(hide yes)
@@
 			(project "PS-PrechargeBoard"
 				(path "/74d17fe6-68d4-4bd7-954a-e2bbb58b1f1e/0def18ef-81e8-47ac-b719-2d9f8237a855"
-					(reference "#PWR035")
+					(reference "#PWR037")
 					(unit 1)
 				)
@@
 		(in_pos_files yes)
 		(dnp no)
-		(property "Reference" "#PWR049"
+		(property "Reference" "#PWR034"
 			(at 194.31 54.61 0)
 			(hide yes)
@@
 			(project "PS-PrechargeBoard"
 				(path "/74d17fe6-68d4-4bd7-954a-e2bbb58b1f1e/0def18ef-81e8-47ac-b719-2d9f8237a855"
-					(reference "#PWR049")
+					(reference "#PWR034")
 					(unit 1)
 				)
@@
 		(in_pos_files yes)
 		(dnp no)
-		(property "Reference" "J11"
+		(property "Reference" "J6"
 			(at 38.1 80.01 0)
 			(show_name no)
@@
 			(project "PS-PrechargeBoard"
 				(path "/74d17fe6-68d4-4bd7-954a-e2bbb58b1f1e/0def18ef-81e8-47ac-b719-2d9f8237a855"
-					(reference "J11")
+					(reference "J6")
 					(unit 1)
 				)
@@
 		(in_pos_files yes)
 		(dnp no)
-		(property "Reference" "#PWR047"
+		(property "Reference" "#PWR026"
 			(at 64.135 59.055 0)
 			(hide yes)
@@
 			(project "PS-PrechargeBoard"
 				(path "/74d17fe6-68d4-4bd7-954a-e2bbb58b1f1e/0def18ef-81e8-47ac-b719-2d9f8237a855"
-					(reference "#PWR047")
+					(reference "#PWR026")
 					(unit 1)
 				)
@@
 		(in_pos_files yes)
 		(dnp no)
-		(property "Reference" "R41"
+		(property "Reference" "R16"
 			(at 197.485 41.91 0)
 			(show_name no)
@@
 			(project "PS-PrechargeBoard"
 				(path "/74d17fe6-68d4-4bd7-954a-e2bbb58b1f1e/0def18ef-81e8-47ac-b719-2d9f8237a855"
-					(reference "R41")
-					(unit 1)
-				)
+					(reference "R16")
+					(unit 1)
+				)

Commit message: mini review notes
Other:
- note added: "CubeMX to check which works for RX and TX"
- note added: "adjust to work with it placed and not placed"
- note added: "could use 5V power instead of label"
- note added: "dis bps CAN"
- note added: "dnp buck and mux"
- note added: "no need for first box, put F4 to CAN Nanos"
- note added: "pair TX and RX"
- moved on the sheet: F4

Commit message: fixed lv
Parts:
- added F5: 2A, LHRS_Power:Fuse-3557-2, symbol lhrs_power:Fuse_3557_2
- J7: now not fitted
- renumbered J6 to J5, J5 to J6
Connections:
- net 12V: no longer J6.1 (12V)
- net VIN_FUSED: now also F4.1, F5.2; no longer F4.2
- net at J7.1 (+12V): now also F5.1; no longer F4.1
- new net: F4.2, J6.1 (12V)
Other:
- note added: "Car LV connector, BPS CAN (12V, GND) with 2A fuse"
- note added: "PB5 and PB6 are general-purpose input/output pins (would be set to CAN) PB5: FDCAN2_RX (AF9), recieves CAN PB6: FDCAN2_TX (AF9), transmit CAN"
- note removed: "Car LV connector (12V, GND) with 2A fuse"
- note removed: "CubeMX to check which works for RX and TX"
- note removed: "adjust to work with it placed and not placed"
- note removed: "could use 5V power instead of label"
- note removed: "dis bps CAN"
- note removed: "dnp buck and mux"
- note removed: "no need for first box, put F4 to CAN Nanos"
- note removed: "pair TX and RX"
- moved on the sheet: J5, J6, J8, R14, R15, R16

Commit message: shifted hierarchical sheets
Parts:
- removed F5: 2A, LHRS_Power:Fuse-3557-2, symbol lhrs_power:Fuse_3557_2
- removed J7: CarLVPowerConnector, LHRS_Connectors:Molex_Nano-Fit_105309-xx02_1x02_P2.50mm_Vertical, symbol lhrs_connectors:CarLVPowerConnector
- J5: value CAN_NANO_01x05 -> CAN_OUT
- J6: value CAN_NANO_01x05 -> CAN_IN
Connections:
- net 12V: no longer J8.1 (12V)
- net VIN_PREFUSE: now reaches F4.2, J6.1 (12V)
- net VIN_PREFUSE: now also J8.1 (12V)
- no-connect marks 31 -> 29
Other:
- note removed: "Car LV connector, BPS CAN (12V, GND) with 2A fuse"
- moved on the sheet: F4, J5, J6, J8, R14, R15, R16
