File: 48PinMCU.kicad_sch (KiCad schematic)
At the start: 34 parts

Commit message: CAN nano & CAN debug nano
Parts:
- gave numbers to parts that had none: 34

Commit message: battery voltage & motor voltage
Parts:
- renumbered C1 to C28, C2 to C29, C3 to C30, C4 to C31, C5 to C32, C6 to C33, C7 to C34, C8 to C35, C9 to C36, C10 to C37, C11 to C38, C12 to C39, C13 to C40, C14 to C41, C15 to C42, D1 to D7, D2 to D8, D3 to D9, J2 to J10, J1 to J9, R1 to R26, R2 to R27, R3 to R28, R4 to R29, R5 to R30, R6 to R31, R7 to R32, R8 to R33, U1 to U7

Commit message: mini review notes
Parts:
- renumbered D8 to D10, D9 to D11, D7 to D9
Changed lines of the file:
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@@
 		(dnp no)
 		(fields_autoplaced yes)
-		(property "Reference" "D8"
+		(property "Reference" "D10"
 			(at 238.76 101.5999 90)
 			(show_name no)
@@
 			(project "PS-PrechargeBoard"
 				(path "/74d17fe6-68d4-4bd7-954a-e2bbb58b1f1e/0def18ef-81e8-47ac-b719-2d9f8237a855/02a41495-882b-4810-b33b-fbf874cacbbd"
-					(reference "D8")
+					(reference "D10")
 					(unit 1)
 				)
@@
 		(dnp no)
 		(fields_autoplaced yes)
-		(property "Reference" "D7"
+		(property "Reference" "D9"
 			(at 194.31 142.2399 90)
 			(show_name no)
@@
 			(project "PS-PrechargeBoard"
 				(path "/74d17fe6-68d4-4bd7-954a-e2bbb58b1f1e/0def18ef-81e8-47ac-b719-2d9f8237a855/02a41495-882b-4810-b33b-fbf874cacbbd"
-					(reference "D7")
+					(reference "D9")
 					(unit 1)
 				)
@@
 		(dnp no)
 		(fields_autoplaced yes)
-		(property "Reference" "D9"
+		(property "Reference" "D11"
 			(at 261.62 103.1874 90)
 			(show_name no)
@@
 			(project "PS-PrechargeBoard"
 				(path "/74d17fe6-68d4-4bd7-954a-e2bbb58b1f1e/0def18ef-81e8-47ac-b719-2d9f8237a855/02a41495-882b-4810-b33b-fbf874cacbbd"
-					(reference "D9")
+					(reference "D11")
 					(unit 1)
 				)
