File: 48PinMCU.kicad_sch (KiCad schematic)
At the start: 34 parts, among them J7 SWD_Header, J8 SWD, SW1 Reset, SW2 SW_SPDT, U10 STM32G473CETx, Y1 Crystal

Commit message: final schematic REV-A?
Parts:
- renumbered C57 to C47, C58 to C48, C59 to C49, C60 to C50, C61 to C51, C62 to C52, C63 to C53, C64 to C54, C65 to C55, C66 to C56, C67 to C57, C68 to C58, C69 to C59, C70 to C60, C71 to C61, D13 to D15, D14 to D16, D15 to D17, R57 to R62, R58 to R63, R59 to R64, R60 to R65, R61 to R66, R62 to R67, R63 to R68, R64 to R69, U10 to U5
Changed lines of the file:
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@@
 		(dnp no)
 		(fields_autoplaced yes)
-		(property "Reference" "C65"
+		(property "Reference" "C55"
 			(at 204.597 57.4039 0)
 			(show_name no)
@@
 			(project "PS-PrechargeBoard"
 				(path "/74d17fe6-68d4-4bd7-954a-e2bbb58b1f1e/00a9aff9-854f-4fe5-b1cf-85d3d4e30c03"
-					(reference "C65")
+					(reference "C55")
 					(unit 1)
 				)
@@
 		(in_pos_files yes)
 		(dnp no)
-		(property "Reference" "R59"
+		(property "Reference" "R64"
 			(at 183.388 154.686 0)
 			(show_name no)
@@
 			(project "PS-PrechargeBoard"
 				(path "/74d17fe6-68d4-4bd7-954a-e2bbb58b1f1e/00a9aff9-854f-4fe5-b1cf-85d3d4e30c03"
-					(reference "R59")
+					(reference "R64")
 					(unit 1)
 				)
@@
 		(dnp no)
 		(fields_autoplaced yes)
-		(property "Reference" "R58"
+		(property "Reference" "R63"
 			(at 180.848 96.0119 0)
 			(show_name no)
@@
 			(project "PS-PrechargeBoard"
 				(path "/74d17fe6-68d4-4bd7-954a-e2bbb58b1f1e/00a9aff9-854f-4fe5-b1cf-85d3d4e30c03"
-					(reference "R58")
+					(reference "R63")
 					(unit 1)
 				)
@@
 		(dnp no)
 		(fields_autoplaced yes)
-		(property "Reference" "D14"
+		(property "Reference" "D16"
 			(at 238.76 101.5999 90)
 			(show_name no)
@@
 			(project "PS-PrechargeBoard"
 				(path "/74d17fe6-68d4-4bd7-954a-e2bbb58b1f1e/00a9aff9-854f-4fe5-b1cf-85d3d4e30c03"
-					(reference "D14")
+					(reference "D16")
 					(unit 1)
 				)
@@
 		(in_pos_files yes)
 		(dnp no)
-		(property "Reference" "U10"
+		(property "Reference" "U5"
 			(at 88.392 73.66 0)
 			(hide yes)
@@
 			(project "PS-PrechargeBoard"
 				(path "/74d17fe6-68d4-4bd7-954a-e2bbb58b1f1e/00a9aff9-854f-4fe5-b1cf-85d3d4e30c03"
-					(reference "U10")
+					(reference "U5")
 					(unit 1)
 				)
@@
 		(in_pos_files yes)
 		(dnp no)
-		(property "Reference" "C70"
+		(property "Reference" "C60"
 			(at 247.142 32.258 0)
 			(show_name no)
@@
 			(project "PS-PrechargeBoard"
 				(path "/74d17fe6-68d4-4bd7-954a-e2bbb58b1f1e/00a9aff9-854f-4fe5-b1cf-85d3d4e30c03"
-					(reference "C70")
+					(reference "C60")
 					(unit 1)
 				)
@@
 		(dnp no)
 		(fields_autoplaced yes)
-		(property "Reference" "C63"
+		(property "Reference" "C53"
 			(at 189.992 57.4039 0)
 			(show_name no)
@@
 			(project "PS-PrechargeBoard"
 				(path "/74d17fe6-68d4-4bd7-954a-e2bbb58b1f1e/00a9aff9-854f-4fe5-b1cf-85d3d4e30c03"
-					(reference "C63")
+					(reference "C53")
 					(unit 1)
 				)
@@
 		(in_pos_files yes)
 		(dnp no)
-		(property "Reference" "C62"
+		(property "Reference" "C52"
 			(at 185.166 33.02 0)
 			(show_name no)
@@
 			(project "PS-PrechargeBoard"
 				(path "/74d17fe6-68d4-4bd7-954a-e2bbb58b1f1e/00a9aff9-854f-4fe5-b1cf-85d3d4e30c03"
-					(reference "C62")
+					(reference "C52")
 					(unit 1)
 				)
@@
 		(dnp no)
 		(fields_autoplaced yes)
-		(property "Reference" "C59"
+		(property "Reference" "C49"
 			(at 174.752 57.4039 0)
 			(show_name no)
@@
 			(project "PS-PrechargeBoard"
 				(path "/74d17fe6-68d4-4bd7-954a-e2bbb58b1f1e/00a9aff9-854f-4fe5-b1cf-85d3d4e30c03"
-					(reference "C59")
+					(reference "C49")
 					(unit 1)
 				)
@@
 		(dnp no)
 		(fields_autoplaced yes)
-		(property "Reference" "C71"
+		(property "Reference" "C61"
 			(at 257.937 57.277 0)
 			(show_name no)
@@
 			(project "PS-PrechargeBoard"
 				(path "/74d17fe6-68d4-4bd7-954a-e2bbb58b1f1e/00a9aff9-854f-4fe5-b1cf-85d3d4e30c03"
-					(reference "C71")
+					(reference "C61")
 					(unit 1)
 				)
@@
 		(in_pos_files yes)
 		(dnp no)
-		(property "Reference" "C66"
+		(property "Reference" "C56"
 			(at 210.82 32.766 0)
 			(show_name no)
@@
 			(project "PS-PrechargeBoard"
 				(path "/74d17fe6-68d4-4bd7-954a-e2bbb58b1f1e/00a9aff9-854f-4fe5-b1cf-85d3d4e30c03"
-					(reference "C66")
+					(reference "C56")
 					(unit 1)
 				)
@@
 		(dnp no)
 		(fields_autoplaced yes)
-		(property "Reference" "C68"
+		(property "Reference" "C58"
 			(at 224.028 33.0199 0)
 			(show_name no)
@@
 			(project "PS-PrechargeBoard"
 				(path "/74d17fe6-68d4-4bd7-954a-e2bbb58b1f1e/00a9aff9-854f-4fe5-b1cf-85d3d4e30c03"
-					(reference "C68")
+					(reference "C58")
 					(unit 1)
 				)
@@
 		(dnp no)
 		(fields_autoplaced yes)
-		(property "Reference" "D13"
+		(property "Reference" "D15"
 			(at 194.31 142.2399 90)
 			(show_name no)
@@
 			(project "PS-PrechargeBoard"
 				(path "/74d17fe6-68d4-4bd7-954a-e2bbb58b1f1e/00a9aff9-854f-4fe5-b1cf-85d3d4e30c03"
-					(reference "D13")
+					(reference "D15")
 					(unit 1)
 				)
@@
 		(in_pos_files yes)
 		(dnp no)
-		(property "Reference" "R60"
+		(property "Reference" "R65"
 			(at 191.008 154.686 0)
 			(show_name no)
@@
 			(project "PS-PrechargeBoard"
 				(path "/74d17fe6-68d4-4bd7-954a-e2bbb58b1f1e/00a9aff9-854f-4fe5-b1cf-85d3d4e30c03"
-					(reference "R60")
+					(reference "R65")
 					(unit 1)
 				)
@@
 		(in_pos_files yes)
 		(dnp no)
-		(property "Reference" "R64"
+		(property "Reference" "R69"
 			(at 259.588 110.236 0)
 			(show_name no)
@@
 			(project "PS-PrechargeBoard"
 				(path "/74d17fe6-68d4-4bd7-954a-e2bbb58b1f1e/00a9aff9-854f-4fe5-b1cf-85d3d4e30c03"
-					(reference "R64")
+					(reference "R69")
 					(unit 1)
 				)
@@
 		(in_pos_files yes)
 		(dnp no)
-		(property "Reference" "C57"
+		(property "Reference" "C47"
 			(at 34.544 39.624 90)
 			(show_name no)
@@
 			(project "PS-PrechargeBoard"
 				(path "/74d17fe6-68d4-4bd7-954a-e2bbb58b1f1e/00a9aff9-854f-4fe5-b1cf-85d3d4e30c03"
-					(reference "C57")
+					(reference "C47")
 					(unit 1)
 				)
@@
 		(in_pos_files yes)
 		(dnp no)
-		(property "Reference" "C60"
+		(property "Reference" "C50"
 			(at 173.99 33.02 0)
 			(show_name no)
@@
 			(project "PS-PrechargeBoard"
 				(path "/74d17fe6-68d4-4bd7-954a-e2bbb58b1f1e/00a9aff9-854f-4fe5-b1cf-85d3d4e30c03"
-					(reference "C60")
+					(reference "C50")
 					(unit 1)
 				)
@@
 		(in_pos_files yes)
 		(dnp no)
-		(property "Reference" "R57"
+		(property "Reference" "R62"
 			(at 175.768 154.686 0)
 			(show_name no)
@@
 			(project "PS-PrechargeBoard"
 				(path "/74d17fe6-68d4-4bd7-954a-e2bbb58b1f1e/00a9aff9-854f-4fe5-b1cf-85d3d4e30c03"
-					(reference "R57")
+					(reference "R62")
 					(unit 1)
 				)
@@
 		(dnp no)
 		(fields_autoplaced yes)
-		(property "Reference" "D15"
+		(property "Reference" "D17"
 			(at 261.62 103.1874 90)
 			(show_name no)
@@
 			(project "PS-PrechargeBoard"
 				(path "/74d17fe6-68d4-4bd7-954a-e2bbb58b1f1e/00a9aff9-854f-4fe5-b1cf-85d3d4e30c03"
-					(reference "D15")
+					(reference "D17")
 					(unit 1)
 				)
@@
 		(in_pos_files yes)
 		(dnp no)
-		(property "Reference" "C67"
+		(property "Reference" "C57"
 			(at 217.17 56.642 0)
 			(show_name no)
@@
 			(project "PS-PrechargeBoard"
 				(path "/74d17fe6-68d4-4bd7-954a-e2bbb58b1f1e/00a9aff9-854f-4fe5-b1cf-85d3d4e30c03"
-					(reference "C67")
+					(reference "C57")
 					(unit 1)
 				)
@@
 		(in_pos_files yes)
 		(dnp no)
-		(property "Reference" "R62"
+		(property "Reference" "R67"
 			(at 226.06 149.225 90)
 			(show_name no)
@@
 			(project "PS-PrechargeBoard"
 				(path "/74d17fe6-68d4-4bd7-954a-e2bbb58b1f1e/00a9aff9-854f-4fe5-b1cf-85d3d4e30c03"
-					(reference "R62")
+					(reference "R67")
 					(unit 1)
 				)
@@
 		(in_pos_files yes)
 		(dnp no)
-		(property "Reference" "C61"
+		(property "Reference" "C51"
 			(at 169.672 106.934 0)
 			(show_name no)
@@
 			(project "PS-PrechargeBoard"
 				(path "/74d17fe6-68d4-4bd7-954a-e2bbb58b1f1e/00a9aff9-854f-4fe5-b1cf-85d3d4e30c03"
-					(reference "C61")
+					(reference "C51")
 					(unit 1)
 				)
@@
 		(in_pos_files yes)
 		(dnp no)
-		(property "Reference" "R63"
+		(property "Reference" "R68"
 			(at 248.285 101.5999 0)
 			(show_name no)
@@
 			(project "PS-PrechargeBoard"
 				(path "/74d17fe6-68d4-4bd7-954a-e2bbb58b1f1e/00a9aff9-854f-4fe5-b1cf-85d3d4e30c03"
-					(reference "R63")
+					(reference "R68")
 					(unit 1)
 				)
@@
 		(in_pos_files yes)
 		(dnp no)
-		(property "Reference" "C64"
+		(property "Reference" "C54"
 			(at 197.358 33.02 0)
 			(show_name no)
@@
 			(project "PS-PrechargeBoard"
 				(path "/74d17fe6-68d4-4bd7-954a-e2bbb58b1f1e/00a9aff9-854f-4fe5-b1cf-85d3d4e30c03"
-					(reference "C64")
+					(reference "C54")
 					(unit 1)
 				)
@@
 		(dnp no)
 		(fields_autoplaced yes)
-		(property "Reference" "C58"
+		(property "Reference" "C48"
 			(at 34.798 58.928 90)
 			(show_name no)
@@
 			(project "PS-PrechargeBoard"
 				(path "/74d17fe6-68d4-4bd7-954a-e2bbb58b1f1e/00a9aff9-854f-4fe5-b1cf-85d3d4e30c03"
-					(reference "C58")
+					(reference "C48")
 					(unit 1)
 				)
@@
 		(dnp no)
 		(fields_autoplaced yes)
-		(property "Reference" "R61"
+		(property "Reference" "R66"
 			(at 226.06 137.795 90)
 			(show_name no)
@@
 			(project "PS-PrechargeBoard"
 				(path "/74d17fe6-68d4-4bd7-954a-e2bbb58b1f1e/00a9aff9-854f-4fe5-b1cf-85d3d4e30c03"
-					(reference "R61")
+					(reference "R66")
 					(unit 1)
 				)
@@
 		(in_pos_files yes)
 		(dnp no)
-		(property "Reference" "C69"
+		(property "Reference" "C59"
 			(at 233.172 32.004 0)
 			(show_name no)
@@
 			(project "PS-PrechargeBoard"
 				(path "/74d17fe6-68d4-4bd7-954a-e2bbb58b1f1e/00a9aff9-854f-4fe5-b1cf-85d3d4e30c03"
-					(reference "C69")
+					(reference "C59")
 					(unit 1)
 				)

Commit message: AGND
Parts:
- renumbered C47 to C40, C48 to C41, C49 to C42, C50 to C43, C51 to C44, C52 to C45, C53 to C46, C54 to C47, C55 to C48, C56 to C49, C57 to C50, C58 to C51, C59 to C52, C60 to C53, C61 to C54, D15 to D13, D16 to D14, D17 to D15, J7 to J13, J8 to J14, R62 to R65, R63 to R66, R64 to R67, R65 to R68, R66 to R69, R67 to R70, R68 to R71, R69 to R72, U5 to U6
Changed lines of the file:
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@@
 		(dnp no)
 		(fields_autoplaced yes)
-		(property "Reference" "C55"
+		(property "Reference" "C48"
 			(at 204.597 57.4039 0)
 			(show_name no)
@@
 			(project "PS-PrechargeBoard"
 				(path "/74d17fe6-68d4-4bd7-954a-e2bbb58b1f1e/00a9aff9-854f-4fe5-b1cf-85d3d4e30c03"
-					(reference "C55")
+					(reference "C48")
 					(unit 1)
 				)
@@
 		(in_pos_files yes)
 		(dnp no)
-		(property "Reference" "R64"
+		(property "Reference" "R67"
 			(at 183.388 154.686 0)
 			(show_name no)
@@
 			(project "PS-PrechargeBoard"
 				(path "/74d17fe6-68d4-4bd7-954a-e2bbb58b1f1e/00a9aff9-854f-4fe5-b1cf-85d3d4e30c03"
-					(reference "R64")
+					(reference "R67")
 					(unit 1)
 				)
@@
 		(dnp no)
 		(fields_autoplaced yes)
-		(property "Reference" "R63"
+		(property "Reference" "R66"
 			(at 180.848 96.0119 0)
 			(show_name no)
@@
 			(project "PS-PrechargeBoard"
 				(path "/74d17fe6-68d4-4bd7-954a-e2bbb58b1f1e/00a9aff9-854f-4fe5-b1cf-85d3d4e30c03"
-					(reference "R63")
+					(reference "R66")
 					(unit 1)
 				)
@@
 		(dnp no)
 		(fields_autoplaced yes)
-		(property "Reference" "D16"
+		(property "Reference" "D14"
 			(at 238.76 101.5999 90)
 			(show_name no)
@@
 			(project "PS-PrechargeBoard"
 				(path "/74d17fe6-68d4-4bd7-954a-e2bbb58b1f1e/00a9aff9-854f-4fe5-b1cf-85d3d4e30c03"
-					(reference "D16")
+					(reference "D14")
 					(unit 1)
 				)
@@
 		(in_pos_files yes)
 		(dnp no)
-		(property "Reference" "U5"
+		(property "Reference" "U6"
 			(at 88.392 73.66 0)
 			(hide yes)
@@
 			(project "PS-PrechargeBoard"
 				(path "/74d17fe6-68d4-4bd7-954a-e2bbb58b1f1e/00a9aff9-854f-4fe5-b1cf-85d3d4e30c03"
-					(reference "U5")
+					(reference "U6")
 					(unit 1)
 				)
@@
 		(in_pos_files yes)
 		(dnp no)
-		(property "Reference" "J7"
+		(property "Reference" "J13"
 			(at 259.334 135.89 0)
 			(show_name no)
@@
 			(project "PS-PrechargeBoard"
 				(path "/74d17fe6-68d4-4bd7-954a-e2bbb58b1f1e/00a9aff9-854f-4fe5-b1cf-85d3d4e30c03"
-					(reference "J7")
+					(reference "J13")
 					(unit 1)
 				)
@@
 		(in_pos_files yes)
 		(dnp no)
-		(property "Reference" "C60"
+		(property "Reference" "C53"
 			(at 247.142 32.258 0)
 			(show_name no)
@@
 			(project "PS-PrechargeBoard"
 				(path "/74d17fe6-68d4-4bd7-954a-e2bbb58b1f1e/00a9aff9-854f-4fe5-b1cf-85d3d4e30c03"
-					(reference "C60")
+					(reference "C53")
 					(unit 1)
 				)
@@
 		(dnp no)
 		(fields_autoplaced yes)
-		(property "Reference" "C53"
+		(property "Reference" "C46"
 			(at 189.992 57.4039 0)
 			(show_name no)
@@
 			(project "PS-PrechargeBoard"
 				(path "/74d17fe6-68d4-4bd7-954a-e2bbb58b1f1e/00a9aff9-854f-4fe5-b1cf-85d3d4e30c03"
-					(reference "C53")
+					(reference "C46")
 					(unit 1)
 				)
@@
 		(in_pos_files yes)
 		(dnp no)
-		(property "Reference" "C52"
+		(property "Reference" "C45"
 			(at 185.166 33.02 0)
 			(show_name no)
@@
 			(project "PS-PrechargeBoard"
 				(path "/74d17fe6-68d4-4bd7-954a-e2bbb58b1f1e/00a9aff9-854f-4fe5-b1cf-85d3d4e30c03"
-					(reference "C52")
+					(reference "C45")
 					(unit 1)
 				)
@@
 		(dnp no)
 		(fields_autoplaced yes)
-		(property "Reference" "C49"
+		(property "Reference" "C42"
 			(at 174.752 57.4039 0)
 			(show_name no)
@@
 			(project "PS-PrechargeBoard"
 				(path "/74d17fe6-68d4-4bd7-954a-e2bbb58b1f1e/00a9aff9-854f-4fe5-b1cf-85d3d4e30c03"
-					(reference "C49")
+					(reference "C42")
 					(unit 1)
 				)
@@
 		(dnp no)
 		(fields_autoplaced yes)
-		(property "Reference" "C61"
+		(property "Reference" "C54"
 			(at 257.937 57.277 0)
 			(show_name no)
@@
 			(project "PS-PrechargeBoard"
 				(path "/74d17fe6-68d4-4bd7-954a-e2bbb58b1f1e/00a9aff9-854f-4fe5-b1cf-85d3d4e30c03"
-					(reference "C61")
+					(reference "C54")
 					(unit 1)
 				)
@@
 		(in_pos_files yes)
 		(dnp no)
-		(property "Reference" "C56"
+		(property "Reference" "C49"
 			(at 210.82 32.766 0)
 			(show_name no)
@@
 			(project "PS-PrechargeBoard"
 				(path "/74d17fe6-68d4-4bd7-954a-e2bbb58b1f1e/00a9aff9-854f-4fe5-b1cf-85d3d4e30c03"
-					(reference "C56")
+					(reference "C49")
 					(unit 1)
 				)
@@
 		(dnp no)
 		(fields_autoplaced yes)
-		(property "Reference" "C58"
+		(property "Reference" "C51"
 			(at 224.028 33.0199 0)
 			(show_name no)
@@
 			(project "PS-PrechargeBoard"
 				(path "/74d17fe6-68d4-4bd7-954a-e2bbb58b1f1e/00a9aff9-854f-4fe5-b1cf-85d3d4e30c03"
-					(reference "C58")
+					(reference "C51")
 					(unit 1)
 				)
@@
 		(dnp no)
 		(fields_autoplaced yes)
-		(property "Reference" "D15"
+		(property "Reference" "D13"
 			(at 194.31 142.2399 90)
 			(show_name no)
@@
 			(project "PS-PrechargeBoard"
 				(path "/74d17fe6-68d4-4bd7-954a-e2bbb58b1f1e/00a9aff9-854f-4fe5-b1cf-85d3d4e30c03"
-					(reference "D15")
+					(reference "D13")
 					(unit 1)
 				)
@@
 		(in_pos_files yes)
 		(dnp no)
-		(property "Reference" "R65"
+		(property "Reference" "R68"
 			(at 191.008 154.686 0)
 			(show_name no)
@@
 			(project "PS-PrechargeBoard"
 				(path "/74d17fe6-68d4-4bd7-954a-e2bbb58b1f1e/00a9aff9-854f-4fe5-b1cf-85d3d4e30c03"
-					(reference "R65")
+					(reference "R68")
 					(unit 1)
 				)
@@
 		(in_pos_files yes)
 		(dnp no)
-		(property "Reference" "R69"
+		(property "Reference" "R72"
 			(at 259.588 110.236 0)
 			(show_name no)
@@
 			(project "PS-PrechargeBoard"
 				(path "/74d17fe6-68d4-4bd7-954a-e2bbb58b1f1e/00a9aff9-854f-4fe5-b1cf-85d3d4e30c03"
-					(reference "R69")
+					(reference "R72")
 					(unit 1)
 				)
@@
 		(in_pos_files yes)
 		(dnp no)
-		(property "Reference" "C47"
+		(property "Reference" "C40"
 			(at 34.544 39.624 90)
 			(show_name no)
@@
 			(project "PS-PrechargeBoard"
 				(path "/74d17fe6-68d4-4bd7-954a-e2bbb58b1f1e/00a9aff9-854f-4fe5-b1cf-85d3d4e30c03"
-					(reference "C47")
+					(reference "C40")
 					(unit 1)
 				)
@@
 		(in_pos_files yes)
 		(dnp no)
-		(property "Reference" "C50"
+		(property "Reference" "C43"
 			(at 173.99 33.02 0)
 			(show_name no)
@@
 			(project "PS-PrechargeBoard"
 				(path "/74d17fe6-68d4-4bd7-954a-e2bbb58b1f1e/00a9aff9-854f-4fe5-b1cf-85d3d4e30c03"
-					(reference "C50")
+					(reference "C43")
 					(unit 1)
 				)
@@
 		(in_pos_files yes)
 		(dnp no)
-		(property "Reference" "R62"
+		(property "Reference" "R65"
 			(at 175.768 154.686 0)
 			(show_name no)
@@
 			(project "PS-PrechargeBoard"
 				(path "/74d17fe6-68d4-4bd7-954a-e2bbb58b1f1e/00a9aff9-854f-4fe5-b1cf-85d3d4e30c03"
-					(reference "R62")
+					(reference "R65")
 					(unit 1)
 				)
@@
 		(dnp no)
 		(fields_autoplaced yes)
-		(property "Reference" "D17"
+		(property "Reference" "D15"
 			(at 261.62 103.1874 90)
 			(show_name no)
@@
 			(project "PS-PrechargeBoard"
 				(path "/74d17fe6-68d4-4bd7-954a-e2bbb58b1f1e/00a9aff9-854f-4fe5-b1cf-85d3d4e30c03"
-					(reference "D17")
+					(reference "D15")
 					(unit 1)
 				)
@@
 		(in_pos_files yes)
 		(dnp no)
-		(property "Reference" "C57"
+		(property "Reference" "C50"
 			(at 217.17 56.642 0)
 			(show_name no)
@@
 			(project "PS-PrechargeBoard"
 				(path "/74d17fe6-68d4-4bd7-954a-e2bbb58b1f1e/00a9aff9-854f-4fe5-b1cf-85d3d4e30c03"
-					(reference "C57")
+					(reference "C50")
 					(unit 1)
 				)
@@
 		(in_pos_files yes)
 		(dnp no)
-		(property "Reference" "R67"
+		(property "Reference" "R70"
 			(at 226.06 149.225 90)
 			(show_name no)
@@
 			(project "PS-PrechargeBoard"
 				(path "/74d17fe6-68d4-4bd7-954a-e2bbb58b1f1e/00a9aff9-854f-4fe5-b1cf-85d3d4e30c03"
-					(reference "R67")
+					(reference "R70")
 					(unit 1)
 				)
@@
 		(in_pos_files yes)
 		(dnp no)
-		(property "Reference" "C51"
+		(property "Reference" "C44"
 			(at 169.672 106.934 0)
 			(show_name no)
@@
 			(project "PS-PrechargeBoard"
 				(path "/74d17fe6-68d4-4bd7-954a-e2bbb58b1f1e/00a9aff9-854f-4fe5-b1cf-85d3d4e30c03"
-					(reference "C51")
+					(reference "C44")
 					(unit 1)
 				)
@@
 		(in_pos_files yes)
 		(dnp no)
-		(property "Reference" "R68"
+		(property "Reference" "R71"
 			(at 248.285 101.5999 0)
 			(show_name no)
@@
 			(project "PS-PrechargeBoard"
 				(path "/74d17fe6-68d4-4bd7-954a-e2bbb58b1f1e/00a9aff9-854f-4fe5-b1cf-85d3d4e30c03"
-					(reference "R68")
+					(reference "R71")
 					(unit 1)
 				)
@@
 		(in_pos_files yes)
 		(dnp no)
-		(property "Reference" "C54"
+		(property "Reference" "C47"
 			(at 197.358 33.02 0)
 			(show_name no)
@@
 			(project "PS-PrechargeBoard"
 				(path "/74d17fe6-68d4-4bd7-954a-e2bbb58b1f1e/00a9aff9-854f-4fe5-b1cf-85d3d4e30c03"
-					(reference "C54")
+					(reference "C47")
 					(unit 1)
 				)
@@
 		(in_pos_files yes)
 		(dnp no)
-		(property "Reference" "J8"
+		(property "Reference" "J14"
 			(at 254 151.384 0)
 			(show_name no)
@@
 			(project "PS-PrechargeBoard"
 				(path "/74d17fe6-68d4-4bd7-954a-e2bbb58b1f1e/00a9aff9-854f-4fe5-b1cf-85d3d4e30c03"
-					(reference "J8")
+					(reference "J14")
 					(unit 1)
 				)
@@
 		(dnp no)
 		(fields_autoplaced yes)
-		(property "Reference" "C48"
+		(property "Reference" "C41"
 			(at 34.798 58.928 90)
 			(show_name no)
@@
 			(project "PS-PrechargeBoard"
 				(path "/74d17fe6-68d4-4bd7-954a-e2bbb58b1f1e/00a9aff9-854f-4fe5-b1cf-85d3d4e30c03"
-					(reference "C48")
+					(reference "C41")
 					(unit 1)
 				)
@@
 		(dnp no)
 		(fields_autoplaced yes)
-		(property "Reference" "R66"
+		(property "Reference" "R69"
 			(at 226.06 137.795 90)
 			(show_name no)
@@
 			(project "PS-PrechargeBoard"
 				(path "/74d17fe6-68d4-4bd7-954a-e2bbb58b1f1e/00a9aff9-854f-4fe5-b1cf-85d3d4e30c03"
-					(reference "R66")
+					(reference "R69")
 					(unit 1)
 				)
@@
 		(in_pos_files yes)
 		(dnp no)
-		(property "Reference" "C59"
+		(property "Reference" "C52"
 			(at 233.172 32.004 0)
 			(show_name no)
@@
 			(project "PS-PrechargeBoard"
 				(path "/74d17fe6-68d4-4bd7-954a-e2bbb58b1f1e/00a9aff9-854f-4fe5-b1cf-85d3d4e30c03"
-					(reference "C59")
+					(reference "C52")
 					(unit 1)
 				)
