File: 48PinMCU.kicad_sch (KiCad schematic)
At the start: 34 parts, among them J13 SWD_Header, J14 SWD, SW1 Reset, SW2 SW_SPDT, U6 STM32G473CETx, Y1 Crystal

Commit message: isolated precharge from fuse
Parts:
- renumbered C40 to C42, C41 to C43, C42 to C44, C43 to C45, C44 to C46, C45 to C47, C46 to C48, C47 to C49, C48 to C50, C49 to C51, C50 to C52, C51 to C53, C52 to C54, C53 to C55, C54 to C56, J13 to J8, J14 to J9
Changed lines of the file:
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@@
 		(dnp no)
 		(fields_autoplaced yes)
-		(property "Reference" "C48"
+		(property "Reference" "C50"
 			(at 204.597 57.4039 0)
 			(show_name no)
@@
 			(project "PS-PrechargeBoard"
 				(path "/74d17fe6-68d4-4bd7-954a-e2bbb58b1f1e/00a9aff9-854f-4fe5-b1cf-85d3d4e30c03"
-					(reference "C48")
+					(reference "C50")
 					(unit 1)
 				)
@@
 		(in_pos_files yes)
 		(dnp no)
-		(property "Reference" "J13"
+		(property "Reference" "J8"
 			(at 259.334 135.89 0)
 			(show_name no)
@@
 			(project "PS-PrechargeBoard"
 				(path "/74d17fe6-68d4-4bd7-954a-e2bbb58b1f1e/00a9aff9-854f-4fe5-b1cf-85d3d4e30c03"
-					(reference "J13")
+					(reference "J8")
 					(unit 1)
 				)
@@
 		(in_pos_files yes)
 		(dnp no)
-		(property "Reference" "C53"
+		(property "Reference" "C55"
 			(at 247.142 32.258 0)
 			(show_name no)
@@
 			(project "PS-PrechargeBoard"
 				(path "/74d17fe6-68d4-4bd7-954a-e2bbb58b1f1e/00a9aff9-854f-4fe5-b1cf-85d3d4e30c03"
-					(reference "C53")
+					(reference "C55")
 					(unit 1)
 				)
@@
 		(dnp no)
 		(fields_autoplaced yes)
-		(property "Reference" "C46"
+		(property "Reference" "C48"
 			(at 189.992 57.4039 0)
 			(show_name no)
@@
 			(project "PS-PrechargeBoard"
 				(path "/74d17fe6-68d4-4bd7-954a-e2bbb58b1f1e/00a9aff9-854f-4fe5-b1cf-85d3d4e30c03"
-					(reference "C46")
+					(reference "C48")
 					(unit 1)
 				)
@@
 		(in_pos_files yes)
 		(dnp no)
-		(property "Reference" "C45"
+		(property "Reference" "C47"
 			(at 185.166 33.02 0)
 			(show_name no)
@@
 			(project "PS-PrechargeBoard"
 				(path "/74d17fe6-68d4-4bd7-954a-e2bbb58b1f1e/00a9aff9-854f-4fe5-b1cf-85d3d4e30c03"
-					(reference "C45")
+					(reference "C47")
 					(unit 1)
 				)
@@
 		(dnp no)
 		(fields_autoplaced yes)
-		(property "Reference" "C42"
+		(property "Reference" "C44"
 			(at 174.752 57.4039 0)
 			(show_name no)
@@
 			(project "PS-PrechargeBoard"
 				(path "/74d17fe6-68d4-4bd7-954a-e2bbb58b1f1e/00a9aff9-854f-4fe5-b1cf-85d3d4e30c03"
-					(reference "C42")
+					(reference "C44")
 					(unit 1)
 				)
@@
 		(dnp no)
 		(fields_autoplaced yes)
-		(property "Reference" "C54"
+		(property "Reference" "C56"
 			(at 257.937 57.277 0)
 			(show_name no)
@@
 			(project "PS-PrechargeBoard"
 				(path "/74d17fe6-68d4-4bd7-954a-e2bbb58b1f1e/00a9aff9-854f-4fe5-b1cf-85d3d4e30c03"
-					(reference "C54")
+					(reference "C56")
 					(unit 1)
 				)
@@
 		(in_pos_files yes)
 		(dnp no)
-		(property "Reference" "C49"
+		(property "Reference" "C51"
 			(at 210.82 32.766 0)
 			(show_name no)
@@
 			(project "PS-PrechargeBoard"
 				(path "/74d17fe6-68d4-4bd7-954a-e2bbb58b1f1e/00a9aff9-854f-4fe5-b1cf-85d3d4e30c03"
-					(reference "C49")
+					(reference "C51")
 					(unit 1)
 				)
@@
 		(dnp no)
 		(fields_autoplaced yes)
-		(property "Reference" "C51"
+		(property "Reference" "C53"
 			(at 224.028 33.0199 0)
 			(show_name no)
@@
 			(project "PS-PrechargeBoard"
 				(path "/74d17fe6-68d4-4bd7-954a-e2bbb58b1f1e/00a9aff9-854f-4fe5-b1cf-85d3d4e30c03"
-					(reference "C51")
+					(reference "C53")
 					(unit 1)
 				)
@@
 		(in_pos_files yes)
 		(dnp no)
-		(property "Reference" "C40"
+		(property "Reference" "C42"
 			(at 34.544 39.624 90)
 			(show_name no)
@@
 			(project "PS-PrechargeBoard"
 				(path "/74d17fe6-68d4-4bd7-954a-e2bbb58b1f1e/00a9aff9-854f-4fe5-b1cf-85d3d4e30c03"
-					(reference "C40")
+					(reference "C42")
 					(unit 1)
 				)
@@
 		(in_pos_files yes)
 		(dnp no)
-		(property "Reference" "C43"
+		(property "Reference" "C45"
 			(at 173.99 33.02 0)
 			(show_name no)
@@
 			(project "PS-PrechargeBoard"
 				(path "/74d17fe6-68d4-4bd7-954a-e2bbb58b1f1e/00a9aff9-854f-4fe5-b1cf-85d3d4e30c03"
-					(reference "C43")
+					(reference "C45")
 					(unit 1)
 				)
@@
 		(in_pos_files yes)
 		(dnp no)
-		(property "Reference" "C50"
+		(property "Reference" "C52"
 			(at 217.17 56.642 0)
 			(show_name no)
@@
 			(project "PS-PrechargeBoard"
 				(path "/74d17fe6-68d4-4bd7-954a-e2bbb58b1f1e/00a9aff9-854f-4fe5-b1cf-85d3d4e30c03"
-					(reference "C50")
+					(reference "C52")
 					(unit 1)
 				)
@@
 		(in_pos_files yes)
 		(dnp no)
-		(property "Reference" "C44"
+		(property "Reference" "C46"
 			(at 169.672 106.934 0)
 			(show_name no)
@@
 			(project "PS-PrechargeBoard"
 				(path "/74d17fe6-68d4-4bd7-954a-e2bbb58b1f1e/00a9aff9-854f-4fe5-b1cf-85d3d4e30c03"
-					(reference "C44")
+					(reference "C46")
 					(unit 1)
 				)
@@
 		(in_pos_files yes)
 		(dnp no)
-		(property "Reference" "C47"
+		(property "Reference" "C49"
 			(at 197.358 33.02 0)
 			(show_name no)
@@
 			(project "PS-PrechargeBoard"
 				(path "/74d17fe6-68d4-4bd7-954a-e2bbb58b1f1e/00a9aff9-854f-4fe5-b1cf-85d3d4e30c03"
-					(reference "C47")
+					(reference "C49")
 					(unit 1)
 				)
@@
 		(in_pos_files yes)
 		(dnp no)
-		(property "Reference" "J14"
+		(property "Reference" "J9"
 			(at 254 151.384 0)
 			(show_name no)
@@
 			(project "PS-PrechargeBoard"
 				(path "/74d17fe6-68d4-4bd7-954a-e2bbb58b1f1e/00a9aff9-854f-4fe5-b1cf-85d3d4e30c03"
-					(reference "J14")
+					(reference "J9")
 					(unit 1)
 				)
@@
 		(dnp no)
 		(fields_autoplaced yes)
-		(property "Reference" "C41"
+		(property "Reference" "C43"
 			(at 34.798 58.928 90)
 			(show_name no)
@@
 			(project "PS-PrechargeBoard"
 				(path "/74d17fe6-68d4-4bd7-954a-e2bbb58b1f1e/00a9aff9-854f-4fe5-b1cf-85d3d4e30c03"
-					(reference "C41")
+					(reference "C43")
 					(unit 1)
 				)
@@
 		(in_pos_files yes)
 		(dnp no)
-		(property "Reference" "C52"
+		(property "Reference" "C54"
 			(at 233.172 32.004 0)
 			(show_name no)
@@
 			(project "PS-PrechargeBoard"
 				(path "/74d17fe6-68d4-4bd7-954a-e2bbb58b1f1e/00a9aff9-854f-4fe5-b1cf-85d3d4e30c03"
-					(reference "C52")
+					(reference "C54")
 					(unit 1)
 				)
