File: HV.kicad_sch (KiCad schematic)
At the start: 70 parts, among them J1 HVConnector, U1 TLV9002QDRQ1

Commit message: CAN nano & CAN debug nano
Parts:
- gave numbers to parts that had none: 52
- renumbered C2 to C43, C5 to C59, D1 to D10, J1 to J4, R1 to R22, R2 to R23, R3 to R24, R6 to R27, R7 to R28, TP6 to TP11, TP1 to TP5, TP2 to TP6, TP3 to TP8, TP4 to TP9, U1 to U6
Other:
- moved on the sheet: C40, C41, C42, C43, C44, C45, C46, C47, C48, C49, C50, C51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

Commit message: battery voltage & motor voltage
Parts:
- removed C42, C43, C47, C48, C52, C53: 1uF, symbol Device:C
- removed C45, C46, C55, C56: 100nF, symbol Device:C
- removed C49, C50: 1nF, symbol Device:C
- removed IC3, IC4: AMC1350DWVR, ActivePrecharge-RevB:SOIC127P1150X280-8N, symbol AMC1350:AMC1350DWVR
- removed R25, R26, R27, R28: R, Package_DIP:DIP-8_W7.62mm, symbol Device:R
- removed TP10: V_IN_1, symbol Connector:TestPoint
- removed TP11: V_IN_2, symbol Connector:TestPoint
- removed TP13, TP14: V+, symbol Connector:TestPoint
- removed TP15, TP16: V-, symbol Connector:TestPoint
- renumbered C40 to C1, C41 to C2, C44 to C3, C54 to C4, C51 to C5, C58 to C6, C59 to C7, C57 to C8, D10 to D1, D11 to D2, D12 to D3, J4 to J1, J5 to J2, J6 to J3, J7 to J4, R22 to R1, R35 to R10, R36 to R11, R37 to R12, R38 to R13, R23 to R2, R24 to R3, R29 to R4, R30 to R5, R31 to R6, R32 to R7, R33 to R8, R34 to R9, TP5 to TP1, TP19 to TP10, TP6 to TP2, TP7 to TP3, TP8 to TP4, TP9 to TP5, TP17 to TP6, TP12 to TP7, TP20 to TP8, TP18 to TP9, U6 to U1, U5 to U2, U7 to U3
Other:
- added sheet Battery_Voltage (Battery_Voltage.kicad_sch)
- added sheet Motor_Voltage (Motor_Voltage.kicad_sch)
- note removed: "Battery Voltage"
- note removed: "Motor Voltage"
- moved on the sheet: C4, C6, C7, R10, R11, R12, R13, R4, R5, R6, R7, R8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

Commit message: mini review notes
Parts:
- added D1, D3: RSX068MP2STR, ActivePrecharge-RevB:RSX068MP2STR, symbol Device:D_Schottky
- renumbered D1 to D2, D2 to D4, D3 to D5
Connections:
- net HV-: now also D1.1 (K); no longer F2.2
- net HVGND: now also D3.2 (A); no longer J1.2 (Pin_2)
- new net: D3.1 (K), J1.2 (Pin_2)
- new net: D1.2 (A), F2.2
Other:
- note added: "12V for relay"
- note added: "12V or 3V3 input"
- note added: "5V turn into 3V3"
- note added: "change HVGND and LVGND global labels into just a hierarchal pin"
- note added: "change icu?"
- note added: "change to relays"
- note added: "contactor design block but change resistor value for peak of whole current for fitst time vs entire"
- note added: "econimizer circuitry"
- note added: "main"
- note added: "motor"
- note added: "on notion doc relay"
- note added: "put on main"
- note added: "update sharepoint and put in lhr test points"
- moved on the sheet: C8, D4, D5, F3, J2, J3, J4, R1, R2, R3, TP1, TP10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

Commit message: fixed battery voltage & motor voltage
Other:
- sheet Battery_Voltage ports: added none; removed HV+, V1+, V1-, V_IN_1
- sheet Motor_Voltage ports: added none; removed HV+, V2+, V2-, V_IN_2

Commit message: fixed lv
Parts:
- removed TP2: HVGND, symbol Connector:TestPoint
- removed TP4: HV+, symbol Connector:TestPoint
- removed TP5: HV-, symbol Connector:TestPoint
- added TP?: HV+, TestPoint:TestPoint_Loop_D1.80mm_Drill1.0mm_Beaded, symbol lhrs_misc:Multimeter_TP
- added TP?: HV-, TestPoint:TestPoint_Loop_D1.80mm_Drill1.0mm_Beaded, symbol lhrs_misc:Multimeter_TP
- added TP? (x2): HVGND, TestPoint:TestPoint_Loop_D1.80mm_Drill1.0mm_Beaded, symbol lhrs_misc:Multimeter_TP
- renumbered D2 to D1, D1 to D2
Connections:
- net HV+: now also TP?.1
- net HV-: now also TP?.1
- net HVGND: now also TP?.1
Other:
- note removed: "change HVGND and LVGND global labels into just a hierarchal pin"
- moved on the sheet: D1, D2, D3, F1, F2, J1

Commit message: shifted hierarchical sheets
Parts:
- removed C3, C5: 10uF, symbol Device:C
- removed TP10: GND, symbol Connector:TestPoint
- removed TP6: V_OUT_1, symbol Connector:TestPoint
- removed TP7: REG_3V3, symbol Connector:TestPoint
- removed TP8: V_OUT_2, symbol Connector:TestPoint
- removed TP9: 3V3, symbol Connector:TestPoint
- removed U2: LT1963AEST-3.3#TRPBF, ActivePrecharge-RevB:VREG_LT1963AEST-3.3_TRPBF, symbol Regulator_Linear:LT1963AxST-3.3
- added C? (x2): 10u, Capacitor_SMD:C_0805_2012Metric_Pad1.18x1.45mm_HandSolder, symbol Device:C_Small
- added D?: SBA130CH-AU_R1_000A1, Diode_SMD:D_SOD-323_HandSoldering, symbol Device:D_Schottky_Small
- added TP?: V_OUT_MOT, TestPoint:TestPoint_Loop_D1.80mm_Drill1.0mm_Beaded, symbol lhrs_misc:Multimeter_TP
- added TP?: 3V3, TestPoint:TestPoint_Loop_D1.80mm_Drill1.0mm_Beaded, symbol lhrs_misc:Multimeter_TP
- added TP?: REG_3V3, TestPoint:TestPoint_Loop_D1.80mm_Drill1.0mm_Beaded, symbol lhrs_misc:Multimeter_TP
- added TP?: GND, TestPoint:TestPoint_Loop_D1.80mm_Drill1.0mm_Beaded, symbol lhrs_misc:Multimeter_TP
- added U?: MCP1826S, Package_TO_SOT_SMD:SOT-223-3_TabPin2, symbol Regulator_Linear:MCP1826S
- TP?: value HVGND -> V_OUT_BAT
Connections:
- net V_OUT_1 is gone; now on net V_OUT_BAT: C4.1, J2.7 (Pin_7), R8.2
- net 3V3: now also TP?.1
- net HVGND: now also C?.1, C?.1, U?.2 (GND)
- net ISO_5V: now also D?.2 (A)
- net LVGND: now also TP?.1
- net REG_3V3: now also C?.2, TP?.1, U?.3 (VO)
- net V_OUT_BAT: now reaches TP?.1
- net V1+ renamed BAT_V+
- net V1- renamed BAT_V-
- net V2+ renamed MOT_V+
- net V2- renamed MOT_V-
- net V_OUT_2 renamed V_OUT_MOT
- net V_OUT_MOT: now also TP?.1
- new net: C?.2, D?.1 (K), U?.1 (VI)
Other:
- sheet Battery_Voltage ports: added 3V3, BAT_V+, BAT_V-, HV+, HVGND, LVGND, REG_3V3; removed none
- sheet Motor_Voltage ports: added 3V3, HV+, HVGND, LVGND, MOT_V+, MOT_V-, REG_3V3; removed none
- note added: "HV Battery Voltage Sense (Isolated)"
- note added: "HV Motor Voltage Sense (Isolated)"
- note added: "calc use lv ldo"
- moved on the sheet: C1, C2, C4, C6, C7, C8, D4, D5, F3, J2, J3, J4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
