File: Battery_OpAmp.kicad_sch (KiCad schematic)
At the start: 10 parts

Commit message: commit work?
Other:
- note added: "make universal in hieracvrchal pin"
Changed lines of the file:
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@@
+		)
+	)
+	(text "make universal in hieracvrchal pin"
+		(exclude_from_sim no)
+		(at 83.82 52.705 0)
+		(effects
+			(font
+				(size 1.27 1.27)
+			)
 		)
 	)
