File: PS-PrechargeBoard.kicad_sch (KiCad schematic)
At the start: 26 parts, among them J1 HV_Main, J10 DEBUG_NANO, J11 MOT, J12 USB, J2 HV_Motor, J3 DIAG, J4 TX, J5 RX, J6 MAIN, J7 CAN_IN, J8 CAN_OUT, J9 PRECHARGE_CTRL

Commit message: hv/lv big schematic label
Other:
- note added: "HV"
- note added: "LV"
Changed lines of the file:
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@@
+		)
+	)
+	(text "        LV"
+		(exclude_from_sim no)
+		(at 143.51 9.906 0)
+		(effects
+			(font
+				(size 2.54 2.54)
+				(thickness 0.508)
+				(bold yes)
+			)
+			(justify left bottom)
 		)
 	)
@@
 		)
 	)
+	(text "HV        "
+		(exclude_from_sim no)
+		(at 143.51 9.906 0)
+		(effects
+			(font
+				(size 2.54 2.54)
+				(thickness 0.508)
+				(bold yes)
+			)
+			(justify right bottom)
+		)
+	)
 	(text "CAN debug nano connector: passive bus \nmonitor, powered from VIN_PROT"
 		(exclude_from_sim no)
@@
 	(polyline
 		(pts
-			(xy 144.78 10.16) (xy 144.78 200.66)
-		)
-		(stroke
+			(xy 143.51 10.16) (xy 143.51 200.279)
+		)
+		(stroke
