File: PS-PrechargeBoard.kicad_sch (KiCad schematic)
At the start: 25 parts, among them J1 HV_Main, J2 HV_Motor, J3 DIAG, J4 CAN_IN, J5 CAN_OUT, J6 DEBUG_NANO, J7 PRECHARGE_CTRL

Commit message: starting layout
Parts:
- J3, J7: footprint Connector:CUI_PD-30 -> Connector_PinHeader_2.54mm:PinHeader_1x02_P2.54mm_Vertical
- R1: footprint Package_DIP:DIP-8_W7.62mm -> Resistor_SMD:R_0603_1608Metric_Pad0.98x0.95mm_HandSolder
Changed lines of the file:
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@@
 			)
 		)
-		(property "Footprint" "Connector:CUI_PD-30"
+		(property "Footprint" "Connector_PinHeader_2.54mm:PinHeader_1x02_P2.54mm_Vertical"
 			(at 196.85 109.22 0)
 			(hide yes)
@@
 			)
 		)
-		(property "Footprint" "Package_DIP:DIP-8_W7.62mm"
+		(property "Footprint" "Resistor_SMD:R_0603_1608Metric_Pad0.98x0.95mm_HandSolder"
 			(at 237.998 31.75 90)
 			(hide yes)
@@
 			)
 		)
-		(property "Footprint" "Connector:CUI_PD-30"
+		(property "Footprint" "Connector_PinHeader_2.54mm:PinHeader_1x02_P2.54mm_Vertical"
 			(at 270.51 124.46 0)
 			(hide yes)
