File: PS-PrechargeBoard.kicad_sch (KiCad schematic)
At the start: 25 parts, among them J1 HV_Main, J2 HV_Motor, J3 DIAG, J4 CAN_IN, J5 CAN_OUT, J6 DEBUG_NANO, J7 PRECHARGE_CTRL

Commit message: fixed hv placement
Parts:
- removed TP12: AGND, TestPoint:TestPoint_Loop_D1.80mm_Drill1.0mm_Beaded, symbol lhrs_misc:Multimeter_TP
- removed TP16: GND, TestPoint:TestPoint_Loop_D1.80mm_Drill1.0mm_Beaded, symbol lhrs_misc:Multimeter_TP
- removed TP9: VDDA, TestPoint:TestPoint_Loop_D1.80mm_Drill1.0mm_Beaded, symbol lhrs_misc:Multimeter_TP
- added TP11: GND, TestPoint:TestPoint_THTPad_D3.0mm_Drill1.5mm, symbol lhrs_misc:Multimeter_TP
- TP1, TP2, TP3, TP4, TP5, TP6, TP7, TP8: footprint TestPoint:TestPoint_Loop_D1.80mm_Drill1.0mm_Beaded -> TestPoint:TestPoint_THTPad_D3.0mm_Drill1.5mm
- TP10: renamed from TP11; footprint TestPoint:TestPoint_Loop_D1.80mm_Drill1.0mm_Beaded -> TestPoint:TestPoint_THTPad_D3.0mm_Drill1.5mm
- TP12: renamed from TP13; footprint TestPoint:TestPoint_Loop_D1.80mm_Drill1.0mm_Beaded -> TestPoint:TestPoint_THTPad_D3.0mm_Drill1.5mm
- TP13: renamed from TP14; footprint TestPoint:TestPoint_Loop_D1.80mm_Drill1.0mm_Beaded -> TestPoint:TestPoint_THTPad_D3.0mm_Drill1.5mm
- TP14: renamed from TP15; footprint TestPoint:TestPoint_Loop_D1.80mm_Drill1.0mm_Beaded -> TestPoint:TestPoint_THTPad_D3.0mm_Drill1.5mm
- TP9: renamed from TP10; footprint TestPoint:TestPoint_Loop_D1.80mm_Drill1.0mm_Beaded -> TestPoint:TestPoint_THTPad_D3.0mm_Drill1.5mm
Connections:
- net GND: now also TP11.1
- no-connect marks 19 -> 21
Other:
- sheet Main_VoltageSensor ports: added none; removed AGND
- sheet Motor_VoltageSensor ports: added none; removed AGND
