File: PS-PrechargeBoard.kicad_pcb (KiCad board)
At the start: 2 copper layers, 230 parts, among them IC1 LM74502DDFR, IC2 TCAN3413DR, J1 HV_Main, J10 SWD, J2 HV_Motor, J3 DIAG, J4 CAN_IN, J5 CAN_OUT, J6 DEBUG_NANO, J7 PRECHARGE_CTRL, J8 USB_C_Receptacle_USB2.0_16P, J9 SWD_Header, K1 DE1a-12V, K2 DE1a-12V, Q1 NMOS, Q2 NMOS, Q3 PSMN012-100YS, Q4 PSMN012-100YS, SW1 Reset, SW2 SW_SPDT, U1 TLV9002QDRQ1, U4 TLV9002QDRQ1, U7 MCP1826S, U8 STM32G473CETx, Y1 Crystal

Commit message: basic layout grouping
Parts:
- moved J7 274.5 mm to (354.4, 106.1)
- moved J3 266.9 mm to (320.6, 128.7)
- moved TP14 257.8 mm to (355.7, 116.3)
- moved TP15 257.8 mm to (355.7, 120.9)
- moved TP10 226.9 mm to (320.8, 109.7)
- moved TP11 226.9 mm to (320.8, 114.4)
- moved TP12 226.9 mm to (320.8, 119.0)
- moved TP9 226.9 mm to (320.8, 105.1)
- moved C64 204.5 mm to (330.9, 104.4)
- moved C65 204.5 mm to (330.9, 106.9)
- moved C66 204.5 mm to (330.9, 109.4)
- moved C67 204.5 mm to (330.9, 111.9)
- moved C68 204.5 mm to (330.9, 114.4)
- moved C69 204.5 mm to (330.9, 116.9)
- moved D17 204.5 mm to (330.7, 131.3)
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Other:
- board text added: "CAN Debug"
- board text added: "CAN Nanos"
- board text added: "HV"
- board text added: "Isolated HV+ Sensing"
- board text added: "Isolated HV- Sensing"
- board text added: "LV"
- board text added: "LV Power"
- board text added: "MCU"
- board text added: "Main Precharge"
- board text added: "Motor Precharge"
- board text added: "Op-amp"
- board text added: "Precharge Relay"
- board text added: "Voltage Divider HV+"
- board text added: "Voltage Divider HV-"

Commit message: hv placement 1.0
Parts:
- moved R33 117.1 mm to (62.5, 90.3)
- moved R32 116.5 mm to (62.5, 78.7)
- moved R35 116.1 mm to (62.5, 117.1)
- moved R34 116.1 mm to (62.5, 104.5)
- moved D7 101.6 mm to (50.9, 99.4)
- moved D5 99.6 mm to (50.9, 95.4)
- moved R45 99.1 mm to (92.0, 104.0), turned to 180 degrees
- moved J2 98.7 mm to (24.2, 99.9), turned to 180 degrees
- moved C23 98.0 mm to (98.5, 104.0), turned to 180 degrees
- moved R44 93.9 mm to (91.3, 102.1)
- moved R61 93.8 mm to (119.9, 97.7)
- moved R43 89.8 mm to (91.3, 99.8)
- moved D6 89.3 mm to (31.7, 97.4)
- moved R3 89.0 mm to (62.4, 34.2)
- moved R5 88.8 mm to (62.4, 59.9)
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Other:
- board text added: "Main Isolated HV+ Sensing"
- board text added: "Main Isolated HV- Sensing"
- board text added: "Motor Isolated HV+ Sensing"
- board text added: "Motor Isolated HV- Sensing"
- board text removed: "HV"
- board text removed: "Isolated HV+ Sensing"
- board text removed: "Isolated HV- Sensing"
- board text removed: "LV"
- board text removed: "Voltage Divider HV+"
- board text removed: "Voltage Divider HV-"

Commit message: hv placement 1.1
Parts:
- TP5: value MAIN_HV- -> MOT_HV-
- moved TP1 30.4 mm to (49.3, 81.7)
- moved TP5 30.3 mm to (49.3, 113.2)
- moved TP4 26.9 mm to (49.3, 57.0)
- moved TP3 19.7 mm to (73.0, 18.5)
- moved C23 3.86 mm to (94.6, 103.9)
- moved C29 3.86 mm to (94.6, 81.1)
- moved C30 3.86 mm to (94.6, 82.6)
- moved C32 3.86 mm to (109.8, 83.8)
- moved C37 3.86 mm to (94.6, 100.9)
- moved C38 3.86 mm to (94.6, 102.4)
- moved R36 3.86 mm to (87.4, 75.3)
- moved R37 3.86 mm to (87.4, 77.6)
- moved R38 3.86 mm to (87.4, 79.9)
- moved R39 3.86 mm to (87.4, 82.2)
- moved R42 3.86 mm to (87.4, 97.4)
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
Commit message: op-amp & precharge relay placement
Parts:
- moved TP7 151.6 mm to (90.8, 73.9)
- moved Q2 130.3 mm to (117.4, 88.0)
- moved K2 129.3 mm to (90.8, 92.0)
- moved D8 128.4 mm to (87.1, 88.2)
- moved C57 124.1 mm to (253.9, 42.8)
- moved C61 124.1 mm to (253.9, 50.4)
- moved C70 124.1 mm to (262.6, 42.8)
- moved C71 124.1 mm to (262.6, 45.4)
- moved FB1 124.1 mm to (262.6, 47.9)
- moved FB2 124.1 mm to (262.6, 50.4)
- moved J9 124.1 mm to (274.6, 45.9)
- moved R73 124.1 mm to (262.6, 52.9)
- moved R74 124.1 mm to (262.6, 55.4)
- moved TP14 124.1 mm to (283.1, 54.8)
- moved TP15 124.1 mm to (283.1, 59.4)
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Other:
- board text added: "Main Op-amp"
- board text added: "Main Precharge Relay"
- board text added: "Motor Op-amp"
- board text added: "Motor Precharge Relay"
- board text removed: "Op-amp"
- board text removed: "Precharge Relay"

Commit message: pp placement
Parts:
- moved F1 110.0 mm to (219.7, -40.3), turned to 180 degrees
- moved TP13 107.9 mm to (213.0, -45.9)
- moved R1 98.5 mm to (228.3, -35.7), turned to 180 degrees
- moved TP8 89.1 mm to (213.0, -34.6), turned to 180 degrees
- moved J5 85.5 mm to (232.3, -36.5)
- moved J4 83.4 mm to (232.3, -53.9)
- moved D10 82.5 mm to (165.6, 47.4), turned to 180 degrees
- moved IC1 78.5 mm to (177.2, 47.4)
- moved R68 75.7 mm to (177.5, 43.4), turned to 180 degrees
- moved R67 75.1 mm to (177.5, 41.9), turned to 180 degrees
- moved R63 74.6 mm to (177.5, 37.3)
- moved R66 74.5 mm to (177.5, 40.4)
- moved R65 74.0 mm to (177.5, 38.9), turned to 180 degrees
- moved TP16 72.8 mm to (225.3, -45.9)
- moved R62 70.1 mm to (184.9, 47.5), turned to 180 degrees
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Other:
- board text added: "Main Fuse"
- board text added: "Motor Fuse"
- board text added: "Power Protection"
- board text removed: "LV Power"
- board text removed: "Main Precharge Relay"
- board text removed: "Motor Precharge Relay"
