File: Fused_Relay.kicad_sch (KiCad schematic)
At the start: 9 parts

Commit message: footprints & schematic cute-ification
Parts:
- D1, D2, D3: footprint ActivePrecharge-RevB:RSX068MP2STR -> Diode_SMD:D_SOD-123
- F2, F3: footprint (none) -> LHRS_Power:HV-Fuse
Changed lines of the file:
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@@
 			)
 		)
-		(property "Footprint" ""
+		(property "Footprint" "LHRS_Power:HV-Fuse"
 			(at 38.1 55.118 90)
 			(hide yes)
@@
 			)
 		)
-		(property "Footprint" "ActivePrecharge-RevB:RSX068MP2STR"
+		(property "Footprint" "Diode_SMD:D_SOD-123"
 			(at 48.26 39.37 0)
 			(hide yes)
@@
 			)
 		)
-		(property "Footprint" ""
+		(property "Footprint" "LHRS_Power:HV-Fuse"
 			(at 38.1 25.908 90)
 			(hide yes)
@@
 			)
 		)
-		(property "Footprint" "ActivePrecharge-RevB:RSX068MP2STR"
+		(property "Footprint" "Diode_SMD:D_SOD-123"
 			(at 48.26 24.13 0)
 			(hide yes)
@@
 			)
 		)
-		(property "Footprint" "ActivePrecharge-RevB:RSX068MP2STR"
+		(property "Footprint" "Diode_SMD:D_SOD-123"
 			(at 48.26 53.34 0)
 			(hide yes)

Commit message: finished schematic & footprint
Parts:
- R2: renamed from R3; footprint PWR263S-35-3300F:RES_PWR263S-35-3300F -> Precharge_Board:RES_PWR263S-35-3300F
- R3: renamed from R4; footprint PWR263S-35-3300F:RES_PWR263S-35-3300F -> Precharge_Board:RES_PWR263S-35-3300F
- R4: renamed from R5; footprint PWR263S-35-3300F:RES_PWR263S-35-3300F -> Precharge_Board:RES_PWR263S-35-3300F
- R5: renamed from R6; footprint PWR263S-35-3300F:RES_PWR263S-35-3300F -> Precharge_Board:RES_PWR263S-35-3300F
Changed lines of the file:
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@@
 		(in_pos_files yes)
 		(dnp no)
-		(property "Reference" "R3"
+		(property "Reference" "R2"
 			(at 100.33 23.622 0)
 			(show_name no)
@@
 			)
 		)
-		(property "Footprint" "PWR263S-35-3300F:RES_PWR263S-35-3300F"
+		(property "Footprint" "Precharge_Board:RES_PWR263S-35-3300F"
 			(at 100.33 26.67 0)
 			(hide yes)
@@
 			(project "PS-PrechargeBoard"
 				(path "/74d17fe6-68d4-4bd7-954a-e2bbb58b1f1e/90c6c4b7-1465-4e8f-80ba-ec6b0750446b"
-					(reference "R33")
+					(reference "R32")
 					(unit 1)
 				)
 				(path "/74d17fe6-68d4-4bd7-954a-e2bbb58b1f1e/9d2e20d2-bc37-4993-8fa8-5a82459dba6b"
-					(reference "R3")
+					(reference "R2")
 					(unit 1)
 				)
@@
 		(in_pos_files yes)
 		(dnp yes)
-		(property "Reference" "R6"
+		(property "Reference" "R5"
 			(at 100.33 57.912 0)
 			(show_name no)
@@
 			)
 		)
-		(property "Footprint" "PWR263S-35-3300F:RES_PWR263S-35-3300F"
+		(property "Footprint" "Precharge_Board:RES_PWR263S-35-3300F"
 			(at 100.33 60.96 0)
 			(hide yes)
@@
 			(project "PS-PrechargeBoard"
 				(path "/74d17fe6-68d4-4bd7-954a-e2bbb58b1f1e/90c6c4b7-1465-4e8f-80ba-ec6b0750446b"
-					(reference "R36")
+					(reference "R35")
 					(unit 1)
 				)
 				(path "/74d17fe6-68d4-4bd7-954a-e2bbb58b1f1e/9d2e20d2-bc37-4993-8fa8-5a82459dba6b"
-					(reference "R6")
+					(reference "R5")
 					(unit 1)
 				)
@@
 		(in_pos_files yes)
 		(dnp no)
-		(property "Reference" "R5"
+		(property "Reference" "R4"
 			(at 100.33 46.482 0)
 			(show_name no)
@@
 			)
 		)
-		(property "Footprint" "PWR263S-35-3300F:RES_PWR263S-35-3300F"
+		(property "Footprint" "Precharge_Board:RES_PWR263S-35-3300F"
 			(at 100.33 49.53 0)
 			(hide yes)
@@
 			(project "PS-PrechargeBoard"
 				(path "/74d17fe6-68d4-4bd7-954a-e2bbb58b1f1e/90c6c4b7-1465-4e8f-80ba-ec6b0750446b"
-					(reference "R35")
+					(reference "R34")
 					(unit 1)
 				)
 				(path "/74d17fe6-68d4-4bd7-954a-e2bbb58b1f1e/9d2e20d2-bc37-4993-8fa8-5a82459dba6b"
-					(reference "R5")
+					(reference "R4")
 					(unit 1)
 				)
@@
 		(in_pos_files yes)
 		(dnp no)
-		(property "Reference" "R4"
+		(property "Reference" "R3"
 			(at 100.33 35.052 0)
 			(show_name no)
@@
 			)
 		)
-		(property "Footprint" "PWR263S-35-3300F:RES_PWR263S-35-3300F"
+		(property "Footprint" "Precharge_Board:RES_PWR263S-35-3300F"
 			(at 100.33 38.1 0)
 			(hide yes)
@@
 			(project "PS-PrechargeBoard"
 				(path "/74d17fe6-68d4-4bd7-954a-e2bbb58b1f1e/90c6c4b7-1465-4e8f-80ba-ec6b0750446b"
-					(reference "R34")
+					(reference "R33")
 					(unit 1)
 				)
 				(path "/74d17fe6-68d4-4bd7-954a-e2bbb58b1f1e/9d2e20d2-bc37-4993-8fa8-5a82459dba6b"
-					(reference "R4")
-					(unit 1)
-				)
+					(reference "R3")
+					(unit 1)
+				)

Commit message: restored pp placement
Parts:
- removed R5: 50, Precharge_Board:RES_PWR263S-35-3300F, symbol Precharge-R:PWR263S-35-3300F
Changed lines of the file:
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@@
 	(rectangle
 		(start 71.755 13.335)
-		(end 128.27 66.675)
+		(end 128.27 61.595)
 		(stroke
 			(width 0)
@@
 	(text "Resistor (R) = 50 ohms :\nBattery Vmax: 135V\nTarget Time (Tmax): 0.25 s\nPrecharge Level: 95%\nSystem Capacitance (C): 1420µF\n\nFuse = 5A :\nPeak Inrush Current: 2.7A\n3A fuse too close to 2.7A peak"
 		(exclude_from_sim no)
-		(at 71.12 68.58 0)
+		(at 72.136 63.246 0)
 		(effects
 			(font
@@
 	)
 	(junction
-		(at 110.49 60.96)
+		(at 110.49 38.1)
 		(diameter 0)
 		(color 0 0 0 0)
@@
 	)
 	(junction
-		(at 88.9 50.8)
-		(diameter 0)
-		(color 0 0 0 0)
-	)
-	(junction
-		(at 110.49 38.1)
-		(diameter 0)
-		(color 0 0 0 0)
-	)
-	(junction
 		(at 88.9 27.94)
 		(diameter 0)
@@
 	(wire
 		(pts
-			(xy 110.49 38.1) (xy 110.49 60.96)
+			(xy 83.82 25.4) (xy 90.17 25.4)
 		)
 		(stroke
@@
 	(wire
 		(pts
-			(xy 83.82 25.4) (xy 90.17 25.4)
+			(xy 83.82 27.94) (xy 88.9 27.94)
 		)
 		(stroke
@@
 	(wire
 		(pts
-			(xy 83.82 27.94) (xy 88.9 27.94)
+			(xy 88.9 27.94) (xy 90.17 27.94)
 		)
 		(stroke
@@
 	(wire
 		(pts
-			(xy 88.9 27.94) (xy 90.17 27.94)
+			(xy 52.07 53.34) (xy 57.15 53.34)
 		)
 		(stroke
@@
 	(wire
 		(pts
-			(xy 52.07 53.34) (xy 57.15 53.34)
+			(xy 33.02 24.13) (xy 33.02 34.29)
 		)
 		(stroke
@@
 	(wire
 		(pts
-			(xy 33.02 24.13) (xy 33.02 34.29)
+			(xy 41.91 53.34) (xy 44.45 53.34)
 		)
 		(stroke
@@
 	(wire
 		(pts
-			(xy 41.91 53.34) (xy 44.45 53.34)
+			(xy 110.49 26.67) (xy 110.49 38.1)
 		)
 		(stroke
@@
 	(wire
 		(pts
-			(xy 110.49 26.67) (xy 110.49 38.1)
+			(xy 88.9 39.37) (xy 90.17 39.37)
 		)
 		(stroke
@@
 	(wire
 		(pts
-			(xy 88.9 39.37) (xy 90.17 39.37)
+			(xy 110.49 49.53) (xy 115.57 49.53)
 		)
 		(stroke
@@
 	(wire
 		(pts
-			(xy 110.49 60.96) (xy 115.57 60.96)
+			(xy 44.45 24.13) (xy 41.91 24.13)
 		)
 		(stroke
@@
 	(wire
 		(pts
-			(xy 88.9 62.23) (xy 90.17 62.23)
+			(xy 34.29 24.13) (xy 33.02 24.13)
 		)
 		(stroke
@@
 	(wire
 		(pts
-			(xy 83.82 59.69) (xy 90.17 59.69)
+			(xy 88.9 39.37) (xy 88.9 50.8)
 		)
 		(stroke
@@
 	(wire
 		(pts
-			(xy 44.45 24.13) (xy 41.91 24.13)
+			(xy 83.82 48.26) (xy 90.17 48.26)
 		)
 		(stroke
@@
 	(wire
 		(pts
-			(xy 34.29 24.13) (xy 33.02 24.13)
+			(xy 83.82 36.83) (xy 90.17 36.83)
 		)
 		(stroke
@@
 	(wire
 		(pts
-			(xy 88.9 50.8) (xy 88.9 62.23)
+			(xy 52.07 39.37) (xy 57.15 39.37)
 		)
 		(stroke
@@
 	(wire
 		(pts
-			(xy 88.9 39.37) (xy 88.9 50.8)
+			(xy 34.29 53.34) (xy 33.02 53.34)
 		)
 		(stroke
@@
 	(wire
 		(pts
-			(xy 83.82 48.26) (xy 90.17 48.26)
+			(xy 88.9 50.8) (xy 90.17 50.8)
 		)
 		(stroke
@@
 	(wire
 		(pts
-			(xy 83.82 36.83) (xy 90.17 36.83)
+			(xy 88.9 27.94) (xy 88.9 39.37)
 		)
 		(stroke
@@
 	(wire
 		(pts
-			(xy 52.07 39.37) (xy 57.15 39.37)
+			(xy 33.02 53.34) (xy 33.02 43.18)
 		)
 		(stroke
@@
 	(wire
 		(pts
-			(xy 34.29 53.34) (xy 33.02 53.34)
+			(xy 52.07 24.13) (xy 57.15 24.13)
 		)
 		(stroke
@@
 	(wire
 		(pts
-			(xy 88.9 50.8) (xy 90.17 50.8)
-		)
-		(stroke
-			(width 0)
-			(type default)
-		)
-	)
-	(wire
-		(pts
-			(xy 88.9 27.94) (xy 88.9 39.37)
-		)
-		(stroke
-			(width 0)
-			(type default)
-		)
-	)
-	(wire
-		(pts
-			(xy 33.02 53.34) (xy 33.02 43.18)
-		)
-		(stroke
-			(width 0)
-			(type default)
-		)
-	)
-	(wire
-		(pts
-			(xy 52.07 24.13) (xy 57.15 24.13)
+			(xy 110.49 38.1) (xy 110.49 49.53)
 		)
 		(stroke
@@
 	)
 	(label "RESISTOR"
-		(at 83.82 59.69 180)
-		(effects
-			(font
-				(size 1.27 1.27)
-			)
-			(justify right bottom)
-		)
-	)
-	(label "RESISTOR"
 		(at 83.82 48.26 180)
 		(effects
@@
 			)
 			(justify right bottom)
+		)
+	)
+	(hierarchical_label "RES_HV-"
+		(shape output)
+		(at 115.57 49.53 0)
+		(effects
+			(font
+				(size 1.27 1.27)
+			)
+			(justify left)
 		)
 	)
@@
 		(shape output)
 		(at 57.15 53.34 0)
-		(effects
-			(font
-				(size 1.27 1.27)
-			)
-			(justify left)
-		)
-	)
-	(hierarchical_label "RES_HV-"
-		(shape output)
-		(at 115.57 60.96 0)
 		(effects
 			(font
@@
 					(unit 1)
 				)
-			)
-		)
-	)
-	(symbol
-		(lib_name "PWR263S-35-3300F_1")
-		(lib_id "Precharge-R:PWR263S-35-3300F")
-		(at 100.33 60.96 180)
-		(unit 1)
-		(body_style 1)
-		(exclude_from_sim no)
-		(in_bom yes)
-		(on_board yes)
-		(in_pos_files yes)
-		(dnp yes)
-		(property "Reference" "R5"
-			(at 100.33 57.912 0)
-			(show_name no)
-			(do_not_autoplace no)
-			(effects
-				(font
-					(size 1.27 1.27)
-				)
-			)
-		)
-		(property "Value" "50"
-			(at 100.584 64.262 0)
-			(show_name no)
-			(do_not_autoplace no)
-			(effects
-				(font
-					(size 1.27 1.27)
-				)
-			)
-		)
-		(property "Footprint" "Precharge_Board:RES_PWR263S-35-3300F"
-			(at 100.33 60.96 0)
-			(hide yes)
-			(show_name no)
-			(do_not_autoplace no)
-			(effects
-				(font
-					(size 1.27 1.27)
-				)
-				(justify bottom)
-			)
-		)
-		(property "Datasheet" "kicad-embed://pwr263s-35.pdf"
-			(at 100.33 60.96 0)
-			(hide yes)
-			(show_name no)
-			(do_not_autoplace no)
-			(effects
-				(font
-					(size 1.27 1.27)
-				)
-			)
-		)
-		(property "Description" "Precharge Resistor"
-			(at 100.33 60.96 0)
-			(hide yes)
-			(show_name no)
-			(do_not_autoplace no)
-			(effects
-				(font
-					(size 1.27 1.27)
-				)
-			)
-		)
-		(property "PARTREV" "12/20"
-			(at 100.33 60.96 0)
-			(hide yes)
-			(show_name no)
-			(do_not_autoplace no)
-			(effects
-				(font
-					(size 1.27 1.27)
-				)
-				(justify bottom)
-			)
-		)
-		(property "MANUFACTURER" "Bourns"
-			(at 100.33 60.96 0)
-			(hide yes)
-			(show_name no)
-			(do_not_autoplace no)
-			(effects
-				(font
-					(size 1.27 1.27)
-				)
-				(justify bottom)
-			)
-		)
-		(property "MAXIMUM_PACKAGE_HEIGHT" "4.5mm"
-			(at 100.33 60.96 0)
-			(hide yes)
-			(show_name no)
-			(do_not_autoplace no)
-			(effects
-				(font
-					(size 1.27 1.27)
-				)
-				(justify bottom)
-			)
-		)
-		(property "STANDARD" "Manufacturer Recommendations"
-			(at 100.33 60.96 0)
-			(hide yes)
-			(show_name no)
-			(do_not_autoplace no)
-			(effects
-				(font
-					(size 1.27 1.27)
-				)
-				(justify bottom)
-			)
-		)
-		(property "P/N" "  PWR263S-35-3300F"
-			(at 100.33 60.96 0)
-			(hide yes)
-			(show_name no)
-			(do_not_autoplace no)
-			(effects
-				(font
-					(size 1.27 1.27)
-				)
-			)
-		)
-		(property "Sim.Device" ""
-			(at 100.33 60.96 0)
-			(hide yes)
-			(show_name no)
-			(do_not_autoplace no)
-			(effects
-				(font
-					(size 1.27 1.27)
-				)
-			)
-		)
-		(property "Sim.Library" ""
-			(at 100.33 60.96 0)
-			(hide yes)
-			(show_name no)
-			(do_not_autoplace no)
-			(effects
-				(font
-					(size 1.27 1.27)
-				)
-			)
-		)
-		(property "Sim.Name" ""
-			(at 100.33 60.96 0)
-			(hide yes)
-			(show_name no)
-			(do_not_autoplace no)
-			(effects
-				(font
-					(size 1.27 1.27)
-				)
-			)
-		)
-		(pin "2"
-		)
-		(pin "1"
-		)
-		(pin "3"
-		)
-		(instances
-			(project "PS-PrechargeBoard"
-				(path "/74d17fe6-68d4-4bd7-954a-e2bbb58b1f1e/90c6c4b7-1465-4e8f-80ba-ec6b0750446b"
-					(reference "R36")
-					(unit 1)
-				)
-				(path "/74d17fe6-68d4-4bd7-954a-e2bbb58b1f1e/9d2e20d2-bc37-4993-8fa8-5a82459dba6b"
-					(reference "R5")
-					(unit 1)
-				)
